File: ColecoVision Clone.sch (KiCad schematic (older format))
At the start: 20 parts, among them J1 Cartridge Slot, U1 Z80CPU, U12 74LS138 (Mem. Mapped), U13 74LS138 (I/O), U14 74LS02, U19 74HC04, U2 Work RAM, U3 BIOS ROM 27C256

Commit message: /BUSRQ
Connections:
- net labels removed: !BUSACK, !BUSRQ
- wire segments 167 -> 166
- no-connect marks 11 -> 12
Changed lines of the file:
@@
 Wire Wire Line
 	1100 4175 1100 1675
-Wire Wire Line
-	1100 4175 975  4175
-Connection ~ 1100 4175
-Text GLabel 975  4175 0    50   Input ~ 0
-!BUSRQ
 $Comp
 L Device:R_Small_US R3
@@
 Wire Wire Line
 	625  1950 625  1000
-Text GLabel 1875 4275 0    50   Input ~ 0
-!BUSACK
 Connection ~ 9750 3325
 Wire Wire Line
@@
 	1    0    0    -1
 $EndComp
+NoConn ~ 1875 4275
 Wire Bus Line
 	5475 1550 5475 2950

Commit message: HALT pullup
Connections:
- net labels removed: !HALT
Changed lines of the file:
@@
 Text GLabel 1875 2475 0    50   Input ~ 0
 !NMI
-Text GLabel 625  3175 0    50   Input ~ 0
-!HALT
 Wire Wire Line
 	1875 3175 625  3175

Commit message: Fix clock circuit - v0.2
Parts:
- U19: footprint (none) -> Housings_SOIC:SOIC-14_3.9x8.7mm_Pitch1.27mm
Changed lines of the file:
@@
 F 0 "U19" H 3250 1692 50  0000 C CNN
 F 1 "74HC04" H 3250 1601 50  0000 C CNN
-F 2 "" H 3250 1375 50  0001 C CNN
+F 2 "Housings_SOIC:SOIC-14_3.9x8.7mm_Pitch1.27mm" H 3250 1375 50  0001 C CNN
 F 3 "https://assets.nexperia.com/documents/data-sheet/74HC_HCT04.pdf" H 3250 1375 50  0001 C CNN
 	4    3250 1375

Commit message: Drop a 74ls05 and use a NOR gate instead
Parts:
- removed U19: 74HC04, Housings_SOIC:SOIC-14_3.9x8.7mm_Pitch1.27mm, symbol 74xx:74HC04
- added unit 2 of U14
Connections:
- wire segments 166 -> 168
Changed lines of the file:
@@
 Wire Wire Line
 	9750 3325 10775 3325
+NoConn ~ 1875 4275
 $Comp
-L 74xx:74HC04 U19
-U 4 1 5E457D38
+L 74xx:74LS02 U14
+U 2 1 5E5C8B29
 P 3250 1375
-F 0 "U19" H 3250 1692 50  0000 C CNN
-F 1 "74HC04" H 3250 1601 50  0000 C CNN
-F 2 "Housings_SOIC:SOIC-14_3.9x8.7mm_Pitch1.27mm" H 3250 1375 50  0001 C CNN
-F 3 "https://assets.nexperia.com/documents/data-sheet/74HC_HCT04.pdf" H 3250 1375 50  0001 C CNN
-	4    3250 1375
+F 0 "U14" H 3250 1700 50  0000 C CNN
+F 1 "74LS02" H 3250 1609 50  0000 C CNN
+F 2 "" H 3250 1375 50  0001 C CNN
+F 3 "http://www.ti.com/lit/gpn/sn74ls02" H 3250 1375 50  0001 C CNN
+	2    3250 1375
 	1    0    0    -1
 $EndComp
-NoConn ~ 1875 4275
+Wire Wire Line
+	2950 1275 2950 1375
 Wire Bus Line
 	5475 1550 5475 2950
@@
 Wire Bus Line
 	3475 1550 3475 3475
+Connection ~ 2950 1375
+Wire Wire Line
+	2950 1375 2950 1475
 $EndSCHEMATC

Commit message: More DigiKey fields
Parts:
- U12, U13: DigiKey (none) -> 296-14883-2-ND
- U14: DigiKey (none) -> 1727-2829-2-ND
- U14: footprint (none) -> Housings_SOIC:SOIC-14_3.9x8.7mm_Pitch1.27mm
Changed lines of the file:
@@
 F 2 "Housings_SOIC:SOIC-16_3.9x9.9mm_Pitch1.27mm" H 4475 4150 50  0001 C CNN
 F 3 "https://www.digikey.ca/product-detail/en/texas-instruments/SN74LS138DR/296-14883-2-ND/562882" H 4475 4150 50  0001 C CNN
+F 4 "296-14883-2-ND" H 4475 4150 50  0001 C CNN "DigiKey"
 	1    4475 4150
 	1    0    0    -1
@@
 F 2 "Housings_SOIC:SOIC-16_3.9x9.9mm_Pitch1.27mm" H 4475 2425 50  0001 C CNN
 F 3 "https://www.digikey.ca/product-detail/en/texas-instruments/SN74LS138DR/296-14883-2-ND/562882" H 4475 2425 50  0001 C CNN
+F 4 "296-14883-2-ND" H 4475 2425 50  0001 C CNN "DigiKey"
 	1    4475 2425
 	1    0    0    -1
@@
 F 2 "Housings_SOIC:SOIC-14_3.9x8.7mm_Pitch1.27mm" H 7850 4200 50  0001 C CNN
 F 3 "https://www.digikey.ca/product-detail/en/nexperia-usa-inc/74HCT02D653/1727-2829-2-ND/763104" H 7850 4200 50  0001 C CNN
+F 4 "1727-2829-2-ND" H 7850 4200 50  0001 C CNN "DigiKey"
 	1    7850 4200
 	1    0    0    -1
@@
 F 0 "U14" H 3250 1700 50  0000 C CNN
 F 1 "74LS02" H 3250 1609 50  0000 C CNN
-F 2 "" H 3250 1375 50  0001 C CNN
-F 3 "http://www.ti.com/lit/gpn/sn74ls02" H 3250 1375 50  0001 C CNN
+F 2 "Housings_SOIC:SOIC-14_3.9x8.7mm_Pitch1.27mm" H 3250 1375 50  0001 C CNN
+F 3 "https://www.digikey.ca/product-detail/en/nexperia-usa-inc/74HCT02D653/1727-2829-2-ND/763104" H 3250 1375 50  0001 C CNN
 	2    3250 1375
 	1    0    0    -1

Commit message: new cart slot, hope clearance is good
Parts:
- J1: footprint Socket_Strips:Socket_Strip_Straight_2x15_Pitch2.54mm -> LeakyChips:Sullins_Cart_Slot; DigiKey (none) -> S3305-ND
Changed lines of the file:
@@
 F 0 "J1" H 9750 6167 50  0000 C CNN
 F 1 "Cartridge Slot" H 9750 6076 50  0000 C CNN
-F 2 "Socket_Strips:Socket_Strip_Straight_2x15_Pitch2.54mm" H 9700 5250 50  0001 C CNN
+F 2 "LeakyChips:Sullins_Cart_Slot" H 9700 5250 50  0001 C CNN
 F 3 "https://www.digikey.ca/product-detail/en/sullins-connector-solutions/EBC15DCWN/S3305-ND/927257" H 9700 5250 50  0001 C CNN
+F 4 "S3305-ND" H 9700 5250 50  0001 C CNN "DigiKey"
 	1    9700 5250
 	1    0    0    -1
