File: Video.sch (KiCad schematic (older format))
At the start: 2 parts, among them U4 TMS9918A

Commit message: Added a bunch of shit we don't need to distract me from doing RAM decoding
Parts:
- added C2, C3: 0.1µF, Capacitors_SMD:C_0805_HandSoldering, symbol Device:C
- added C5: 0.1µF, Capacitors_ThroughHole:CP_Radial_D4.0mm_P1.50mm, symbol Device:CP
- added J2: Composite video, Jacks:CUI_RCJ-017, symbol RCJ-017:RCJ-017
- added Q1, Q2: 2n2222, TO_SOT_Packages_THT:TO-92_Inline_Wide, symbol Device:Q_NPN_BCE
- added R1: 22Ω, Resistors_SMD:R_0805_HandSoldering, symbol Device:R_Small_US
- added U5: VRAM, LeakyChips:SOIC-40, symbol LeakoChips:LC331632M-12
Connections:
- net labels added: Composite
- wire segments 8 -> 30
Changed lines of the file:
@@
 $Descr A4 11693 8268
 encoding utf-8
-Sheet 2 2
+Sheet 2 3
 Title ""
 Date ""
@@
 $EndComp
 $Comp
-L power:VCC #PWR?
+L power:VCC #PWR0105
 U 1 1 5E38AA71
 P 6050 825
-F 0 "#PWR?" H 6050 675 50  0001 C CNN
+F 0 "#PWR0105" H 6050 675 50  0001 C CNN
 F 1 "VCC" H 6067 998 50  0000 C CNN
 F 2 "" H 6050 825 50  0001 C CNN
@@
 $EndComp
 $Comp
-L power:GND #PWR?
+L power:GND #PWR0106
 U 1 1 5E38B057
 P 5750 1325
-F 0 "#PWR?" H 5750 1075 50  0001 C CNN
+F 0 "#PWR0106" H 5750 1075 50  0001 C CNN
 F 1 "GND" H 5755 1152 50  0000 C CNN
 F 2 "" H 5750 1325 50  0001 C CNN
@@
 	4875 3200 4875 1150
 Wire Wire Line
-	4875 1150 5750 1150
+	4875 1150 5450 1150
 Connection ~ 5750 1150
+$Comp
+L LeakoChips:LC331632M-12 U5
+U 1 1 5E39317A
+P 8025 3025
+F 0 "U5" H 8050 4290 50  0000 C CNN
+F 1 "VRAM" H 8050 4199 50  0000 C CNN
+F 2 "LeakyChips:SOIC-40" H 8025 3575 50  0001 C CNN
+F 3 "https://html.alldatasheet.com/html-pdf/40652/SANYO/LC331632M-12/267/2/LC331632M-12.html" H 8025 3575 50  0001 C CNN
+	1    8025 3025
+	1    0    0    -1
+$EndComp
+$Comp
+L Device:C C2
+U 1 1 5E397437
+P 8050 1550
+F 0 "C2" V 7798 1550 50  0000 C CNN
+F 1 "0.1µF" V 7889 1550 50  0000 C CNN
+F 2 "Capacitors_SMD:C_0805_HandSoldering" H 8088 1400 50  0001 C CNN
+F 3 "~" H 8050 1550 50  0001 C CNN
+	1    8050 1550
+	0    1    1    0
+$EndComp
+$Comp
+L Device:C C3
+U 1 1 5E397A02
+P 8050 4425
+F 0 "C3" V 7798 4425 50  0000 C CNN
+F 1 "0.1µF" V 7889 4425 50  0000 C CNN
+F 2 "Capacitors_SMD:C_0805_HandSoldering" H 8088 4275 50  0001 C CNN
+F 3 "~" H 8050 4425 50  0001 C CNN
+	1    8050 4425
+	0    1    1    0
+$EndComp
+Wire Wire Line
+	7900 1550 7425 1550
+Wire Wire Line
+	5450 1550 5450 1150
+Connection ~ 5450 1150
+Wire Wire Line
+	5450 1150 5750 1150
+Wire Wire Line
+	7150 1150 8200 1150
+Wire Wire Line
+	8200 1150 8200 1550
+Connection ~ 7150 1150
+Wire Wire Line
+	8200 1550 8675 1550
+Wire Wire Line
+	8675 1550 8675 2075
+Connection ~ 8200 1550
+Wire Wire Line
+	7425 2075 7425 1550
+Connection ~ 7425 1550
+Wire Wire Line
+	7425 1550 5450 1550
+Wire Wire Line
+	7900 4425 7425 4425
+Wire Wire Line
+	7425 4425 7425 3975
+Wire Wire Line
+	8200 4425 8675 4425
+Wire Wire Line
+	8675 4425 8675 3975
+$Comp
+L power:VCC #PWR0107
+U 1 1 5E39B890
+P 8950 4425
+F 0 "#PWR0107" H 8950 4275 50  0001 C CNN
+F 1 "VCC" H 8967 4598 50  0000 C CNN
+F 2 "" H 8950 4425 50  0001 C CNN
+F 3 "" H 8950 4425 50  0001 C CNN
+	1    8950 4425
+	1    0    0    -1
+$EndComp
+$Comp
+L power:GND #PWR0108
+U 1 1 5E39C917
+P 7125 4425
+F 0 "#PWR0108" H 7125 4175 50  0001 C CNN
+F 1 "GND" H 7130 4252 50  0000 C CNN
+F 2 "" H 7125 4425 50  0001 C CNN
+F 3 "" H 7125 4425 50  0001 C CNN
+	1    7125 4425
+	1    0    0    -1
+$EndComp
+Wire Wire Line
+	7425 4425 7125 4425
+Connection ~ 7425 4425
+Wire Wire Line
+	8675 4425 8950 4425
+Connection ~ 8675 4425
+$Comp
+L Device:Q_NPN_BCE Q1
+U 1 1 5E39E220
+P 3000 1675
+F 0 "Q1" H 3191 1721 50  0000 L CNN
+F 1 "2n2222" H 3191 1630 50  0000 L CNN
+F 2 "TO_SOT_Packages_THT:TO-92_Inline_Wide" H 3200 1775 50  0001 C CNN
+F 3 "~" H 3000 1675 50  0001 C CNN
+	1    3000 1675
+	1    0    0    -1
+$EndComp
+$Comp
+L Device:Q_NPN_BCE Q2
+U 1 1 5E39E78C
+P 3375 2025
+F 0 "Q2" H 3566 2071 50  0000 L CNN
+F 1 "2n2222" H 3566 1980 50  0000 L CNN
+F 2 "TO_SOT_Packages_THT:TO-92_Inline_Wide" H 3575 2125 50  0001 C CNN
+F 3 "~" H 3375 2025 50  0001 C CNN
+	1    3375 2025
+	1    0    0    -1
+$EndComp
+Wire Wire Line
+	3175 2025 3100 2025
+Wire Wire Line
+	3100 2025 3100 1875
+$Comp
+L power:VCC #PWR0109
+U 1 1 5E39F48C
+P 3325 1050
+F 0 "#PWR0109" H 3325 900 50  0001 C CNN
+F 1 "VCC" H 3342 1223 50  0000 C CNN
+F 2 "" H 3325 1050 50  0001 C CNN
+F 3 "" H 3325 1050 50  0001 C CNN
+	1    3325 1050
+	1    0    0    -1
+$EndComp
+Wire Wire Line
+	3325 1050 3100 1050
+Wire Wire Line
+	3100 1050 3100 1475
+Wire Wire Line
+	3325 1050 3475 1050
+Wire Wire Line
+	3475 1050 3475 1825
+Connection ~ 3325 1050
+Text GLabel 6400 2500 2    50   Input ~ 0
+Composite
+Text GLabel 2800 1675 0    50   Input ~ 0
+Composite
+$Comp
+L Device:CP C5
+U 1 1 5E3A12C1
+P 3725 1200
+F 0 "C5" H 3843 1246 50  0000 L CNN
+F 1 "0.1µF" H 3843 1155 50  0000 L CNN
+F 2 "Capacitors_ThroughHole:CP_Radial_D4.0mm_P1.50mm" H 3763 1050 50  0001 C CNN
+F 3 "~" H 3725 1200 50  0001 C CNN
+	1    3725 1200
+	1    0    0    -1
+$EndComp
+$Comp
+L power:GND #PWR0110
+U 1 1 5E3A219C
+P 3725 1350
+F 0 "#PWR0110" H 3725 1100 50  0001 C CNN
+F 1 "GND" H 3730 1177 50  0000 C CNN
+F 2 "" H 3725 1350 50  0001 C CNN
+F 3 "" H 3725 1350 50  0001 C CNN
+	1    3725 1350
+	1    0    0    -1
+$EndComp
+Wire Wire Line
+	3725 1050 3475 1050
+Connection ~ 3475 1050
+$Comp
+L Device:R_Small_US R1
+U 1 1 5E3A332F
+P 3475 2325
+F 0 "R1" H 3543 2371 50  0000 L CNN
+F 1 "22Ω" H 3543 2280 50  0000 L CNN
+F 2 "Resistors_SMD:R_0805_HandSoldering" H 3475 2325 50  0001 C CNN
+F 3 "~" H 3475 2325 50  0001 C CNN
+	1    3475 2325
+	1    0    0    -1
+$EndComp
+$Comp
+L power:GND #PWR0111
+U 1 1 5E3A60DD
+P 3475 2625
+F 0 "#PWR0111" H 3475 2375 50  0001 C CNN
+F 1 "GND" H 3480 2452 50  0000 C CNN
+F 2 "" H 3475 2625 50  0001 C CNN
+F 3 "" H 3475 2625 50  0001 C CNN
+	1    3475 2625
+	1    0    0    -1
+$EndComp
+$Comp
+L RCJ-017:RCJ-017 J2
+U 1 1 5E3A6E8A
+P 3775 2525
+F 0 "J2" H 3617 2474 50  0000 R CNN
+F 1 "Composite video" H 3617 2565 50  0000 R CNN
+F 2 "Jacks:CUI_RCJ-017" H 3775 2525 50  0001 L BNN
+F 3 "CUI Inc" H 3775 2525 50  0001 L BNN
+F 4 "B" H 3775 2525 50  0001 L BNN "Field4"
+F 5 "Manufacturer recommendations" H 3775 2525 50  0001 L BNN "Field5"
+	1    3775 2525
+	-1   0    0    1
+$EndComp
 $EndSCHEMATC

Commit message: Maybe bus
Connections:
- net labels added: D0, D1, D2, D3, D4, D5, D6, D7, D[0..7]
- wire segments 30 -> 46
Changed lines of the file:
@@
 	-1   0    0    1
 $EndComp
+Text GLabel 6700 4825 0    50   BiDi ~ 0
+D[0..7]
+Wire Bus Line
+	6700 4825 6700 4700
+Wire Bus Line
+	6700 4225 5200 4225
+Wire Bus Line
+	6700 4700 6975 4700
+Wire Bus Line
+	6975 4700 6975 4225
+Connection ~ 6700 4700
+Wire Bus Line
+	6700 4700 6700 4225
+Wire Wire Line
+	7425 3175 7225 3175
+Wire Wire Line
+	7425 3275 7225 3275
+Wire Wire Line
+	7425 3375 7225 3375
+Wire Wire Line
+	7425 3475 7225 3475
+Wire Wire Line
+	7425 3575 7225 3575
+Wire Wire Line
+	7425 3675 7225 3675
+Wire Wire Line
+	7425 3775 7225 3775
+Wire Wire Line
+	7425 3875 7225 3875
+Entry Wire Line
+	7125 3075 7225 3175
+Entry Wire Line
+	7125 3175 7225 3275
+Entry Wire Line
+	7125 3275 7225 3375
+Entry Wire Line
+	7125 3375 7225 3475
+Entry Wire Line
+	7125 3475 7225 3575
+Entry Wire Line
+	7125 3575 7225 3675
+Entry Wire Line
+	7125 3675 7225 3775
+Entry Wire Line
+	7125 3775 7225 3875
+Wire Bus Line
+	6975 4225 7125 4225
+Text Label 7425 3175 2    50   ~ 0
+D0
+Text Label 7425 3275 2    50   ~ 0
+D1
+Text Label 7425 3375 2    50   ~ 0
+D2
+Text Label 7425 3475 2    50   ~ 0
+D3
+Text Label 7425 3575 2    50   ~ 0
+D4
+Text Label 7425 3675 2    50   ~ 0
+D5
+Text Label 7425 3775 2    50   ~ 0
+D6
+Text Label 7425 3875 2    50   ~ 0
+D7
+Text Label 6400 3700 0    50   ~ 0
+D0
+Text Label 6400 3800 0    50   ~ 0
+D1
+Text Label 6400 3900 0    50   ~ 0
+D2
+Text Label 6400 4000 0    50   ~ 0
+D3
+Text Label 5400 4000 2    50   ~ 0
+D4
+Text Label 5400 3900 2    50   ~ 0
+D5
+Text Label 5400 3800 2    50   ~ 0
+D6
+Text Label 5400 3700 2    50   ~ 0
+D7
+Entry Wire Line
+	6600 3700 6700 3800
+Entry Wire Line
+	6600 3800 6700 3900
+Entry Wire Line
+	6600 3900 6700 4000
+Entry Wire Line
+	6600 4000 6700 4100
+Wire Wire Line
+	6400 3700 6600 3700
+Wire Wire Line
+	6400 3800 6600 3800
+Wire Wire Line
+	6400 3900 6600 3900
+Wire Wire Line
+	6400 4000 6600 4000
+Connection ~ 6700 4225
+Wire Wire Line
+	5400 4000 5300 4000
+Wire Wire Line
+	5400 3900 5300 3900
+Wire Wire Line
+	5400 3800 5300 3800
+Wire Wire Line
+	5400 3700 5300 3700
+Entry Wire Line
+	5200 3600 5300 3700
+Entry Wire Line
+	5200 3700 5300 3800
+Entry Wire Line
+	5200 3800 5300 3900
+Entry Wire Line
+	5200 3900 5300 4000
+Wire Bus Line
+	6700 3800 6700 4225
+Wire Bus Line
+	5200 3600 5200 4225
+Wire Bus Line
+	7125 3075 7125 4225
 $EndSCHEMATC

Commit message: Blindly hooking up vram bus
Connections:
- net labels added: RD[0..7], Reset, VD0, VD1, VD2, VD3, VD4, VD5, VD6, VD7, VD[0..7]
- wire segments 46 -> 54
Changed lines of the file:
@@
 D[0..7]
 Wire Bus Line
-	6700 4825 6700 4700
-Wire Bus Line
 	6700 4225 5200 4225
-Wire Bus Line
-	6700 4700 6975 4700
-Wire Bus Line
-	6975 4700 6975 4225
-Connection ~ 6700 4700
-Wire Bus Line
-	6700 4700 6700 4225
 Wire Wire Line
 	7425 3175 7225 3175
@@
 Wire Wire Line
 	7425 3875 7225 3875
-Entry Wire Line
-	7125 3075 7225 3175
-Entry Wire Line
-	7125 3175 7225 3275
-Entry Wire Line
-	7125 3275 7225 3375
-Entry Wire Line
-	7125 3375 7225 3475
-Entry Wire Line
-	7125 3475 7225 3575
-Entry Wire Line
-	7125 3575 7225 3675
-Entry Wire Line
-	7125 3675 7225 3775
-Entry Wire Line
-	7125 3775 7225 3875
-Wire Bus Line
-	6975 4225 7125 4225
 Text Label 7425 3175 2    50   ~ 0
-D0
+VD0
 Text Label 7425 3275 2    50   ~ 0
-D1
+VD1
 Text Label 7425 3375 2    50   ~ 0
-D2
+VD2
 Text Label 7425 3475 2    50   ~ 0
-D3
+VD3
 Text Label 7425 3575 2    50   ~ 0
-D4
+VD4
 Text Label 7425 3675 2    50   ~ 0
-D5
+VD5
 Text Label 7425 3775 2    50   ~ 0
-D6
+VD6
 Text Label 7425 3875 2    50   ~ 0
-D7
+VD7
 Text Label 6400 3700 0    50   ~ 0
 D0
@@
 	5200 3900 5300 4000
 Wire Bus Line
+	6700 4225 6700 4825
+Entry Wire Line
+	7125 3775 7225 3875
+Entry Wire Line
+	7125 3675 7225 3775
+Entry Wire Line
+	7125 3575 7225 3675
+Entry Wire Line
+	7125 3475 7225 3575
+Entry Wire Line
+	7125 3375 7225 3475
+Entry Wire Line
+	7125 3275 7225 3375
+Entry Wire Line
+	7125 3175 7225 3275
+Entry Wire Line
+	7125 3075 7225 3175
+Wire Wire Line
+	6400 3600 6600 3600
+Wire Wire Line
+	6400 3500 6600 3500
+Wire Wire Line
+	6400 3400 6600 3400
+Wire Wire Line
+	6400 3300 6600 3300
+Wire Wire Line
+	6400 3200 6600 3200
+Wire Wire Line
+	6400 3100 6600 3100
+Wire Wire Line
+	6400 3000 6600 3000
+Wire Wire Line
+	6400 2900 6600 2900
+Entry Wire Line
+	6600 3600 6700 3700
+Entry Wire Line
+	6600 3500 6700 3600
+Entry Wire Line
+	6600 3400 6700 3500
+Entry Wire Line
+	6600 3300 6700 3400
+Entry Wire Line
+	6600 3200 6700 3300
+Entry Wire Line
+	6600 3100 6700 3200
+Entry Wire Line
+	6600 3000 6700 3100
+Entry Wire Line
+	6600 2900 6700 3000
+Wire Bus Line
+	6700 3000 7125 3000
+Wire Bus Line
 	6700 3800 6700 4225
 Wire Bus Line
 	5200 3600 5200 4225
 Wire Bus Line
-	7125 3075 7125 4225
+	6700 3000 6700 3700
+Wire Bus Line
+	7125 3000 7125 3775
+Text Label 7125 3025 0    50   ~ 0
+VD[0..7]
+Text Label 6800 3000 3    50   ~ 0
+RD[0..7]
+Text Label 6400 3600 0    50   ~ 0
+VD7
+Text Label 6400 3500 0    50   ~ 0
+VD6
+Text Label 6400 3400 0    50   ~ 0
+VD5
+Text Label 6400 3300 0    50   ~ 0
+VD4
+Text Label 6400 3200 0    50   ~ 0
+VD3
+Text Label 6400 3100 0    50   ~ 0
+VD2
+Text Label 6400 3000 0    50   ~ 0
+VD1
+Text Label 6400 2900 0    50   ~ 0
+VD0
+Text GLabel 6400 2700 2    50   Input ~ 0
+Reset
 $EndSCHEMATC

Commit message: Not sure I know enough to set up the VRAM bus yet
Parts:
- removed C5: 0.1µF, Capacitors_ThroughHole:CP_Radial_D4.0mm_P1.50mm, symbol Device:CP
- removed Q1, Q2: 2n2222, TO_SOT_Packages_THT:TO-92_Inline_Wide, symbol Device:Q_NPN_BCE
- R1: value 22Ω -> 470Ω
Connections:
- net labels added: A0, A[0..7]
- wire segments 54 -> 63
Other:
- note added: ""Bit order numbering is backwards. 0 is the MSB and 7 is the LSB."\nTODO: invert CPU bus?"
- note added: "Composite video jack"
Changed lines of the file:
@@
 	8675 4425 8950 4425
 Connection ~ 8675 4425
-$Comp
-L Device:Q_NPN_BCE Q1
-U 1 1 5E39E220
-P 3000 1675
-F 0 "Q1" H 3191 1721 50  0000 L CNN
-F 1 "2n2222" H 3191 1630 50  0000 L CNN
-F 2 "TO_SOT_Packages_THT:TO-92_Inline_Wide" H 3200 1775 50  0001 C CNN
-F 3 "~" H 3000 1675 50  0001 C CNN
-	1    3000 1675
-	1    0    0    -1
-$EndComp
-$Comp
-L Device:Q_NPN_BCE Q2
-U 1 1 5E39E78C
-P 3375 2025
-F 0 "Q2" H 3566 2071 50  0000 L CNN
-F 1 "2n2222" H 3566 1980 50  0000 L CNN
-F 2 "TO_SOT_Packages_THT:TO-92_Inline_Wide" H 3575 2125 50  0001 C CNN
-F 3 "~" H 3375 2025 50  0001 C CNN
-	1    3375 2025
-	1    0    0    -1
-$EndComp
-Wire Wire Line
-	3175 2025 3100 2025
-Wire Wire Line
-	3100 2025 3100 1875
-$Comp
-L power:VCC #PWR0109
-U 1 1 5E39F48C
-P 3325 1050
-F 0 "#PWR0109" H 3325 900 50  0001 C CNN
-F 1 "VCC" H 3342 1223 50  0000 C CNN
-F 2 "" H 3325 1050 50  0001 C CNN
-F 3 "" H 3325 1050 50  0001 C CNN
-	1    3325 1050
-	1    0    0    -1
-$EndComp
-Wire Wire Line
-	3325 1050 3100 1050
-Wire Wire Line
-	3100 1050 3100 1475
-Wire Wire Line
-	3325 1050 3475 1050
-Wire Wire Line
-	3475 1050 3475 1825
-Connection ~ 3325 1050
 Text GLabel 6400 2500 2    50   Input ~ 0
 Composite
-Text GLabel 2800 1675 0    50   Input ~ 0
+Text GLabel 2300 1675 0    50   Input ~ 0
 Composite
-$Comp
-L Device:CP C5
-U 1 1 5E3A12C1
-P 3725 1200
-F 0 "C5" H 3843 1246 50  0000 L CNN
-F 1 "0.1µF" H 3843 1155 50  0000 L CNN
-F 2 "Capacitors_ThroughHole:CP_Radial_D4.0mm_P1.50mm" H 3763 1050 50  0001 C CNN
-F 3 "~" H 3725 1200 50  0001 C CNN
-	1    3725 1200
-	1    0    0    -1
-$EndComp
-$Comp
-L power:GND #PWR0110
-U 1 1 5E3A219C
-P 3725 1350
-F 0 "#PWR0110" H 3725 1100 50  0001 C CNN
-F 1 "GND" H 3730 1177 50  0000 C CNN
-F 2 "" H 3725 1350 50  0001 C CNN
-F 3 "" H 3725 1350 50  0001 C CNN
-	1    3725 1350
-	1    0    0    -1
-$EndComp
-Wire Wire Line
-	3725 1050 3475 1050
-Connection ~ 3475 1050
-$Comp
-L Device:R_Small_US R1
-U 1 1 5E3A332F
-P 3475 2325
-F 0 "R1" H 3543 2371 50  0000 L CNN
-F 1 "22Ω" H 3543 2280 50  0000 L CNN
-F 2 "Resistors_SMD:R_0805_HandSoldering" H 3475 2325 50  0001 C CNN
-F 3 "~" H 3475 2325 50  0001 C CNN
-	1    3475 2325
-	1    0    0    -1
-$EndComp
 $Comp
 L power:GND #PWR0111
@@
 Wire Bus Line
 	6700 3000 7125 3000
-Wire Bus Line
-	6700 3800 6700 4225
-Wire Bus Line
-	5200 3600 5200 4225
-Wire Bus Line
-	6700 3000 6700 3700
-Wire Bus Line
-	7125 3000 7125 3775
-Text Label 7125 3025 0    50   ~ 0
-VD[0..7]
 Text Label 6800 3000 3    50   ~ 0
 RD[0..7]
@@
 Text GLabel 6400 2700 2    50   Input ~ 0
 Reset
+Wire Notes Line
+	4650 800  4650 2950
+Wire Notes Line
+	4650 2950 1775 2950
+Wire Notes Line
+	1775 2950 1775 800
+Wire Notes Line
+	1775 800  4650 800
+Text Notes 1825 2900 0    50   ~ 0
+Composite video jack
+Wire Wire Line
+	3475 1675 3475 2425
+$Comp
+L Device:R_Small_US R1
+U 1 1 5E424465
+P 2800 2000
+F 0 "R1" H 2868 2046 50  0000 L CNN
+F 1 "470Ω" H 2868 1955 50  0000 L CNN
+F 2 "Resistors_SMD:R_0805_HandSoldering" H 2800 2000 50  0001 C CNN
+F 3 "~" H 2800 2000 50  0001 C CNN
+	1    2800 2000
+	1    0    0    -1
+$EndComp
+Wire Wire Line
+	3475 2625 2800 2625
+Wire Wire Line
+	2800 2625 2800 2100
+Connection ~ 3475 2625
+Wire Wire Line
+	2300 1675 2800 1675
+Wire Wire Line
+	2800 1900 2800 1675
+Connection ~ 2800 1675
+Wire Wire Line
+	2800 1675 3475 1675
+Text Notes 3900 4500 0    50   ~ 0
+"Bit order numbering is backwards. 0 is the MSB and 7 is the LSB."\nTODO: invert CPU bus?
+Wire Wire Line
+	5400 3300 4650 3300
+Wire Bus Line
+	4350 3200 4350 4075
+Entry Wire Line
+	4550 3200 4650 3300
+Text Label 5400 3300 2    50   ~ 0
+A0
+Text GLabel 4350 4075 0    50   Input ~ 0
+A[0..7]
+Wire Wire Line
+	5400 3100 5325 3100
+Wire Wire Line
+	5400 3000 5325 3000
+Wire Wire Line
+	5400 2900 5325 2900
+Wire Wire Line
+	5400 2800 5325 2800
+Wire Wire Line
+	5400 2700 5325 2700
+Wire Wire Line
+	5400 2600 5325 2600
+Wire Wire Line
+	5400 2500 5325 2500
+Wire Wire Line
+	5400 2400 5325 2400
+Wire Wire Line
+	5400 2300 5325 2300
+Text Label 7125 3025 0    50   ~ 0
+VD[0..7]
+Wire Bus Line
+	4350 3200 4700 3200
+Wire Bus Line
+	6700 3000 6700 3700
+Wire Bus Line
+	7125 3000 7125 3775
+Wire Bus Line
+	5200 3600 5200 4225
+Wire Bus Line
+	6700 3800 6700 4225
 $EndSCHEMATC

Commit message: Get rid of RD0 speculation
Connections:
- net labels removed: RD[0..7], VD[0..7]
- wire segments 63 -> 46
Changed lines of the file:
@@
 Wire Bus Line
 	6700 4225 5200 4225
-Wire Wire Line
-	7425 3175 7225 3175
-Wire Wire Line
-	7425 3275 7225 3275
-Wire Wire Line
-	7425 3375 7225 3375
-Wire Wire Line
-	7425 3475 7225 3475
-Wire Wire Line
-	7425 3575 7225 3575
-Wire Wire Line
-	7425 3675 7225 3675
-Wire Wire Line
-	7425 3775 7225 3775
-Wire Wire Line
-	7425 3875 7225 3875
-Text Label 7425 3175 2    50   ~ 0
-VD0
-Text Label 7425 3275 2    50   ~ 0
-VD1
-Text Label 7425 3375 2    50   ~ 0
-VD2
-Text Label 7425 3475 2    50   ~ 0
-VD3
-Text Label 7425 3575 2    50   ~ 0
-VD4
-Text Label 7425 3675 2    50   ~ 0
-VD5
-Text Label 7425 3775 2    50   ~ 0
-VD6
-Text Label 7425 3875 2    50   ~ 0
-VD7
 Text Label 6400 3700 0    50   ~ 0
 D0
@@
 D7
 Entry Wire Line
-	6600 3700 6700 3800
-Entry Wire Line
 	6600 3800 6700 3900
 Entry Wire Line
@@
 Entry Wire Line
 	6600 4000 6700 4100
-Wire Wire Line
-	6400 3700 6600 3700
 Wire Wire Line
 	6400 3800 6600 3800
@@
 Wire Bus Line
 	6700 4225 6700 4825
-Entry Wire Line
-	7125 3775 7225 3875
-Entry Wire Line
-	7125 3675 7225 3775
-Entry Wire Line
-	7125 3575 7225 3675
-Entry Wire Line
-	7125 3475 7225 3575
-Entry Wire Line
-	7125 3375 7225 3475
-Entry Wire Line
-	7125 3275 7225 3375
-Entry Wire Line
-	7125 3175 7225 3275
-Entry Wire Line
-	7125 3075 7225 3175
-Wire Wire Line
-	6400 3600 6600 3600
-Wire Wire Line
-	6400 3500 6600 3500
-Wire Wire Line
-	6400 3400 6600 3400
-Wire Wire Line
-	6400 3300 6600 3300
-Wire Wire Line
-	6400 3200 6600 3200
-Wire Wire Line
-	6400 3100 6600 3100
-Wire Wire Line
-	6400 3000 6600 3000
-Wire Wire Line
-	6400 2900 6600 2900
-Entry Wire Line
-	6600 3600 6700 3700
-Entry Wire Line
-	6600 3500 6700 3600
-Entry Wire Line
-	6600 3400 6700 3500
-Entry Wire Line
-	6600 3300 6700 3400
-Entry Wire Line
-	6600 3200 6700 3300
-Entry Wire Line
-	6600 3100 6700 3200
-Entry Wire Line
-	6600 3000 6700 3100
-Entry Wire Line
-	6600 2900 6700 3000
-Wire Bus Line
-	6700 3000 7125 3000
-Text Label 6800 3000 3    50   ~ 0
-RD[0..7]
 Text Label 6400 3600 0    50   ~ 0
 VD7
@@
 Wire Wire Line
 	5400 2300 5325 2300
-Text Label 7125 3025 0    50   ~ 0
-VD[0..7]
 Wire Bus Line
 	4350 3200 4700 3200
 Wire Bus Line
-	6700 3000 6700 3700
-Wire Bus Line
-	7125 3000 7125 3775
-Wire Bus Line
 	5200 3600 5200 4225

Commit message: COMVID and Crystal from PDF
Parts:
- added C1, C2: 27pF, Capacitors_SMD:C_0805_HandSoldering, symbol Device:CP1_Small
- added C3: 0.1µF, Capacitors_SMD:C_0805_HandSoldering, symbol Device:CP1_Small
- added FB1: Bead, Choke_SMD:Choke_SMD_1206_Handsoldering, symbol Device:Ferrite_Bead_Small
- added Q1: 2n4401, TO_SOT_Packages_THT:TO-92_Molded_Narrow, symbol Device:Q_NPN_Darlington_BCE
- added R4: 0Ω, Resistors_SMD:R_0805_HandSoldering, symbol Device:R_Small_US
- added R6: 75Ω, Resistors_SMD:R_0805_HandSoldering, symbol Device:R_Small_US
- added Y1: 10.7MHz, Crystals:Crystal_HC49-U_Vertical, symbol Device:Crystal
- renumbered C1 to C4, C2 to C5, C3 to C6, R1 to R5, U4 to U3, U5 to U4
Connections:
- net labels added: VIDVCC, XTAL1, XTAL2
- wire segments 46 -> 55
Other:
- note added: "TMS99x8 Crystal"

Commit message: Entire VRAM decoder laid out
Parts:
- added C4, C6, C7, C8: 0.1µF, Capacitors_SMD:C_0805_HandSoldering, symbol Device:C
- added U3: 74HCT04, Housings_SOIC:SOIC-14_3.9x8.7mm_Pitch1.27mm, symbol 74xx:74HCT04
- added U5, U6, U7: 74LS574, Housings_SOIC:SOIC-20W_7.5x12.8mm_Pitch1.27mm, symbol 74xx:74LS574
- renumbered C6 to C10, C4 to C5, C5 to C9, U3 to U4, U4 to U8
Connections:
- net labels added: AD0, AD1, AD2, AD3, AD4, AD5, AD6, AD7, CAS, COL, P35, P37, P38, RAM_A0, RAM_A1, RAM_A10, RAM_A11, RAM_A12, RAM_A13, RAM_A2, RAM_A3, RAM_A4, RAM_A5, RAM_A6, RAM_A7, RAM_A8, RAM_A9, RAS, RD, ROW, RW, VDP_RD, VDP_WR, VIRQ, WR
- wire segments 55 -> 108
- no-connect marks 0 -> 12
Other:
- note added: "CD0 = MSB, CD7 = LSB!!! Be careful!"
- note added: "TODO: Should the upper byte be tied to ground,\ninstead of floating? Nothing uses those data lines..."
- note removed: ""Bit order numbering is backwards. 0 is the MSB and 7 is the LSB."\nTODO: invert CPU bus?"

Commit message: little notes
Other:
- note added: "TODO: Does RD\nactually go anywhere?"
Changed lines of the file:
@@
 Wire Wire Line
 	4250 7500 4375 7500
-Wire Bus Line
-	4350 3200 4700 3200
-Wire Bus Line
-	5200 3600 5200 4225
-Wire Bus Line
-	6700 3800 6700 4225
 Connection ~ 5375 7500
 Connection ~ 4375 7500
@@
 Wire Wire Line
 	4750 7000 4675 7000
+Wire Bus Line
+	4350 3200 4700 3200
+Wire Bus Line
+	5200 3600 5200 4225
+Wire Bus Line
+	6700 3800 6700 4225
+Text Notes 4325 6300 0    50   ~ 0
+TODO: Does RD\nactually go anywhere?
 $EndSCHEMATC
