File: Video.sch (KiCad schematic (older format))
At the start: 21 parts, among them J2 Composite video, Q1 2n4401, U4 74HCT04, U5 TMS9918A, U6 74LS574, U7 74LS574, U8 74LS574, U9 VRAM

Commit message: Move RAMs to J-lead package
Parts:
- U9: footprint LeakyChips:SOIC-40 -> LeakyChips:SOIC-40-JLead
Changed lines of the file:
@@
 F 0 "U9" H 10175 4765 50  0000 C CNN
 F 1 "VRAM" H 10175 4674 50  0000 C CNN
-F 2 "LeakyChips:SOIC-40" H 10150 4050 50  0001 C CNN
+F 2 "LeakyChips:SOIC-40-JLead" H 10150 4050 50  0001 C CNN
 F 3 "https://html.alldatasheet.com/html-pdf/40652/SANYO/LC331632M-12/267/2/LC331632M-12.html" H 10150 4050 50  0001 C CNN
 	1    10150 3500

Commit message: Pull-ups on WRAM and VRAM upper byte
Parts:
- added R?: 2kΩ, Resistors_SMD:R_0805_HandSoldering, symbol Device:R_Small_US
Connections:
- net labels added: VRAM_Upper_Byte_PU
- wire segments 102 -> 125
- no-connect marks 17 -> 7
Other:
- note removed: "TODO: Should the upper byte be tied to ground,\ninstead of floating? Nothing uses those data lines..."
Changed lines of the file:
@@
 Connection ~ 5750 1150
-$Comp
-L LeakoChips:LC331632M-12 U9
-U 1 1 5E39317A
-P 10150 3500
-F 0 "U9" H 10175 4765 50  0000 C CNN
-F 1 "VRAM" H 10175 4674 50  0000 C CNN
-F 2 "LeakyChips:SOIC-40-JLead" H 10150 4050 50  0001 C CNN
-F 3 "https://html.alldatasheet.com/html-pdf/40652/SANYO/LC331632M-12/267/2/LC331632M-12.html" H 10150 4050 50  0001 C CNN
-	1    10150 3500
-	1    0    0    -1
-$EndComp
 $Comp
 L Device:C C10
@@
 	10325 2025 10800 2025
 Wire Wire Line
-	10800 2025 10800 2550
+	10800 2025 10800 2125
 Connection ~ 10325 2025
 Wire Wire Line
@@
 Text GLabel 10800 3550 2    50   Input ~ 0
 CAS
-NoConn ~ 10800 3350
-NoConn ~ 10800 2650
-NoConn ~ 10800 3650
-NoConn ~ 10800 3750
-NoConn ~ 10800 3850
-NoConn ~ 10800 3950
-NoConn ~ 10800 4050
-NoConn ~ 10800 4150
-NoConn ~ 10800 4250
-NoConn ~ 10800 4350
-Text Notes 11100 1600 2    50   ~ 0
-TODO: Should the upper byte be tied to ground,\ninstead of floating? Nothing uses those data lines...
 Text GLabel 7475 2975 0    50   Input ~ 0
 AD0
@@
 NoConn ~ 6400 2300
 NoConn ~ 4675 6400
+$Comp
+L Device:R_Small_US R?
+U 1 1 5E88CCE0
+P 11100 2325
+F 0 "R?" H 11033 2279 50  0000 R CNN
+F 1 "2kΩ" H 11033 2370 50  0000 R CNN
+F 2 "Resistors_SMD:R_0805_HandSoldering" H 11100 2325 50  0001 C CNN
+F 3 "~" H 11100 2325 50  0001 C CNN
+	1    11100 2325
+	1    0    0    1
+$EndComp
+Wire Wire Line
+	10800 2650 11100 2650
+Wire Wire Line
+	11100 2650 11100 2425
+$Comp
+L LeakoChips:LC331632M-12 U9
+U 1 1 5E39317A
+P 10150 3500
+F 0 "U9" H 10175 4765 50  0000 C CNN
+F 1 "VRAM" H 10175 4674 50  0000 C CNN
+F 2 "LeakyChips:SOIC-40-JLead" H 10150 4050 50  0001 C CNN
+F 3 "https://html.alldatasheet.com/html-pdf/40652/SANYO/LC331632M-12/267/2/LC331632M-12.html" H 10150 4050 50  0001 C CNN
+	1    10150 3500
+	1    0    0    -1
+$EndComp
+Wire Wire Line
+	11100 2225 11100 2125
+Wire Wire Line
+	11100 2125 10800 2125
+Connection ~ 10800 2125
+Wire Wire Line
+	10800 2125 10800 2550
+Wire Wire Line
+	11100 2650 11100 3350
+Wire Wire Line
+	11100 3350 10800 3350
+Connection ~ 11100 2650
+Wire Wire Line
+	11100 3350 11100 3650
+Wire Wire Line
+	11100 3650 10800 3650
+Connection ~ 11100 3350
+Wire Wire Line
+	10800 4350 11100 4350
+Connection ~ 11100 3650
+Wire Wire Line
+	10800 3750 11100 3750
+Connection ~ 11100 3750
+Wire Wire Line
+	11100 3750 11100 3650
+Wire Wire Line
+	10800 3850 11100 3850
+Connection ~ 11100 3850
+Wire Wire Line
+	11100 3850 11100 3750
+Wire Wire Line
+	10800 3950 11100 3950
+Connection ~ 11100 3950
+Wire Wire Line
+	11100 3950 11100 3850
+Wire Wire Line
+	10800 4050 11100 4050
+Connection ~ 11100 4050
+Wire Wire Line
+	11100 4050 11100 3950
+Wire Wire Line
+	10800 4150 11100 4150
+Connection ~ 11100 4150
+Wire Wire Line
+	11100 4150 11100 4050
+Wire Wire Line
+	11100 4350 11100 4250
+Wire Wire Line
+	10800 4250 11100 4250
 Wire Bus Line
 	4350 3200 4700 3200
@@
 Wire Bus Line
 	6700 3800 6700 4225
+Connection ~ 11100 4250
+Wire Wire Line
+	11100 4250 11100 4150
+Text Label 11100 2525 0    50   ~ 0
+VRAM_Upper_Byte_PU
 $EndSCHEMATC

Commit message: Numbering
Parts:
- gave numbers to parts that had none: 1
Changed lines of the file:
@@
 NoConn ~ 4675 6400
 $Comp
-L Device:R_Small_US R?
+L Device:R_Small_US R46
 U 1 1 5E88CCE0
 P 11100 2325
-F 0 "R?" H 11033 2279 50  0000 R CNN
+F 0 "R46" H 11033 2279 50  0000 R CNN
 F 1 "2kΩ" H 11033 2370 50  0000 R CNN
 F 2 "Resistors_SMD:R_0805_HandSoldering" H 11100 2325 50  0001 C CNN

Commit message: Remapped VRAM SRAM according to https://www.leonardomiliani.com/en/2019/lm80c-tms9918a/
Other:
- note added: "Note address pins are not in numerical\norder - changed to improve reliability\nof slow RAM"
- note added: "leonardomiliani.com/en/2019/lm80c-tms9918a/"
Changed lines of the file:
@@
 Text GLabel 5400 2200 0    50   Input ~ 0
 CAS
-Text GLabel 10800 3150 2    50   Input ~ 0
-RAM_A13
-Text GLabel 10800 3050 2    50   Input ~ 0
-RAM_A12
-Text GLabel 10800 2950 2    50   Input ~ 0
-RAM_A11
-Text GLabel 10800 2850 2    50   Input ~ 0
-RAM_A10
 Text GLabel 9550 3650 0    50   Input ~ 0
 VD0
@@
 Text GLabel 8475 3675 2    50   Input ~ 0
 RAM_A6
-Text GLabel 9550 3550 0    50   Input ~ 0
-RAM_A0
-Text GLabel 9550 3450 0    50   Input ~ 0
-RAM_A1
-Text GLabel 9550 3350 0    50   Input ~ 0
-RAM_A2
-Text GLabel 9550 3250 0    50   Input ~ 0
-RAM_A3
-Text GLabel 9550 3150 0    50   Input ~ 0
-RAM_A4
-Text GLabel 9550 3050 0    50   Input ~ 0
-RAM_A5
-Text GLabel 9550 2950 0    50   Input ~ 0
-RAM_A6
-Text GLabel 9550 2850 0    50   Input ~ 0
-RAM_A7
-Text GLabel 9550 2750 0    50   Input ~ 0
-RAM_A8
-Text GLabel 9550 2650 0    50   Input ~ 0
-RAM_A9
-Text GLabel 10800 3250 2    50   Input ~ 0
-RAM_A13
 Text GLabel 10800 2750 2    50   Input ~ 0
 RW
@@
 Wire Wire Line
 	10800 4250 11100 4250
+Connection ~ 11100 4250
+Wire Wire Line
+	11100 4250 11100 4150
+Text Label 11100 2525 0    50   ~ 0
+VRAM_Upper_Byte_PU
+Text Notes 9400 5350 0    50   ~ 0
+Note address pins are not in numerical\norder - changed to improve reliability\nof slow RAM
 Wire Bus Line
 	4350 3200 4700 3200
@@
 Wire Bus Line
 	6700 3800 6700 4225
-Connection ~ 11100 4250
-Wire Wire Line
-	11100 4250 11100 4150
-Text Label 11100 2525 0    50   ~ 0
-VRAM_Upper_Byte_PU
+Text GLabel 9550 3550 0    50   Input ~ 0
+RAM_A0
+Text GLabel 9550 3450 0    50   Input ~ 0
+RAM_A1
+Text GLabel 9550 3350 0    50   Input ~ 0
+RAM_A2
+Text GLabel 9550 3250 0    50   Input ~ 0
+RAM_A3
+Text GLabel 9550 3150 0    50   Input ~ 10
+RAM_A5
+Text GLabel 9550 3050 0    50   Input ~ 0
+RAM_A6
+Text GLabel 9550 2950 0    50   Input ~ 10
+RAM_A8
+Text GLabel 9550 2850 0    50   Input ~ 0
+RAM_A9
+Text GLabel 9550 2750 0    50   Input ~ 10
+RAM_A12
+Text GLabel 9550 2650 0    50   Input ~ 0
+RAM_A10
+Text GLabel 10800 2850 2    50   Input ~ 0
+RAM_A4
+Text GLabel 10800 2950 2    50   Input ~ 0
+RAM_A7
+Text GLabel 10800 3050 2    50   Input ~ 0
+RAM_A11
+Text GLabel 10800 3150 2    50   Input ~ 0
+RAM_A13
+Text GLabel 10800 3250 2    50   Input Italic 0
+RAM_A13
+Text Notes 11050 5475 2    50   Italic 0
+leonardomiliani.com/en/2019/lm80c-tms9918a/
 $EndSCHEMATC

Commit message: Attach U11 to power, add dedicated crystal for TMS
Parts:
- added C23, C26: 33pF, Capacitors_SMD:C_0805_HandSoldering, symbol Device:C_Small
- added Y1: 10.738635MHZ, Crystals:Crystal_HC49-U_Vertical, symbol Device:Crystal
Connections:
- net labels removed: VID_CLK
- wire segments 125 -> 132
- no-connect marks 7 -> 6
Changed lines of the file:
@@
 Text Notes 6975 2725 2    50   ~ 0
 EXT_VDP_RESET
-NoConn ~ 6400 2200
-Text GLabel 6400 2100 2    50   Input ~ 0
-VID_CLK
 NoConn ~ 6400 2400
 NoConn ~ 6400 2600
@@
 Text Notes 9400 5350 0    50   ~ 0
 Note address pins are not in numerical\norder - changed to improve reliability\nof slow RAM
-Wire Bus Line
-	4350 3200 4700 3200
-Wire Bus Line
-	5200 3600 5200 4225
-Wire Bus Line
-	6700 3800 6700 4225
 Text GLabel 9550 3550 0    50   Input ~ 0
 RAM_A0
@@
 Text Notes 11050 5475 2    50   Italic 0
 leonardomiliani.com/en/2019/lm80c-tms9918a/
+$Comp
+L Device:Crystal Y1
+U 1 1 5E875480
+P 6525 1575
+F 0 "Y1" H 6525 1307 50  0000 C CNN
+F 1 "10.738635MHZ" H 6525 1398 50  0000 C CNN
+F 2 "Crystals:Crystal_HC49-U_Vertical" H 6525 1575 50  0001 C CNN
+F 3 "~" H 6525 1575 50  0001 C CNN
+F 4 "CTX1443-ND" H 6525 1575 50  0001 C CNN "DigiKey"
+	1    6525 1575
+	-1   0    0    1
+$EndComp
+$Comp
+L Device:C_Small C26
+U 1 1 5E87AEF5
+P 6800 1675
+F 0 "C26" H 6892 1721 50  0000 L CNN
+F 1 "33pF" H 6892 1630 50  0000 L CNN
+F 2 "Capacitors_SMD:C_0805_HandSoldering" H 6800 1675 50  0001 C CNN
+F 3 "~" H 6800 1675 50  0001 C CNN
+	1    6800 1675
+	1    0    0    -1
+$EndComp
+$Comp
+L Device:C_Small C23
+U 1 1 5E87B8DE
+P 6250 1675
+F 0 "C23" H 6159 1629 50  0000 R CNN
+F 1 "33pF" H 6159 1720 50  0000 R CNN
+F 2 "Capacitors_SMD:C_0805_HandSoldering" H 6250 1675 50  0001 C CNN
+F 3 "~" H 6250 1675 50  0001 C CNN
+	1    6250 1675
+	1    0    0    1
+$EndComp
+Wire Wire Line
+	6400 2100 6400 1850
+Wire Wire Line
+	6400 1850 6250 1850
+Wire Wire Line
+	6250 1850 6250 1775
+Wire Wire Line
+	6400 2200 6800 2200
+Wire Wire Line
+	6800 2200 6800 1775
+Wire Wire Line
+	6675 1575 6800 1575
+Wire Wire Line
+	6375 1575 6250 1575
+Wire Bus Line
+	4350 3200 4700 3200
+Wire Bus Line
+	5200 3600 5200 4225
+Wire Bus Line
+	6700 3800 6700 4225
 $EndSCHEMATC

Commit message: Add DigiKey part number for 33pF clock caps
Parts:
- C23, C26: DigiKey (none) -> 732-7817-1-ND
Changed lines of the file:
@@
 F 2 "Capacitors_SMD:C_0805_HandSoldering" H 6800 1675 50  0001 C CNN
 F 3 "~" H 6800 1675 50  0001 C CNN
+F 4 "732-7817-1-ND" H 6800 1675 50  0001 C CNN "DigiKey"
 	1    6800 1675
 	1    0    0    -1
@@
 F 2 "Capacitors_SMD:C_0805_HandSoldering" H 6250 1675 50  0001 C CNN
 F 3 "~" H 6250 1675 50  0001 C CNN
+F 4 "732-7817-1-ND" H 6250 1675 50  0001 C CNN "DigiKey"
 	1    6250 1675
 	1    0    0    1

Commit message: Fix TMS9918 clock circuit
Connections:
- wire segments 132 -> 137
Other:
- note added: "Outputs"
Changed lines of the file:
@@
 L Device:Crystal Y1
 U 1 1 5E875480
-P 6525 1575
-F 0 "Y1" H 6525 1307 50  0000 C CNN
-F 1 "10.738635MHZ" H 6525 1398 50  0000 C CNN
-F 2 "Crystals:Crystal_HC49-U_Vertical" H 6525 1575 50  0001 C CNN
-F 3 "~" H 6525 1575 50  0001 C CNN
-F 4 "CTX1443-ND" H 6525 1575 50  0001 C CNN "DigiKey"
-	1    6525 1575
+P 6600 2025
+F 0 "Y1" H 6600 1757 50  0000 C CNN
+F 1 "10.738635MHZ" H 6600 1848 50  0000 C CNN
+F 2 "Crystals:Crystal_HC49-U_Vertical" H 6600 2025 50  0001 C CNN
+F 3 "~" H 6600 2025 50  0001 C CNN
+F 4 "CTX1443-ND" H 6600 2025 50  0001 C CNN "DigiKey"
+	1    6600 2025
 	-1   0    0    1
 $EndComp
@@
 L Device:C_Small C23
 U 1 1 5E87B8DE
-P 6250 1675
-F 0 "C23" H 6159 1629 50  0000 R CNN
-F 1 "33pF" H 6159 1720 50  0000 R CNN
-F 2 "Capacitors_SMD:C_0805_HandSoldering" H 6250 1675 50  0001 C CNN
-F 3 "~" H 6250 1675 50  0001 C CNN
-F 4 "732-7817-1-ND" H 6250 1675 50  0001 C CNN "DigiKey"
-	1    6250 1675
+P 6400 1700
+F 0 "C23" H 6309 1654 50  0000 R CNN
+F 1 "33pF" H 6309 1745 50  0000 R CNN
+F 2 "Capacitors_SMD:C_0805_HandSoldering" H 6400 1700 50  0001 C CNN
+F 3 "~" H 6400 1700 50  0001 C CNN
+F 4 "732-7817-1-ND" H 6400 1700 50  0001 C CNN "DigiKey"
+	1    6400 1700
 	1    0    0    1
 $EndComp
 Wire Wire Line
-	6400 2100 6400 1850
-Wire Wire Line
-	6400 1850 6250 1850
-Wire Wire Line
-	6250 1850 6250 1775
+	6400 2100 6400 2025
 Wire Wire Line
 	6400 2200 6800 2200
 Wire Wire Line
-	6800 2200 6800 1775
+	6800 2200 6800 2025
 Wire Wire Line
-	6675 1575 6800 1575
+	6750 2025 6800 2025
+Connection ~ 6800 2025
 Wire Wire Line
-	6375 1575 6250 1575
+	6800 2025 6800 1775
+Wire Wire Line
+	6450 2025 6400 2025
+Connection ~ 6400 2025
+Wire Wire Line
+	6400 1800 6400 2025
+Wire Wire Line
+	6400 1575 6400 1600
+Wire Wire Line
+	6400 1575 6675 1575
+$Comp
+L power:GND #PWR?
+U 1 1 5EE485EA
+P 6550 1400
+F 0 "#PWR?" H 6550 1150 50  0001 C CNN
+F 1 "GND" H 6555 1227 50  0000 C CNN
+F 2 "" H 6550 1400 50  0001 C CNN
+F 3 "" H 6550 1400 50  0001 C CNN
+	1    6550 1400
+	1    0    0    -1
+$EndComp
+Wire Wire Line
+	6550 1400 6675 1400
+Wire Wire Line
+	6675 1400 6675 1575
 Wire Bus Line
 	4350 3200 4700 3200
@@
 Wire Bus Line
 	6700 3800 6700 4225
+Connection ~ 6675 1575
+Wire Wire Line
+	6675 1575 6800 1575
+Text Notes 6450 2375 0    50   Italic 10
+Outputs
 $EndSCHEMATC

Commit message: 56pF crystal caps
Parts:
- C23, C26: value 33pF -> 56pF
Changed lines of the file:
@@
 P 6800 1675
 F 0 "C26" H 6892 1721 50  0000 L CNN
-F 1 "33pF" H 6892 1630 50  0000 L CNN
+F 1 "56pF" H 6892 1630 50  0000 L CNN
 F 2 "Capacitors_SMD:C_0805_HandSoldering" H 6800 1675 50  0001 C CNN
 F 3 "~" H 6800 1675 50  0001 C CNN
@@
 P 6400 1700
 F 0 "C23" H 6309 1654 50  0000 R CNN
-F 1 "33pF" H 6309 1745 50  0000 R CNN
+F 1 "56pF" H 6309 1745 50  0000 R CNN
 F 2 "Capacitors_SMD:C_0805_HandSoldering" H 6400 1700 50  0001 C CNN
 F 3 "~" H 6400 1700 50  0001 C CNN
@@
 	6400 1575 6675 1575
 $Comp
-L power:GND #PWR?
+L power:GND #PWR0154
 U 1 1 5EE485EA
 P 6550 1400
-F 0 "#PWR?" H 6550 1150 50  0001 C CNN
+F 0 "#PWR0154" H 6550 1150 50  0001 C CNN
 F 1 "GND" H 6555 1227 50  0000 C CNN
 F 2 "" H 6550 1400 50  0001 C CNN
