File: Video.sch (KiCad schematic (older format))
At the start: 25 parts, among them J2 Composite video, Q1 2n4401, U4 74HCT04, U5 TMS9918A, U6 74LS574, U7 74LS574, U8 74LS574, U9 VRAM, Y1 10.738635MHZ

Commit message: Improve routing for VDC_R, VDC_W
Connections:
- wire segments 137 -> 140
Changed lines of the file:
@@
 Text GLabel 4800 3450 0    50   Input ~ 0
 VDC_R
-Text GLabel 5400 3400 0    50   Input ~ 0
+Text GLabel 5175 3375 0    50   Input ~ 0
 VDC_W
 Text GLabel 5325 3000 0    50   Input ~ 0
@@
 Wire Wire Line
 	6675 1400 6675 1575
+Connection ~ 6675 1575
+Wire Wire Line
+	6675 1575 6800 1575
+Text Notes 6450 2375 0    50   Italic 10
+Outputs
+Wire Wire Line
+	5400 3400 5225 3400
+Wire Wire Line
+	5225 3400 5225 3375
+Wire Wire Line
+	5225 3375 5175 3375
 Wire Bus Line
 	4350 3200 4700 3200
@@
 Wire Bus Line
 	6700 3800 6700 4225
-Connection ~ 6675 1575
-Wire Wire Line
-	6675 1575 6800 1575
-Text Notes 6450 2375 0    50   Italic 10
-Outputs
 $EndSCHEMATC

Commit message: Output transistor fix
Parts:
- removed Q1: 2n4401, TO_SOT_Packages_THT:TO-92_Molded_Narrow, symbol Device:Q_NPN_Darlington_BCE
- added Q1: 2n4401, symbol Device:Q_NPN_EBC
Other:
- note added: "Revised June 2020: \nFixed wrong pinout for\n2n4401"
Changed lines of the file:
@@
-	1    0    0    -1
-$EndComp
-$Comp
-L Device:Q_NPN_Darlington_BCE Q1
-U 1 1 5E41A766
-P 2925 1675
-F 0 "Q1" H 3116 1721 50  0000 L CNN
-F 1 "2n4401" H 3116 1630 50  0000 L CNN
-F 2 "TO_SOT_Packages_THT:TO-92_Molded_Narrow" H 3125 1775 50  0001 C CNN
-F 3 "~" H 2925 1675 50  0001 C CNN
-	1    2925 1675
 	1    0    0    -1
 $EndComp
@@
 Wire Bus Line
 	6700 3800 6700 4225
+Text Notes 4150 1675 2    50   ~ 0
+Revised June 2020: \nFixed wrong pinout for\n2n4401
+$Comp
+L Device:Q_NPN_EBC Q1
+U 1 1 5F007C10
+P 2925 1675
+F 0 "Q1" H 3116 1721 50  0000 L CNN
+F 1 "2n4401" H 3116 1630 50  0000 L CNN
+F 2 "" H 3125 1775 50  0001 C CNN
+F 3 "~" H 2925 1675 50  0001 C CNN
+	1    2925 1675
+	1    0    0    -1
+$EndComp
 $EndSCHEMATC

Commit message: Add 220uF output cap
Parts:
- added C25: 220µF, Capacitors_ThroughHole:CP_Radial_D6.3mm_P2.50mm, symbol Device:CP1_Small
- Q1: footprint (none) -> TO_SOT_Packages_THT:TO-92_Inline_Wide
Changed lines of the file:
@@
 L RCJ-017:RCJ-017 J2
 U 1 1 5E3A6E8A
-P 3725 2075
-F 0 "J2" H 3567 2024 50  0000 R CNN
-F 1 "Composite video" H 3567 2115 50  0000 R CNN
-F 2 "Jacks:CUI_RCJ-017" H 3725 2075 50  0001 L BNN
-F 3 "CUI Inc" H 3725 2075 50  0001 L BNN
-F 4 "B" H 3725 2075 50  0001 L BNN "Field4"
-F 5 "Manufacturer recommendations" H 3725 2075 50  0001 L BNN "Field5"
-	1    3725 2075
+P 3925 2075
+F 0 "J2" H 3767 2024 50  0000 R CNN
+F 1 "Composite video" H 3767 2115 50  0000 R CNN
+F 2 "Jacks:CUI_RCJ-017" H 3925 2075 50  0001 L BNN
+F 3 "CUI Inc" H 3925 2075 50  0001 L BNN
+F 4 "B" H 3925 2075 50  0001 L BNN "Field4"
+F 5 "Manufacturer recommendations" H 3925 2075 50  0001 L BNN "Field5"
+	1    3925 2075
 	-1   0    0    1
 $EndComp
@@
 L power:GND #PWR011
 U 1 1 5E3A60DD
-P 3425 2175
-F 0 "#PWR011" H 3425 1925 50  0001 C CNN
-F 1 "GND" H 3430 2002 50  0000 C CNN
-F 2 "" H 3425 2175 50  0001 C CNN
-F 3 "" H 3425 2175 50  0001 C CNN
-	1    3425 2175
+P 3625 2175
+F 0 "#PWR011" H 3625 1925 50  0001 C CNN
+F 1 "GND" H 3630 2002 50  0000 C CNN
+F 2 "" H 3625 2175 50  0001 C CNN
+F 3 "" H 3625 2175 50  0001 C CNN
+	1    3625 2175
 	1    0    0    -1
 $EndComp
@@
 Wire Wire Line
 	3025 1875 3025 1975
-Wire Wire Line
-	3025 1975 3425 1975
 $Comp
 L Device:R_Small_US R6
@@
 	1    0    0    -1
 $EndComp
-Connection ~ 3025 1975
 $Comp
 L power:GND #PWR010
@@
 Wire Wire Line
 	5225 3375 5175 3375
+Text Notes 4150 1675 2    50   ~ 0
+Revised June 2020: \nFixed wrong pinout for\n2n4401
+$Comp
+L Device:Q_NPN_EBC Q1
+U 1 1 5F007C10
+P 2925 1675
+F 0 "Q1" H 3116 1721 50  0000 L CNN
+F 1 "2n4401" H 3116 1630 50  0000 L CNN
+F 2 "TO_SOT_Packages_THT:TO-92_Inline_Wide" H 3125 1775 50  0001 C CNN
+F 3 "~" H 2925 1675 50  0001 C CNN
+	1    2925 1675
+	1    0    0    -1
+$EndComp
+$Comp
+L Device:CP1_Small C25
+U 1 1 5EEBA833
+P 3525 1975
+F 0 "C25" V 3753 1975 50  0000 C CNN
+F 1 "220µF" V 3662 1975 50  0000 C CNN
+F 2 "Capacitors_ThroughHole:CP_Radial_D6.3mm_P2.50mm" H 3525 1975 50  0001 C CNN
+F 3 "~" H 3525 1975 50  0001 C CNN
+	1    3525 1975
+	0    -1   -1   0
+$EndComp
+Wire Wire Line
+	3425 1975 3025 1975
 Wire Bus Line
 	4350 3200 4700 3200
@@
 Wire Bus Line
 	6700 3800 6700 4225
-Text Notes 4150 1675 2    50   ~ 0
-Revised June 2020: \nFixed wrong pinout for\n2n4401
-$Comp
-L Device:Q_NPN_EBC Q1
-U 1 1 5F007C10
-P 2925 1675
-F 0 "Q1" H 3116 1721 50  0000 L CNN
-F 1 "2n4401" H 3116 1630 50  0000 L CNN
-F 2 "" H 3125 1775 50  0001 C CNN
-F 3 "~" H 2925 1675 50  0001 C CNN
-	1    2925 1675
-	1    0    0    -1
-$EndComp
+Connection ~ 3025 1975
 $EndSCHEMATC

Commit message: Change note to mention cap
Other:
- note added: "Revised June 2020: \nFixed wrong pinout for\n2n4401, add output cap"
- note removed: "Revised June 2020: \nFixed wrong pinout for\n2n4401"
Changed lines of the file:
@@
 Wire Wire Line
 	5225 3375 5175 3375
-Text Notes 4150 1675 2    50   ~ 0
-Revised June 2020: \nFixed wrong pinout for\n2n4401
+Text Notes 4375 1650 2    50   ~ 0
+Revised June 2020: \nFixed wrong pinout for\n2n4401, add output cap
 $Comp
 L Device:Q_NPN_EBC Q1
@@
 Wire Wire Line
 	3425 1975 3025 1975
+Connection ~ 3025 1975
 Wire Bus Line
 	4350 3200 4700 3200
@@
 Wire Bus Line
 	6700 3800 6700 4225
-Connection ~ 3025 1975
 $EndSCHEMATC

Commit message: Update symbols to use ~
Other:
- note added: "LSB"
- note added: "MSB"
Changed lines of the file:
@@
 Wire Bus Line
 	6700 3800 6700 4225
+Text Notes 6625 2925 0    50   ~ 0
+MSB
+Text Notes 6625 3650 0    50   ~ 0
+LSB
+Text Notes 6700 3725 0    50   ~ 0
+MSB
+Text Notes 5025 3675 0    50   ~ 0
+LSB
 $EndSCHEMATC

Commit message: Tie VRAM A14 to ground
Connections:
- wire segments 140 -> 142
Changed lines of the file:
@@
 Text GLabel 10800 3150 2    50   Input ~ 0
-RAM_A13
-Text GLabel 10800 3250 2    50   Input Italic 0
 RAM_A13
 Text Notes 11050 5475 2    50   Italic 0
@@
 	3425 1975 3025 1975
 Connection ~ 3025 1975
-Wire Bus Line
-	4350 3200 4700 3200
-Wire Bus Line
-	5200 3600 5200 4225
-Wire Bus Line
-	6700 3800 6700 4225
 Text Notes 6625 2925 0    50   ~ 0
 MSB
@@
 Text Notes 5025 3675 0    50   ~ 0
 LSB
+$Comp
+L power:GND #PWR?
+U 1 1 5EEEDA3D
+P 11000 4525
+F 0 "#PWR?" H 11000 4275 50  0001 C CNN
+F 1 "GND" H 11005 4352 50  0000 C CNN
+F 2 "" H 11000 4525 50  0001 C CNN
+F 3 "" H 11000 4525 50  0001 C CNN
+	1    11000 4525
+	1    0    0    -1
+$EndComp
+Wire Wire Line
+	11000 4525 11000 3250
+Wire Wire Line
+	11000 3250 10800 3250
+Wire Bus Line
+	4350 3200 4700 3200
+Wire Bus Line
+	5200 3600 5200 4225
+Wire Bus Line
+	6700 3800 6700 4225
 $EndSCHEMATC

Commit message: Fix the callouts for the SRAM logic
Parts:
- U6, U7, U8: value 74LS574 -> 74HCT574
Changed lines of the file:
@@
 P 7975 1600
 F 0 "U6" H 7975 2581 50  0000 C CNN
-F 1 "74LS574" H 7975 2490 50  0000 C CNN
+F 1 "74HCT574" H 7975 2490 50  0000 C CNN
 F 2 "Housings_SOIC:SOIC-20W_7.5x12.8mm_Pitch1.27mm" H 7975 1600 50  0001 C CNN
 F 3 "https://www.digikey.ca/product-detail/en/nexperia-usa-inc/74HCT574D653/1727-2856-1-ND/763412" H 7975 1600 50  0001 C CNN
@@
 P 7975 3475
 F 0 "U7" H 7700 4275 50  0000 C CNN
-F 1 "74LS574" H 7700 4175 50  0000 C CNN
+F 1 "74HCT574" H 7700 4175 50  0000 C CNN
 F 2 "Housings_SOIC:SOIC-20W_7.5x12.8mm_Pitch1.27mm" H 7975 3475 50  0001 C CNN
 F 3 "https://www.digikey.ca/product-detail/en/nexperia-usa-inc/74HCT574D653/1727-2856-1-ND/763412" H 7975 3475 50  0001 C CNN
@@
 P 7975 5400
 F 0 "U8" H 7700 6200 50  0000 C CNN
-F 1 "74LS574" H 7700 6125 50  0000 C CNN
+F 1 "74HCT574" H 7700 6125 50  0000 C CNN
 F 2 "Housings_SOIC:SOIC-20W_7.5x12.8mm_Pitch1.27mm" H 7975 5400 50  0001 C CNN
 F 3 "https://www.digikey.ca/product-detail/en/nexperia-usa-inc/74HCT574D653/1727-2856-1-ND/763412" H 7975 5400 50  0001 C CNN
@@
 LSB
 $Comp
-L power:GND #PWR?
+L power:GND #PWR0128
 U 1 1 5EEEDA3D
 P 11000 4525
-F 0 "#PWR?" H 11000 4275 50  0001 C CNN
+F 0 "#PWR0128" H 11000 4275 50  0001 C CNN
 F 1 "GND" H 11005 4352 50  0000 C CNN
 F 2 "" H 11000 4525 50  0001 C CNN

Commit message: 62256 for VRAM and RAM
Parts:
- removed C10, C11: 0.1µF, Capacitors_SMD:C_0805_HandSoldering, symbol Device:C
- removed R46: 2kΩ, Resistors_SMD:R_0805_HandSoldering, symbol Device:R_Small_US
- removed U9: VRAM, LeakyChips:SOIC-40-JLead, symbol LeakoChips:LC331632M-12
- added C11: 0.1µF, Capacitors_SMD:C_0805_HandSoldering, symbol Device:C_Small
- added U101: AS6C62256-DIP, Housings_DIP:DIP-28_W15.24mm_Socket_LongPads, symbol AS6C62256:AS6C62256-DIP
Connections:
- net labels removed: VRAM_Upper_Byte_PU
- wire segments 142 -> 112
