File: Sound.sch (KiCad schematic (older format))
At the start: 4 parts

Commit message: BIOS ROM
Parts:
- gave numbers to parts that had none: 4
Changed lines of the file:
@@
 $EndDescr
 $Comp
-L LeakoChips:SN76489AN U?
+L LeakoChips:SN76489AN U10
 U 1 1 5E3C8002
 P 4750 4025
-F 0 "U?" H 4750 4600 50  0000 C CNN
+F 0 "U10" H 4750 4600 50  0000 C CNN
 F 1 "SN76489AN" H 4750 4509 50  0000 C CNN
 F 2 "Housings_DIP:DIP-16_W7.62mm_Socket_LongPads" H 4750 4575 50  0001 C CNN
@@
 $EndComp
 $Comp
-L power:VCC #PWR?
+L power:VCC #PWR031
 U 1 1 5E3C8979
 P 4725 2350
-F 0 "#PWR?" H 4725 2200 50  0001 C CNN
+F 0 "#PWR031" H 4725 2200 50  0001 C CNN
 F 1 "VCC" H 4742 2523 50  0000 C CNN
 F 2 "" H 4725 2350 50  0001 C CNN
@@
 $EndComp
 $Comp
-L power:GND #PWR?
+L power:GND #PWR032
 U 1 1 5E3C8D13
 P 4775 6375
-F 0 "#PWR?" H 4775 6125 50  0001 C CNN
+F 0 "#PWR032" H 4775 6125 50  0001 C CNN
 F 1 "GND" H 4780 6202 50  0000 C CNN
 F 2 "" H 4775 6375 50  0001 C CNN
@@
 	4300 5175 4300 6375
 $Comp
-L Device:C C?
+L Device:C C13
 U 1 1 5E3C98A8
 P 3550 4975
-F 0 "C?" H 3665 5021 50  0000 L CNN
+F 0 "C13" H 3665 5021 50  0000 L CNN
 F 1 "0.1µF" H 3665 4930 50  0000 L CNN
 F 2 "Capacitors_SMD:C_0805_HandSoldering" H 3588 4825 50  0001 C CNN
@@
 D7
 $Comp
-L Device:R_Small_US R?
+L Device:R_Small_US R8
 U 1 1 5E3CBFF6
 P 3900 2825
-F 0 "R?" H 3968 2871 50  0000 L CNN
+F 0 "R8" H 3968 2871 50  0000 L CNN
 F 1 "2kΩ" H 3968 2780 50  0000 L CNN
 F 2 "Resistors_SMD:R_0805_HandSoldering" H 3900 2825 50  0001 C CNN
@@
 Raw_Audio
 $Comp
-L RCJ-017:RCJ-017 J?
+L RCJ-017:RCJ-017 J4
 U 1 1 5E3DB8E6
 P 7825 4975
-F 0 "J?" H 7667 4924 50  0000 R CNN
+F 0 "J4" H 7667 4924 50  0000 R CNN
 F 1 "RCJ-017" H 7667 5015 50  0000 R CNN
 F 2 "CUI_RCJ-017" H 7825 4975 50  0001 L BNN
@@
 $EndComp
 $Comp
-L power:GND #PWR?
+L power:GND #PWR033
 U 1 1 5E3DD314
 P 7525 5075
-F 0 "#PWR?" H 7525 4825 50  0001 C CNN
+F 0 "#PWR033" H 7525 4825 50  0001 C CNN
 F 1 "GND" H 7530 4902 50  0000 C CNN
 F 2 "" H 7525 5075 50  0001 C CNN

Commit message: Memory Decode
Connections:
- net labels added: !WAIT
- net labels removed: Wait
Changed lines of the file:
@@
 Connection ~ 3900 3975
 Text GLabel 3200 3975 0    50   Input ~ 0
-Wait
+!WAIT
 Text Notes 2425 4575 0    50   ~ 0
 "Ready" (active high)\nmeans that the data\nhas been read off the\nline. When low, the CPU\nshould enter a wait state\nuntil the sound chip is free.

Commit message: LM386 audio amp
Parts:
- added C19: 0.05µF, Capacitors_SMD:C_0805_HandSoldering, symbol Device:C
- added R11: 10Ω, Resistors_SMD:R_0805_HandSoldering, symbol Device:R_Small_US
- added RV1: 10kΩ, Potentiometers:Potentiometer_Trimmer_ACP_CA6v_Horizontal_MountLS, symbol Device:R_POT_TRIM_US
- added U15: LM386, Housings_SOIC:SOIC-8_3.9x4.9mm_Pitch1.27mm, symbol Amplifier_Audio:LM386
Connections:
- wire segments 23 -> 40
- no-connect marks 0 -> 3
Other:
- note removed: "TODO: Amplifier"
Changed lines of the file:
@@
 L RCJ-017:RCJ-017 J4
 U 1 1 5E3DB8E6
-P 7825 4975
-F 0 "J4" H 7667 4924 50  0000 R CNN
-F 1 "RCJ-017" H 7667 5015 50  0000 R CNN
-F 2 "CUI_RCJ-017" H 7825 4975 50  0001 L BNN
-F 3 "CUI Inc" H 7825 4975 50  0001 L BNN
-F 4 "B" H 7825 4975 50  0001 L BNN "Field4"
-F 5 "Manufacturer recommendations" H 7825 4975 50  0001 L BNN "Field5"
-	1    7825 4975
+P 7925 6025
+F 0 "J4" H 7767 5974 50  0000 R CNN
+F 1 "RCJ-017" H 7767 6065 50  0000 R CNN
+F 2 "CUI_RCJ-017" H 7925 6025 50  0001 L BNN
+F 3 "CUI Inc" H 7925 6025 50  0001 L BNN
+F 4 "B" H 7925 6025 50  0001 L BNN "Field4"
+F 5 "Manufacturer recommendations" H 7925 6025 50  0001 L BNN "Field5"
+	1    7925 6025
 	-1   0    0    -1
 $EndComp
@@
 L power:GND #PWR033
 U 1 1 5E3DD314
-P 7525 5075
-F 0 "#PWR033" H 7525 4825 50  0001 C CNN
-F 1 "GND" H 7530 4902 50  0000 C CNN
-F 2 "" H 7525 5075 50  0001 C CNN
-F 3 "" H 7525 5075 50  0001 C CNN
-	1    7525 5075
+P 7625 6125
+F 0 "#PWR033" H 7625 5875 50  0001 C CNN
+F 1 "GND" H 7630 5952 50  0000 C CNN
+F 2 "" H 7625 6125 50  0001 C CNN
+F 3 "" H 7625 6125 50  0001 C CNN
+	1    7625 6125
 	1    0    0    -1
 $EndComp
-Text Notes 6300 5000 0    50   ~ 0
-TODO: Amplifier
+$Comp
+L Amplifier_Audio:LM386 U15
+U 1 1 5E3EEA24
+P 6700 5450
+F 0 "U15" V 7089 5450 50  0000 C CNN
+F 1 "LM386" V 7180 5450 50  0000 C CNN
+F 2 "Housings_SOIC:SOIC-8_3.9x4.9mm_Pitch1.27mm" H 6800 5550 50  0001 C CNN
+F 3 "http://www.ti.com/lit/ds/symlink/lm386.pdf" H 6900 5650 50  0001 C CNN
+	1    6700 5450
+	0    1    1    0
+$EndComp
+Wire Wire Line
+	6700 5750 7275 5750
+Wire Wire Line
+	7625 5750 7625 5925
+Wire Wire Line
+	7000 5350 7625 5350
+Wire Wire Line
+	7625 5350 7625 5125
+$Comp
+L power:VCC #PWR0113
+U 1 1 5E3F2514
+P 7625 5125
+F 0 "#PWR0113" H 7625 4975 50  0001 C CNN
+F 1 "VCC" H 7642 5298 50  0000 C CNN
+F 2 "" H 7625 5125 50  0001 C CNN
+F 3 "" H 7625 5125 50  0001 C CNN
+	1    7625 5125
+	1    0    0    -1
+$EndComp
+$Comp
+L power:GND #PWR0114
+U 1 1 5E3F2F4F
+P 6950 4575
+F 0 "#PWR0114" H 6950 4325 50  0001 C CNN
+F 1 "GND" H 6955 4402 50  0000 C CNN
+F 2 "" H 6950 4575 50  0001 C CNN
+F 3 "" H 6950 4575 50  0001 C CNN
+	1    6950 4575
+	1    0    0    -1
+$EndComp
+Wire Wire Line
+	6950 4575 6950 4375
+Wire Wire Line
+	6950 4375 6600 4375
+Wire Wire Line
+	6600 4375 6600 4950
+$Comp
+L Device:R_POT_TRIM_US RV1
+U 1 1 5E3F4BDD
+P 7425 4550
+F 0 "RV1" H 7357 4504 50  0000 R CNN
+F 1 "10kΩ" H 7357 4595 50  0000 R CNN
+F 2 "Potentiometers:Potentiometer_Trimmer_ACP_CA6v_Horizontal_MountLS" H 7425 4550 50  0001 C CNN
+F 3 "~" H 7425 4550 50  0001 C CNN
+	1    7425 4550
+	-1   0    0    1
+$EndComp
+$Comp
+L power:GND #PWR0115
+U 1 1 5E3F5157
+P 7425 4700
+F 0 "#PWR0115" H 7425 4450 50  0001 C CNN
+F 1 "GND" H 7430 4527 50  0000 C CNN
+F 2 "" H 7425 4700 50  0001 C CNN
+F 3 "" H 7425 4700 50  0001 C CNN
+	1    7425 4700
+	1    0    0    -1
+$EndComp
+Wire Wire Line
+	7275 4550 7200 4550
+Wire Wire Line
+	7200 4550 7200 5150
+Wire Wire Line
+	7200 5150 6800 5150
+$Comp
+L power:GND #PWR0116
+U 1 1 5E3F78BD
+P 7275 6250
+F 0 "#PWR0116" H 7275 6000 50  0001 C CNN
+F 1 "GND" H 7280 6077 50  0000 C CNN
+F 2 "" H 7275 6250 50  0001 C CNN
+F 3 "" H 7275 6250 50  0001 C CNN
+	1    7275 6250
+	1    0    0    -1
+$EndComp
+$Comp
+L Device:R_Small_US R11
+U 1 1 5E3F7EBB
+P 7275 6150
+F 0 "R11" H 7343 6196 50  0000 L CNN
+F 1 "10Ω" H 7343 6105 50  0000 L CNN
+F 2 "Resistors_SMD:R_0805_HandSoldering" H 7275 6150 50  0001 C CNN
+F 3 "~" H 7275 6150 50  0001 C CNN
+	1    7275 6150
+	1    0    0    -1
+$EndComp
+Connection ~ 7275 5750
+Wire Wire Line
+	7275 5750 7625 5750
+$Comp
+L Device:C C19
+U 1 1 5E3F96AC
+P 7275 5900
+F 0 "C19" H 7390 5946 50  0000 L CNN
+F 1 "0.05µF" H 7390 5855 50  0000 L CNN
+F 2 "Capacitors_SMD:C_0805_HandSoldering" H 7313 5750 50  0001 C CNN
+F 3 "~" H 7275 5900 50  0001 C CNN
+	1    7275 5900
+	1    0    0    -1
+$EndComp
+NoConn ~ 7000 5450
+NoConn ~ 6400 5450
+NoConn ~ 6400 5550
+Wire Wire Line
+	6400 5350 6400 4950
+Wire Wire Line
+	6400 4950 6600 4950
+Connection ~ 6600 4950
+Wire Wire Line
+	6600 4950 6600 5150
+Wire Wire Line
+	5875 4875 5875 4200
+Wire Wire Line
+	5875 4200 7425 4200
+Wire Wire Line
+	7425 4200 7425 4400
 $EndSCHEMATC

Commit message: MAXIMUM GAIN
Parts:
- added C?: 220µF, Capacitors_ThroughHole:CP_Radial_D8.0mm_P3.50mm, symbol Device:CP
- added C?: 10µF, Capacitors_ThroughHole:CP_Radial_D6.3mm_P2.50mm, symbol Device:CP
- added C?: 10µF, Capacitors_SMD:C_0805_HandSoldering, symbol Device:C
Connections:
- net labels added: Bypass
- wire segments 40 -> 47
- no-connect marks 3 -> 0
Changed lines of the file:
@@
 L RCJ-017:RCJ-017 J4
 U 1 1 5E3DB8E6
-P 7925 6025
-F 0 "J4" H 7767 5974 50  0000 R CNN
-F 1 "RCJ-017" H 7767 6065 50  0000 R CNN
-F 2 "CUI_RCJ-017" H 7925 6025 50  0001 L BNN
-F 3 "CUI Inc" H 7925 6025 50  0001 L BNN
-F 4 "B" H 7925 6025 50  0001 L BNN "Field4"
-F 5 "Manufacturer recommendations" H 7925 6025 50  0001 L BNN "Field5"
-	1    7925 6025
+P 8600 5850
+F 0 "J4" H 8442 5799 50  0000 R CNN
+F 1 "RCJ-017" H 8442 5890 50  0000 R CNN
+F 2 "CUI_RCJ-017" H 8600 5850 50  0001 L BNN
+F 3 "CUI Inc" H 8600 5850 50  0001 L BNN
+F 4 "B" H 8600 5850 50  0001 L BNN "Field4"
+F 5 "Manufacturer recommendations" H 8600 5850 50  0001 L BNN "Field5"
+	1    8600 5850
 	-1   0    0    -1
 $EndComp
@@
 L power:GND #PWR033
 U 1 1 5E3DD314
-P 7625 6125
-F 0 "#PWR033" H 7625 5875 50  0001 C CNN
-F 1 "GND" H 7630 5952 50  0000 C CNN
-F 2 "" H 7625 6125 50  0001 C CNN
-F 3 "" H 7625 6125 50  0001 C CNN
-	1    7625 6125
+P 8300 5950
+F 0 "#PWR033" H 8300 5700 50  0001 C CNN
+F 1 "GND" H 8305 5777 50  0000 C CNN
+F 2 "" H 8300 5950 50  0001 C CNN
+F 3 "" H 8300 5950 50  0001 C CNN
+	1    8300 5950
 	1    0    0    -1
 $EndComp
@@
 	6700 5750 7275 5750
 Wire Wire Line
-	7625 5750 7625 5925
-Wire Wire Line
 	7000 5350 7625 5350
 Wire Wire Line
@@
 $EndComp
 Connection ~ 7275 5750
-Wire Wire Line
-	7275 5750 7625 5750
 $Comp
 L Device:C C19
@@
 	1    0    0    -1
 $EndComp
-NoConn ~ 7000 5450
-NoConn ~ 6400 5450
-NoConn ~ 6400 5550
 Wire Wire Line
 	6400 5350 6400 4950
@@
 Wire Wire Line
 	7425 4200 7425 4400
+$Comp
+L Device:CP C?
+U 1 1 5E3F1698
+P 8150 5750
+F 0 "C?" V 8405 5750 50  0000 C CNN
+F 1 "220µF" V 8314 5750 50  0000 C CNN
+F 2 "Capacitors_ThroughHole:CP_Radial_D8.0mm_P3.50mm" H 8188 5600 50  0001 C CNN
+F 3 "~" H 8150 5750 50  0001 C CNN
+	1    8150 5750
+	0    -1   -1   0
+$EndComp
+Wire Wire Line
+	7275 5750 8000 5750
+$Comp
+L Device:CP C?
+U 1 1 5E3F358B
+P 6000 5500
+F 0 "C?" H 6118 5546 50  0000 L CNN
+F 1 "10µF" H 6118 5455 50  0000 L CNN
+F 2 "Capacitors_ThroughHole:CP_Radial_D6.3mm_P2.50mm" H 6038 5350 50  0001 C CNN
+F 3 "~" H 6000 5500 50  0001 C CNN
+	1    6000 5500
+	1    0    0    -1
+$EndComp
+Wire Wire Line
+	6400 5550 6400 5650
+Wire Wire Line
+	6400 5650 6000 5650
+Wire Wire Line
+	6400 5450 6325 5450
+Wire Wire Line
+	6325 5450 6325 5350
+Wire Wire Line
+	6325 5350 6000 5350
+Wire Wire Line
+	7000 5450 7000 6125
+Wire Wire Line
+	7000 6125 6375 6125
+Wire Wire Line
+	6375 6125 6375 6250
+$Comp
+L Device:C C?
+U 1 1 5E3F7B65
+P 6375 6400
+F 0 "C?" H 6490 6446 50  0000 L CNN
+F 1 "10µF" H 6490 6355 50  0000 L CNN
+F 2 "Capacitors_SMD:C_0805_HandSoldering" H 6413 6250 50  0001 C CNN
+F 3 "~" H 6375 6400 50  0001 C CNN
+	1    6375 6400
+	1    0    0    -1
+$EndComp
+$Comp
+L power:GND #PWR?
+U 1 1 5E3F80AD
+P 6375 6550
+F 0 "#PWR?" H 6375 6300 50  0001 C CNN
+F 1 "GND" H 6380 6377 50  0000 C CNN
+F 2 "" H 6375 6550 50  0001 C CNN
+F 3 "" H 6375 6550 50  0001 C CNN
+	1    6375 6550
+	1    0    0    -1
+$EndComp
+Text Label 6375 6125 0    50   ~ 0
+Bypass
 $EndSCHEMATC

Commit message: Get rid of amp
Parts:
- removed C19: 0.05µF, Capacitors_SMD:C_0805_HandSoldering, symbol Device:C
- removed C?: 220µF, Capacitors_ThroughHole:CP_Radial_D8.0mm_P3.50mm, symbol Device:CP
- removed C?: 10µF, Capacitors_ThroughHole:CP_Radial_D6.3mm_P2.50mm, symbol Device:CP
- removed C?: 10µF, Capacitors_SMD:C_0805_HandSoldering, symbol Device:C
- removed R11: 10Ω, Resistors_SMD:R_0805_HandSoldering, symbol Device:R_Small_US
- removed RV1: 10kΩ, Potentiometers:Potentiometer_Trimmer_ACP_CA6v_Horizontal_MountLS, symbol Device:R_POT_TRIM_US
- removed U15: LM386, Housings_SOIC:SOIC-8_3.9x4.9mm_Pitch1.27mm, symbol Amplifier_Audio:LM386
- added C?: 0.1µF, Capacitors_SMD:C_0805_HandSoldering, symbol Device:C
- added R?: 1kΩ, Resistors_SMD:R_0805_HandSoldering, symbol Device:R_Small_US
Connections:
- net labels removed: Bypass
- wire segments 47 -> 25
Changed lines of the file:
@@
 Wire Wire Line
 	4250 4125 4250 4075
-Wire Wire Line
-	4050 4875 5875 4875
 Text Label 4600 4875 0    50   ~ 0
 Raw_Audio
@@
 L RCJ-017:RCJ-017 J4
 U 1 1 5E3DB8E6
-P 8600 5850
-F 0 "J4" H 8442 5799 50  0000 R CNN
-F 1 "RCJ-017" H 8442 5890 50  0000 R CNN
-F 2 "CUI_RCJ-017" H 8600 5850 50  0001 L BNN
-F 3 "CUI Inc" H 8600 5850 50  0001 L BNN
-F 4 "B" H 8600 5850 50  0001 L BNN "Field4"
-F 5 "Manufacturer recommendations" H 8600 5850 50  0001 L BNN "Field5"
-	1    8600 5850
+P 6675 4975
+F 0 "J4" H 6517 4924 50  0000 R CNN
+F 1 "RCJ-017" H 6517 5015 50  0000 R CNN
+F 2 "CUI_RCJ-017" H 6675 4975 50  0001 L BNN
+F 3 "CUI Inc" H 6675 4975 50  0001 L BNN
+F 4 "B" H 6675 4975 50  0001 L BNN "Field4"
+F 5 "Manufacturer recommendations" H 6675 4975 50  0001 L BNN "Field5"
+	1    6675 4975
 	-1   0    0    -1
 $EndComp
@@
 L power:GND #PWR033
 U 1 1 5E3DD314
-P 8300 5950
-F 0 "#PWR033" H 8300 5700 50  0001 C CNN
-F 1 "GND" H 8305 5777 50  0000 C CNN
-F 2 "" H 8300 5950 50  0001 C CNN
-F 3 "" H 8300 5950 50  0001 C CNN
-	1    8300 5950
+P 8125 5875
+F 0 "#PWR033" H 8125 5625 50  0001 C CNN
+F 1 "GND" H 8130 5702 50  0000 C CNN
+F 2 "" H 8125 5875 50  0001 C CNN
+F 3 "" H 8125 5875 50  0001 C CNN
+	1    8125 5875
+	1    0    0    -1
+$EndComp
+Wire Wire Line
+	4050 4875 5375 4875
+$Comp
+L power:GND #PWR?
+U 1 1 5E40270A
+P 6375 5075
+F 0 "#PWR?" H 6375 4825 50  0001 C CNN
+F 1 "GND" H 6380 4902 50  0000 C CNN
+F 2 "" H 6375 5075 50  0001 C CNN
+F 3 "" H 6375 5075 50  0001 C CNN
+	1    6375 5075
 	1    0    0    -1
 $EndComp
 $Comp
-L Amplifier_Audio:LM386 U15
-U 1 1 5E3EEA24
-P 6700 5450
-F 0 "U15" V 7089 5450 50  0000 C CNN
-F 1 "LM386" V 7180 5450 50  0000 C CNN
-F 2 "Housings_SOIC:SOIC-8_3.9x4.9mm_Pitch1.27mm" H 6800 5550 50  0001 C CNN
-F 3 "http://www.ti.com/lit/ds/symlink/lm386.pdf" H 6900 5650 50  0001 C CNN
-	1    6700 5450
+L Device:R_Small_US R?
+U 1 1 5E402B88
+P 5475 4875
+F 0 "R?" V 5270 4875 50  0000 C CNN
+F 1 "1kΩ" V 5361 4875 50  0000 C CNN
+F 2 "Resistors_SMD:R_0805_HandSoldering" H 5475 4875 50  0001 C CNN
+F 3 "~" H 5475 4875 50  0001 C CNN
+	1    5475 4875
 	0    1    1    0
 $EndComp
 Wire Wire Line
-	6700 5750 7275 5750
-Wire Wire Line
-	7000 5350 7625 5350
-Wire Wire Line
-	7625 5350 7625 5125
+	5575 4875 5875 4875
 $Comp
-L power:VCC #PWR0113
-U 1 1 5E3F2514
-P 7625 5125
-F 0 "#PWR0113" H 7625 4975 50  0001 C CNN
-F 1 "VCC" H 7642 5298 50  0000 C CNN
-F 2 "" H 7625 5125 50  0001 C CNN
-F 3 "" H 7625 5125 50  0001 C CNN
-	1    7625 5125
-	1    0    0    -1
-$EndComp
-$Comp
-L power:GND #PWR0114
-U 1 1 5E3F2F4F
-P 6950 4575
-F 0 "#PWR0114" H 6950 4325 50  0001 C CNN
-F 1 "GND" H 6955 4402 50  0000 C CNN
-F 2 "" H 6950 4575 50  0001 C CNN
-F 3 "" H 6950 4575 50  0001 C CNN
-	1    6950 4575
-	1    0    0    -1
+L Device:C C?
+U 1 1 5E402ED1
+P 6025 4875
+F 0 "C?" V 5773 4875 50  0000 C CNN
+F 1 "0.1µF" V 5864 4875 50  0000 C CNN
+F 2 "Capacitors_SMD:C_0805_HandSoldering" H 6063 4725 50  0001 C CNN
+F 3 "~" H 6025 4875 50  0001 C CNN
+	1    6025 4875
+	0    1    1    0
 $EndComp
 Wire Wire Line
-	6950 4575 6950 4375
-Wire Wire Line
-	6950 4375 6600 4375
-Wire Wire Line
-	6600 4375 6600 4950
-$Comp
-L Device:R_POT_TRIM_US RV1
-U 1 1 5E3F4BDD
-P 7425 4550
-F 0 "RV1" H 7357 4504 50  0000 R CNN
-F 1 "10kΩ" H 7357 4595 50  0000 R CNN
-F 2 "Potentiometers:Potentiometer_Trimmer_ACP_CA6v_Horizontal_MountLS" H 7425 4550 50  0001 C CNN
-F 3 "~" H 7425 4550 50  0001 C CNN
-	1    7425 4550
-	-1   0    0    1
-$EndComp
-$Comp
-L power:GND #PWR0115
-U 1 1 5E3F5157
-P 7425 4700
-F 0 "#PWR0115" H 7425 4450 50  0001 C CNN
-F 1 "GND" H 7430 4527 50  0000 C CNN
-F 2 "" H 7425 4700 50  0001 C CNN
-F 3 "" H 7425 4700 50  0001 C CNN
-	1    7425 4700
-	1    0    0    -1
-$EndComp
-Wire Wire Line
-	7275 4550 7200 4550
-Wire Wire Line
-	7200 4550 7200 5150
-Wire Wire Line
-	7200 5150 6800 5150
-$Comp
-L power:GND #PWR0116
-U 1 1 5E3F78BD
-P 7275 6250
-F 0 "#PWR0116" H 7275 6000 50  0001 C CNN
-F 1 "GND" H 7280 6077 50  0000 C CNN
-F 2 "" H 7275 6250 50  0001 C CNN
-F 3 "" H 7275 6250 50  0001 C CNN
-	1    7275 6250
-	1    0    0    -1
-$EndComp
-$Comp
-L Device:R_Small_US R11
-U 1 1 5E3F7EBB
-P 7275 6150
-F 0 "R11" H 7343 6196 50  0000 L CNN
-F 1 "10Ω" H 7343 6105 50  0000 L CNN
-F 2 "Resistors_SMD:R_0805_HandSoldering" H 7275 6150 50  0001 C CNN
-F 3 "~" H 7275 6150 50  0001 C CNN
-	1    7275 6150
-	1    0    0    -1
-$EndComp
-Connection ~ 7275 5750
-$Comp
-L Device:C C19
-U 1 1 5E3F96AC
-P 7275 5900
-F 0 "C19" H 7390 5946 50  0000 L CNN
-F 1 "0.05µF" H 7390 5855 50  0000 L CNN
-F 2 "Capacitors_SMD:C_0805_HandSoldering" H 7313 5750 50  0001 C CNN
-F 3 "~" H 7275 5900 50  0001 C CNN
-	1    7275 5900
-	1    0    0    -1
-$EndComp
-Wire Wire Line
-	6400 5350 6400 4950
-Wire Wire Line
-	6400 4950 6600 4950
-Connection ~ 6600 4950
-Wire Wire Line
-	6600 4950 6600 5150
-Wire Wire Line
-	5875 4875 5875 4200
-Wire Wire Line
-	5875 4200 7425 4200
-Wire Wire Line
-	7425 4200 7425 4400
-$Comp
-L Device:CP C?
-U 1 1 5E3F1698
-P 8150 5750
-F 0 "C?" V 8405 5750 50  0000 C CNN
-F 1 "220µF" V 8314 5750 50  0000 C CNN
-F 2 "Capacitors_ThroughHole:CP_Radial_D8.0mm_P3.50mm" H 8188 5600 50  0001 C CNN
-F 3 "~" H 8150 5750 50  0001 C CNN
-	1    8150 5750
-	0    -1   -1   0
-$EndComp
-Wire Wire Line
-	7275 5750 8000 5750
-$Comp
-L Device:CP C?
-U 1 1 5E3F358B
-P 6000 5500
-F 0 "C?" H 6118 5546 50  0000 L CNN
-F 1 "10µF" H 6118 5455 50  0000 L CNN
-F 2 "Capacitors_ThroughHole:CP_Radial_D6.3mm_P2.50mm" H 6038 5350 50  0001 C CNN
-F 3 "~" H 6000 5500 50  0001 C CNN
-	1    6000 5500
-	1    0    0    -1
-$EndComp
-Wire Wire Line
-	6400 5550 6400 5650
-Wire Wire Line
-	6400 5650 6000 5650
-Wire Wire Line
-	6400 5450 6325 5450
-Wire Wire Line
-	6325 5450 6325 5350
-Wire Wire Line
-	6325 5350 6000 5350
-Wire Wire Line
-	7000 5450 7000 6125
-Wire Wire Line
-	7000 6125 6375 6125
-Wire Wire Line
-	6375 6125 6375 6250
-$Comp
-L Device:C C?
-U 1 1 5E3F7B65
-P 6375 6400
-F 0 "C?" H 6490 6446 50  0000 L CNN
-F 1 "10µF" H 6490 6355 50  0000 L CNN
-F 2 "Capacitors_SMD:C_0805_HandSoldering" H 6413 6250 50  0001 C CNN
-F 3 "~" H 6375 6400 50  0001 C CNN
-	1    6375 6400
-	1    0    0    -1
-$EndComp
-$Comp
-L power:GND #PWR?
-U 1 1 5E3F80AD
-P 6375 6550
-F 0 "#PWR?" H 6375 6300 50  0001 C CNN
-F 1 "GND" H 6380 6377 50  0000 C CNN
-F 2 "" H 6375 6550 50  0001 C CNN
-F 3 "" H 6375 6550 50  0001 C CNN
-	1    6375 6550
-	1    0    0    -1
-$EndComp
-Text Label 6375 6125 0    50   ~ 0
-Bypass
+	6375 4875 6175 4875
 $EndSCHEMATC

Commit message: Better power switch found
Parts:
- gave numbers to parts that had none: 2
Changed lines of the file:
@@
 	4050 4875 5375 4875
 $Comp
-L power:GND #PWR?
+L power:GND #PWR0113
 U 1 1 5E40270A
 P 6375 5075
-F 0 "#PWR?" H 6375 4825 50  0001 C CNN
+F 0 "#PWR0113" H 6375 4825 50  0001 C CNN
 F 1 "GND" H 6380 4902 50  0000 C CNN
 F 2 "" H 6375 5075 50  0001 C CNN
@@
 $EndComp
 $Comp
-L Device:R_Small_US R?
+L Device:R_Small_US R11
 U 1 1 5E402B88
 P 5475 4875
-F 0 "R?" V 5270 4875 50  0000 C CNN
+F 0 "R11" V 5270 4875 50  0000 C CNN
 F 1 "1kΩ" V 5361 4875 50  0000 C CNN
 F 2 "Resistors_SMD:R_0805_HandSoldering" H 5475 4875 50  0001 C CNN
@@
 	5575 4875 5875 4875
 $Comp
-L Device:C C?
+L Device:C C19
 U 1 1 5E402ED1
 P 6025 4875
-F 0 "C?" V 5773 4875 50  0000 C CNN
+F 0 "C19" V 5773 4875 50  0000 C CNN
 F 1 "0.1µF" V 5864 4875 50  0000 C CNN
 F 2 "Capacitors_SMD:C_0805_HandSoldering" H 6063 4725 50  0001 C CNN
