File: Sound.sch (KiCad schematic (older format))
At the start: 6 parts, among them J4 RCJ-017, U10 SN76489AN

Commit message: Controller ports
Connections:
- net labels added: To_Speakers
Changed lines of the file:
@@
 Wire Wire Line
 	6375 4875 6175 4875
+Text Label 6325 4875 1    50   ~ 0
+To_Speakers
 $EndSCHEMATC

Commit message: Add test point bodges
Parts:
- J4: footprint CUI_RCJ-017 -> Jacks:CUI_RCJ-017
Changed lines of the file:
@@
 $Descr A4 11693 8268
 encoding utf-8
-Sheet 4 6
+Sheet 4 7
 Title ""
 Date ""
@@
 F 0 "J4" H 6517 4924 50  0000 R CNN
 F 1 "RCJ-017" H 6517 5015 50  0000 R CNN
-F 2 "CUI_RCJ-017" H 6675 4975 50  0001 L BNN
+F 2 "Jacks:CUI_RCJ-017" H 6675 4975 50  0001 L BNN
 F 3 "CUI Inc" H 6675 4975 50  0001 L BNN
 F 4 "B" H 6675 4975 50  0001 L BNN "Field4"

Commit message: Clock crystal bullshit
Connections:
- net labels added: AUD_CLK
- net labels removed: Audio_CLK
Changed lines of the file:
@@
 	5200 3875 5500 3875
 Text GLabel 5500 3875 2    50   Input ~ 0
-Audio_CLK
+AUD_CLK
 Text GLabel 4200 4125 0    50   Input ~ 0
 Audio_WR

Commit message: reverse data bus for 76489
Changed lines of the file:
@@
 Wire Wire Line
 	3550 2725 3550 4825
-Text GLabel 4300 3675 0    50   Input ~ 0
-D2
-Text GLabel 4300 3775 0    50   Input ~ 0
-D1
-Text GLabel 4300 3875 0    50   Input ~ 0
-D0
-Text GLabel 5200 3775 2    50   Input ~ 0
-D3
-Text GLabel 5200 3975 2    50   Input ~ 0
-D4
-Text GLabel 5200 4075 2    50   Input ~ 0
-D5
-Text GLabel 5200 4175 2    50   Input ~ 0
-D6
-Text GLabel 5200 4275 2    50   Input ~ 0
-D7
 $Comp
 L Device:R_Small_US R8
@@
 Text Label 6325 4875 1    50   ~ 0
 To_Speakers
+Text GLabel 4300 3875 0    50   Input ~ 0
+D7
+Text GLabel 4300 3775 0    50   Input ~ 0
+D6
+Text GLabel 4300 3675 0    50   Input ~ 0
+D5
+Text GLabel 5200 3775 2    50   Input ~ 0
+D4
+Text GLabel 5200 3975 2    50   Input ~ 0
+D3
+Text GLabel 5200 4075 2    50   Input ~ 0
+D2
+Text GLabel 5200 4175 2    50   Input ~ 0
+D1
+Text GLabel 5200 4275 2    50   Input ~ 0
+D0
 $EndSCHEMATC

Commit message: Fix clock circuit - v0.2
Changed lines of the file:
@@
 	-1   0    0    1
-$EndComp
-$Comp
-L power:GND #PWR033
-U 1 1 5E3DD314
-P 8125 5875
-F 0 "#PWR033" H 8125 5625 50  0001 C CNN
-F 1 "GND" H 8130 5702 50  0000 C CNN
-F 2 "" H 8125 5875 50  0001 C CNN
-F 3 "" H 8125 5875 50  0001 C CNN
-	1    8125 5875
-	1    0    0    -1
 $EndComp
 Wire Wire Line

Commit message: ECOs added
Other:
- note added: "TODO: REMOVE"
Changed lines of the file:
@@
 	5200 2350 4725 2350
-Wire Wire Line
-	5200 2725 3900 2725
 Wire Wire Line
 	3550 5175 4300 5175
@@
 Wire Wire Line
 	3550 2725 3550 4825
-$Comp
-L Device:R_Small_US R8
-U 1 1 5E3CBFF6
-P 3900 2825
-F 0 "R8" H 3968 2871 50  0000 L CNN
-F 1 "2kΩ" H 3968 2780 50  0000 L CNN
-F 2 "Resistors_SMD:R_0805_HandSoldering" H 3900 2825 50  0001 C CNN
-F 3 "~" H 3900 2825 50  0001 C CNN
-	1    3900 2825
-	1    0    0    -1
-$EndComp
-Connection ~ 3900 2725
-Wire Wire Line
-	3900 2725 3550 2725
-Wire Wire Line
-	4300 3975 3900 3975
-Wire Wire Line
-	3900 3975 3900 2925
-Wire Wire Line
-	3900 3975 3200 3975
-Connection ~ 3900 3975
 Text GLabel 3200 3975 0    50   Input ~ 0
 !WAIT
@@
 Text GLabel 5200 4275 2    50   Input ~ 0
 D0
+Connection ~ 3900 3975
+Wire Wire Line
+	3900 3975 3200 3975
+Wire Wire Line
+	4300 3975 3900 3975
+Connection ~ 3900 2725
+Wire Wire Line
+	3900 2725 3550 2725
+Wire Wire Line
+	5200 2725 3900 2725
+Wire Wire Line
+	3900 3975 3900 2925
+$Comp
+L Device:R_Small_US R8
+U 1 1 5E3CBFF6
+P 3900 2825
+F 0 "R8" H 3968 2871 50  0000 L CNN
+F 1 "2kΩ" H 3968 2780 50  0000 L CNN
+F 2 "Resistors_SMD:R_0805_HandSoldering" H 3900 2825 50  0001 C CNN
+F 3 "~" H 3900 2825 50  0001 C CNN
+	1    3900 2825
+	1    0    0    -1
+$EndComp
+Text Notes 3975 3050 0    50   ~ 10
+TODO: REMOVE
 $EndSCHEMATC

Commit message: Apply all the bodges so far
Parts:
- removed R8: 2kΩ, Resistors_SMD:R_0805_HandSoldering, symbol Device:R_Small_US
Connections:
- net labels added: CPU_CLK
- net labels removed: AUD_CLK
- wire segments 25 -> 22
Other:
- note added: "Revised June 2020:\nExtraneous 2k pullup R8\non /WAIT removed"
- note added: "Revised June 2020:\ntie sound chip to CPU clock directly"
- note removed: "TODO: REMOVE"
Changed lines of the file:
@@
 Wire Wire Line
 	5200 3875 5500 3875
-Text GLabel 5500 3875 2    50   Input ~ 0
-AUD_CLK
 Text GLabel 4200 4125 0    50   Input ~ 0
 Audio_WR
@@
 Text GLabel 5200 4275 2    50   Input ~ 0
 D0
-Connection ~ 3900 3975
 Wire Wire Line
-	3900 3975 3200 3975
+	3550 2725 5200 2725
 Wire Wire Line
-	4300 3975 3900 3975
-Connection ~ 3900 2725
-Wire Wire Line
-	3900 2725 3550 2725
-Wire Wire Line
-	5200 2725 3900 2725
-Wire Wire Line
-	3900 3975 3900 2925
-$Comp
-L Device:R_Small_US R8
-U 1 1 5E3CBFF6
-P 3900 2825
-F 0 "R8" H 3968 2871 50  0000 L CNN
-F 1 "2kΩ" H 3968 2780 50  0000 L CNN
-F 2 "Resistors_SMD:R_0805_HandSoldering" H 3900 2825 50  0001 C CNN
-F 3 "~" H 3900 2825 50  0001 C CNN
-	1    3900 2825
-	1    0    0    -1
-$EndComp
-Text Notes 3975 3050 0    50   ~ 10
-TODO: REMOVE
+	3200 3975 4300 3975
+Text Notes 4625 3275 2    50   ~ 0
+Revised June 2020:\nExtraneous 2k pullup R8\non /WAIT removed
+Text GLabel 5500 3875 2    50   Input ~ 0
+CPU_CLK
+Text Notes 6825 4075 2    50   ~ 0
+Revised June 2020:\ntie sound chip to CPU clock directly
 $EndSCHEMATC
