File: Sound.sch (KiCad schematic (older format))
At the start: 5 parts, among them J4 RCJ-017, U10 SN76489AN

Commit message: Coloured RCA jacks
Parts:
- J4: value RCJ-017 -> RCJ-013; DigiKey (none) -> CP-1402-ND‎
Changed lines of the file:
@@
 P 6675 4975
 F 0 "J4" H 6517 4924 50  0000 R CNN
-F 1 "RCJ-017" H 6517 5015 50  0000 R CNN
+F 1 "RCJ-013" H 6517 5015 50  0000 R CNN
 F 2 "Jacks:CUI_RCJ-017" H 6675 4975 50  0001 L BNN
 F 3 "CUI Inc" H 6675 4975 50  0001 L BNN
 F 4 "B" H 6675 4975 50  0001 L BNN "Field4"
 F 5 "Manufacturer recommendations" H 6675 4975 50  0001 L BNN "Field5"
+F 6 "CP-1402-ND‎" H 6675 4975 50  0001 C CNN "DigiKey"
 	1    6675 4975
 	-1   0    0    1

Commit message: BOM update
Parts:
- C13, C19: DigiKey (none) -> 1276-1099-1-ND
Changed lines of the file:
@@
 F 2 "Capacitors_SMD:C_0805_HandSoldering" H 3588 4825 50  0001 C CNN
 F 3 "~" H 3550 4975 50  0001 C CNN
+F 4 "1276-1099-1-ND" H 3550 4975 50  0001 C CNN "DigiKey"
 	1    3550 4975
 	1    0    0    -1
@@
 F 2 "Capacitors_SMD:C_0805_HandSoldering" H 6063 4725 50  0001 C CNN
 F 3 "~" H 6025 4875 50  0001 C CNN
+F 4 "1276-1099-1-ND" H 6025 4875 50  0001 C CNN "DigiKey"
 	1    6025 4875
 	0    1    1    0

Commit message: DigiKey BOM complete
Parts:
- R11: DigiKey (none) -> RMCF0805FT1K00CT-ND
- U10: DigiKey (none) -> AE9992-ND
Changed lines of the file:
@@
 F 2 "Housings_DIP:DIP-16_W7.62mm_Socket_LongPads" H 4750 4575 50  0001 C CNN
 F 3 "" H 4750 4575 50  0001 C CNN
+F 4 "AE9992-ND" H 4750 4025 50  0001 C CNN "DigiKey"
 	1    4750 4025
 	1    0    0    -1
@@
 F 2 "Resistors_SMD:R_0805_HandSoldering" H 5475 4875 50  0001 C CNN
 F 3 "~" H 5475 4875 50  0001 C CNN
+F 4 "RMCF0805FT1K00CT-ND" H 5475 4875 50  0001 C CNN "DigiKey"
 	1    5475 4875
 	0    1    1    0

Commit message: Replace 1k with 1.5k across the board to reduce BOM
Parts:
- R11: value 1kΩ -> 1.5kΩ
Changed lines of the file:
@@
 P 5475 4875
 F 0 "R11" V 5270 4875 50  0000 C CNN
-F 1 "1kΩ" V 5361 4875 50  0000 C CNN
+F 1 "1.5kΩ" V 5361 4875 50  0000 C CNN
 F 2 "Resistors_SMD:R_0805_HandSoldering" H 5475 4875 50  0001 C CNN
 F 3 "~" H 5475 4875 50  0001 C CNN
