File: Power.sch (KiCad schematic (older format))
At the start: 6 parts, among them J3 PJ-102A, SW1 Power Toggle

Commit message: Swap tip and ring for composite, finish up power
Parts:
- added D2: 50V 2A, Diodes_ThroughHole:D_DO-15_P10.16mm_Horizontal, symbol Device:D_Schottky
- added Q2: Q_NJFET_DGS, TO_SOT_Packages_SMD:SOT-23_Handsoldering, symbol Device:Q_NJFET_DGS
- added R12: 330Ω, Resistors_SMD:R_0805_HandSoldering, symbol Device:R_Small_US
- added R13: 10kΩ, Resistors_SMD:R_0805_HandSoldering, symbol Device:R_Small_US
Connections:
- net labels added: WALL_G, WALL_V
- net labels removed: RAW_5V
- wire segments 18 -> 30
Other:
- note added: "ColecoVision logic power"
- note added: "Should be centre positive"
- note removed: "TODO: power switch\nvery weak (0.1A)"

Commit message: Add test point bodges
Parts:
- added C20: 0.1µF, Capacitors_SMD:C_0805_HandSoldering, symbol Device:C
- added U14: 74LS02, Housings_SOIC:SOIC-14_3.9x8.7mm_Pitch1.27mm, symbol 74xx:74LS02
Connections:
- wire segments 30 -> 34
Changed lines of the file:
@@
 $Descr A4 11693 8268
 encoding utf-8
-Sheet 3 6
+Sheet 3 7
 Title ""
 Date ""
@@
 Text Notes 2350 1525 3    50   ~ 0
 Should be centre positive
+$Comp
+L 74xx:74LS02 U14
+U 5 1 5E4100D4
+P 10475 1725
+F 0 "U14" H 10705 1771 50  0000 L CNN
+F 1 "74LS02" H 10705 1680 50  0000 L CNN
+F 2 "Housings_SOIC:SOIC-14_3.9x8.7mm_Pitch1.27mm" H 10475 1725 50  0001 C CNN
+F 3 "http://www.ti.com/lit/gpn/sn74ls02" H 10475 1725 50  0001 C CNN
+	5    10475 1725
+	1    0    0    -1
+$EndComp
+$Comp
+L power:GND #PWR0116
+U 1 1 5E412F5E
+P 10475 2225
+F 0 "#PWR0116" H 10475 1975 50  0001 C CNN
+F 1 "GND" H 10480 2052 50  0000 C CNN
+F 2 "" H 10475 2225 50  0001 C CNN
+F 3 "" H 10475 2225 50  0001 C CNN
+	1    10475 2225
+	1    0    0    -1
+$EndComp
+$Comp
+L power:VCC #PWR0117
+U 1 1 5E413392
+P 10475 1225
+F 0 "#PWR0117" H 10475 1075 50  0001 C CNN
+F 1 "VCC" H 10492 1398 50  0000 C CNN
+F 2 "" H 10475 1225 50  0001 C CNN
+F 3 "" H 10475 1225 50  0001 C CNN
+	1    10475 1225
+	1    0    0    -1
+$EndComp
+Wire Wire Line
+	10475 1225 10175 1225
+Wire Wire Line
+	10175 1225 10175 1550
+Wire Wire Line
+	10175 2225 10475 2225
+Connection ~ 10475 1225
+Connection ~ 10475 2225
+$Comp
+L Device:C C20
+U 1 1 5E413C90
+P 10175 1700
+F 0 "C20" H 10290 1746 50  0000 L CNN
+F 1 "0.1µF" H 10290 1655 50  0000 L CNN
+F 2 "Capacitors_SMD:C_0805_HandSoldering" H 10213 1550 50  0001 C CNN
+F 3 "~" H 10175 1700 50  0001 C CNN
+	1    10175 1700
+	1    0    0    -1
+$EndComp
+Wire Wire Line
+	10175 1850 10175 2225
 $EndSCHEMATC

Commit message: Reset circuit
Parts:
- added C21: 1µF, Capacitors_SMD:C_0805_HandSoldering, symbol Device:C
- added C?: 0.1µF, Capacitors_SMD:C_0805_HandSoldering, symbol Device:C
- added R16: 91kΩ, Resistors_SMD:R_0805_HandSoldering, symbol Device:R_Small_US
- added R17: 1MΩ, Resistors_SMD:R_0805_HandSoldering, symbol Device:R_Small_US
- added R18, R21: 1kΩ, Resistors_SMD:R_0805_HandSoldering, symbol Device:R_Small_US
- added R19: 3.3kΩ, Resistors_SMD:R_0805_HandSoldering, symbol Device:R_Small_US
- added R20: 22kΩ, Resistors_SMD:R_0805_HandSoldering, symbol Device:R_Small_US
- added SW2: Reset, Buttons_Switches_ThroughHole:SW_PUSH_6mm, symbol Switch:SW_Push
- added U18: 74LS05, Housings_SOIC:SOIC-14_3.9x8.7mm_Pitch1.27mm, symbol 74xx:74LS05
Connections:
- net labels added: !RESET
- wire segments 34 -> 62
Other:
- note added: "EX_RES1"
- note added: "EX_RES2"
- note added: "Power"
- note added: "TODO: put a regulator in here - wall voltage is going to drop so it will be higher than 5V"
- note removed: "TODO: reset"
- note removed: "maybe put a regulator in here too?"

Commit message: Do not allow CPU to reset VDP
Parts:
- gave numbers to parts that had none: 1

Commit message: Clock crystal bullshit
Parts:
- added C2: 100nF, Capacitors_SMD:C_0805_HandSoldering, symbol Device:C
- added C23, C24, C28: 0.1µF, Capacitors_SMD:C_0805_HandSoldering, symbol Device:C
- added C25: 68µF, Capacitors_SMD:C_0805_HandSoldering, symbol Device:C
- added C26: 120nF, Capacitors_SMD:C_0805_HandSoldering, symbol Device:C
- added C27: 82J?, Capacitors_SMD:C_0805_HandSoldering, symbol Device:C
- added C3: 2.2nF, Capacitors_SMD:C_0805_HandSoldering, symbol Device:C
- added L1: 2.7µH, tdk-inductor:MLF2012A2R7KT000, symbol Device:L_Small
- added Q3: 2N3904, TO_SOT_Packages_THT:TO-92_Molded_Narrow, symbol Transistor_BJT:2N3904
- added R22, R28, R30: 1kΩ, Resistors_SMD:R_0805_HandSoldering, symbol Device:R_Small_US
- added R23: 330Ω, Resistors_SMD:R_0805_HandSoldering, symbol Device:R_Small_US
- added R24: 620Ω, Resistors_SMD:R_0805_HandSoldering, symbol Device:R_Small_US
- added R25: 1.1kΩ, Resistors_SMD:R_0805_HandSoldering, symbol Device:R_Small_US
- added R26: 180Ω, Resistors_SMD:R_0805_HandSoldering, symbol Device:R_Small_US
- added R27: 270Ω, Resistors_SMD:R_0805_HandSoldering, symbol Device:R_Small_US
- added R29: 22kΩ, Resistors_SMD:R_0805_HandSoldering, symbol Device:R_Small_US
- added U19, U21: 74HC04, Housings_SOIC:SOIC-14_3.9x8.7mm_Pitch1.27mm, symbol 74xx:74HC04
- added U20: 74LS74, Housings_SOIC:SOIC-14_3.9x8.7mm_Pitch1.27mm, symbol 74xx:74LS74
- added Y1: 7.15909, Crystals:Crystal_HC49-U_Vertical, symbol Device:Crystal
- U18: footprint (none) -> Housings_SOIC:SOIC-14_3.9x8.7mm_Pitch1.27mm
Connections:
- net labels added: !M1, !WAIT, AUD_CLK, CPU_CLK, VID_CLK
- wire segments 62 -> 144
- no-connect marks 1 -> 2
Other:
- note added: "Clock"

Commit message: 2x clock
Parts:
- removed Y1: 7.15909, Crystals:Crystal_HC49-U_Vertical, symbol Device:Crystal
- added C?: 0.1µF, Capacitors_SMD:C_0805_HandSoldering, symbol Device:C
- added U22: 74LS74, Housings_SOIC:SOIC-14_3.9x8.7mm_Pitch1.27mm, symbol 74xx:74LS74
- added Y?: 14.31818 (2x), Crystals:Crystal_HC49-U_Vertical, symbol Device:Crystal
Connections:
- net labels added: 14MHz, 7MHz
- wire segments 144 -> 162
Other:
- note added: "Crystal\n7.15909\nMHz"
Changed lines of the file:
@@
 	9950 5625 9950 5900
-$Comp
-L Device:Crystal Y1
-U 1 1 5E43F394
-P 3575 4425
-F 0 "Y1" H 3575 4693 50  0000 C CNN
-F 1 "7.15909" H 3575 4602 50  0000 C CNN
-F 2 "Crystals:Crystal_HC49-U_Vertical" H 3575 4425 50  0001 C CNN
-F 3 "~" H 3575 4425 50  0001 C CNN
-	1    3575 4425
-	1    0    0    -1
-$EndComp
 $Comp
 L Device:C C3
@@
 Connection ~ 3125 4425
 Wire Wire Line
-	3725 4425 3825 4425
-Wire Wire Line
 	3825 4425 3825 4050
 Wire Wire Line
@@
 Wire Wire Line
 	8900 5650 8900 6025
+$Comp
+L Device:Crystal Y?
+U 1 1 5E5A5EBE
+P 1325 5425
+F 0 "Y?" H 1325 5693 50  0000 C CNN
+F 1 "14.31818 (2x)" H 1325 5602 50  0000 C CNN
+F 2 "Crystals:Crystal_HC49-U_Vertical" H 1325 5425 50  0001 C CNN
+F 3 "https://www.digikey.ca/product-detail/en/9B-14.31818MBBK-B/887-1862-ND/3522029/?itemSeq=317149689" H 1325 5425 50  0001 C CNN
+	1    1325 5425
+	1    0    0    -1
+$EndComp
+$Comp
+L 74xx:74LS74 U22
+U 1 1 5E5A9C25
+P 2100 5425
+F 0 "U22" H 2100 5906 50  0000 C CNN
+F 1 "74LS74" H 2100 5815 50  0000 C CNN
+F 2 "Housings_SOIC:SOIC-14_3.9x8.7mm_Pitch1.27mm" H 2100 5425 50  0001 C CNN
+F 3 "74xx/74hc_hct74.pdf" H 2100 5425 50  0001 C CNN
+	1    2100 5425
+	1    0    0    -1
+$EndComp
+Wire Wire Line
+	1475 5425 1800 5425
+Wire Wire Line
+	2400 5525 2600 5525
+Wire Wire Line
+	2600 5525 2600 4950
+Wire Wire Line
+	2600 4950 1750 4950
+Wire Wire Line
+	1750 4950 1750 5325
+Wire Wire Line
+	1750 5325 1800 5325
+Wire Wire Line
+	2400 5325 3750 5325
+Wire Wire Line
+	3750 5325 3750 4425
+Wire Wire Line
+	3750 4425 3825 4425
+Wire Wire Line
+	1175 5425 800  5425
+Wire Wire Line
+	800  5425 800  4700
+Wire Wire Line
+	800  4700 3425 4700
+Wire Wire Line
+	3425 4700 3425 4425
+Text Notes 3750 4550 2    50   ~ 0
+Crystal\n7.15909\nMHz
+Wire Notes Line
+	3375 4200 3375 4650
+Wire Notes Line
+	3375 4650 3800 4650
+Wire Notes Line
+	3800 4650 3800 4200
+Wire Notes Line
+	3800 4200 3375 4200
+Text Label 3150 5325 2    50   ~ 0
+7MHz
+Text Label 1725 5425 2    50   ~ 0
+14MHz
+$Comp
+L power:VCC #PWR?
+U 1 1 5E5DE5C6
+P 2450 5725
+F 0 "#PWR?" H 2450 5575 50  0001 C CNN
+F 1 "VCC" H 2467 5898 50  0000 C CNN
+F 2 "" H 2450 5725 50  0001 C CNN
+F 3 "" H 2450 5725 50  0001 C CNN
+	1    2450 5725
+	1    0    0    -1
+$EndComp
+Wire Wire Line
+	2450 5725 2100 5725
+Wire Wire Line
+	2100 5125 2775 5125
+$Comp
+L power:VCC #PWR?
+U 1 1 5E5ED51B
+P 2775 5125
+F 0 "#PWR?" H 2775 4975 50  0001 C CNN
+F 1 "VCC" H 2792 5298 50  0000 C CNN
+F 2 "" H 2775 5125 50  0001 C CNN
+F 3 "" H 2775 5125 50  0001 C CNN
+	1    2775 5125
+	1    0    0    -1
+$EndComp
+$Comp
+L 74xx:74LS74 U22
+U 3 1 5E5F0EFF
+P 8300 5525
+F 0 "U22" H 8530 5571 50  0000 L CNN
+F 1 "74LS74" H 8530 5480 50  0000 L CNN
+F 2 "" H 8300 5525 50  0001 C CNN
+F 3 "74xx/74hc_hct74.pdf" H 8300 5525 50  0001 C CNN
+	3    8300 5525
+	1    0    0    -1
+$EndComp
+Wire Wire Line
+	8300 5125 7700 5125
+Wire Wire Line
+	7700 5125 7700 5375
+Wire Wire Line
+	7700 5925 8300 5925
+$Comp
+L Device:C C?
+U 1 1 5E5FFEE5
+P 7700 5525
+F 0 "C?" H 7815 5571 50  0000 L CNN
+F 1 "0.1µF" H 7815 5480 50  0000 L CNN
+F 2 "Capacitors_SMD:C_0805_HandSoldering" H 7738 5375 50  0001 C CNN
+F 3 "~" H 7700 5525 50  0001 C CNN
+	1    7700 5525
+	1    0    0    -1
+$EndComp
+Wire Wire Line
+	7700 5675 7700 5925
 $EndSCHEMATC

Commit message: Clock divider moved
Parts:
- gave numbers to parts that had none: 2
Connections:
- wire segments 162 -> 156
Other:
- note added: "Clock div/2\n(2x crystal was fitted)"
- note added: "TODO: tweak passives for x2 crystal"
- note removed: "Crystal\n7.15909\nMHz"
Changed lines of the file:
@@
 Wire Wire Line
 	7000 2575 7000 2825
-Wire Wire Line
-	7000 4900 5325 4900
 $Comp
 L Device:R_Small_US R27
@@
 Connection ~ 7000 3250
 Wire Wire Line
-	7000 3250 7000 4900
+	7000 3250 7000 4800
 $Comp
 L Device:C C26
@@
 Text GLabel 8950 3675 2    50   Input ~ 0
 VID_CLK
-Text Notes 5950 4500 2    50   ~ 0
+Text Notes 6425 3100 2    118  ~ 0
 Clock
 Wire Wire Line
@@
 	8900 5650 8900 6025
 $Comp
-L Device:Crystal Y?
+L Device:Crystal Y1
 U 1 1 5E5A5EBE
-P 1325 5425
-F 0 "Y?" H 1325 5693 50  0000 C CNN
-F 1 "14.31818 (2x)" H 1325 5602 50  0000 C CNN
-F 2 "Crystals:Crystal_HC49-U_Vertical" H 1325 5425 50  0001 C CNN
-F 3 "https://www.digikey.ca/product-detail/en/9B-14.31818MBBK-B/887-1862-ND/3522029/?itemSeq=317149689" H 1325 5425 50  0001 C CNN
-	1    1325 5425
+P 3575 4425
+F 0 "Y1" H 3575 4693 50  0000 C CNN
+F 1 "14.31818 (2x)" H 3575 4602 50  0000 C CNN
+F 2 "Crystals:Crystal_HC49-U_Vertical" H 3575 4425 50  0001 C CNN
+F 3 "https://www.digikey.ca/product-detail/en/9B-14.31818MBBK-B/887-1862-ND/3522029/?itemSeq=317149689" H 3575 4425 50  0001 C CNN
+	1    3575 4425
 	1    0    0    -1
 $EndComp
@@
 L 74xx:74LS74 U22
 U 1 1 5E5A9C25
-P 2100 5425
-F 0 "U22" H 2100 5906 50  0000 C CNN
-F 1 "74LS74" H 2100 5815 50  0000 C CNN
-F 2 "Housings_SOIC:SOIC-14_3.9x8.7mm_Pitch1.27mm" H 2100 5425 50  0001 C CNN
-F 3 "74xx/74hc_hct74.pdf" H 2100 5425 50  0001 C CNN
-	1    2100 5425
-	1    0    0    -1
-$EndComp
-Wire Wire Line
-	1475 5425 1800 5425
-Wire Wire Line
-	2400 5525 2600 5525
-Wire Wire Line
-	2600 5525 2600 4950
-Wire Wire Line
-	2600 4950 1750 4950
-Wire Wire Line
-	1750 4950 1750 5325
-Wire Wire Line
-	1750 5325 1800 5325
-Wire Wire Line
-	2400 5325 3750 5325
-Wire Wire Line
-	3750 5325 3750 4425
-Wire Wire Line
-	3750 4425 3825 4425
-Wire Wire Line
-	1175 5425 800  5425
-Wire Wire Line
-	800  5425 800  4700
-Wire Wire Line
-	800  4700 3425 4700
-Wire Wire Line
-	3425 4700 3425 4425
-Text Notes 3750 4550 2    50   ~ 0
-Crystal\n7.15909\nMHz
-Wire Notes Line
-	3375 4200 3375 4650
-Wire Notes Line
-	3375 4650 3800 4650
-Wire Notes Line
-	3800 4650 3800 4200
-Wire Notes Line
-	3800 4200 3375 4200
-Text Label 3150 5325 2    50   ~ 0
-7MHz
-Text Label 1725 5425 2    50   ~ 0
-14MHz
-$Comp
-L power:VCC #PWR?
+P 6100 4900
+F 0 "U22" H 6100 5381 50  0000 C CNN
+F 1 "74LS74" H 6100 5290 50  0000 C CNN
+F 2 "Housings_SOIC:SOIC-14_3.9x8.7mm_Pitch1.27mm" H 6100 4900 50  0001 C CNN
+F 3 "74xx/74hc_hct74.pdf" H 6100 4900 50  0001 C CNN
+	1    6100 4900
+	1    0    0    -1
+$EndComp
+$Comp
+L power:VCC #PWR0131
 U 1 1 5E5DE5C6
-P 2450 5725
-F 0 "#PWR?" H 2450 5575 50  0001 C CNN
-F 1 "VCC" H 2467 5898 50  0000 C CNN
-F 2 "" H 2450 5725 50  0001 C CNN
-F 3 "" H 2450 5725 50  0001 C CNN
-	1    2450 5725
-	1    0    0    -1
-$EndComp
-Wire Wire Line
-	2450 5725 2100 5725
-Wire Wire Line
-	2100 5125 2775 5125
-$Comp
-L power:VCC #PWR?
+P 6425 5200
+F 0 "#PWR0131" H 6425 5050 50  0001 C CNN
+F 1 "VCC" H 6442 5373 50  0000 C CNN
+F 2 "" H 6425 5200 50  0001 C CNN
+F 3 "" H 6425 5200 50  0001 C CNN
+	1    6425 5200
+	1    0    0    -1
+$EndComp
+$Comp
+L power:VCC #PWR0132
 U 1 1 5E5ED51B
-P 2775 5125
-F 0 "#PWR?" H 2775 4975 50  0001 C CNN
-F 1 "VCC" H 2792 5298 50  0000 C CNN
-F 2 "" H 2775 5125 50  0001 C CNN
-F 3 "" H 2775 5125 50  0001 C CNN
-	1    2775 5125
+P 6425 4600
+F 0 "#PWR0132" H 6425 4450 50  0001 C CNN
+F 1 "VCC" H 6442 4773 50  0000 C CNN
+F 2 "" H 6425 4600 50  0001 C CNN
+F 3 "" H 6425 4600 50  0001 C CNN
+	1    6425 4600
 	1    0    0    -1
 $EndComp
@@
 	7700 5925 8300 5925
 $Comp
-L Device:C C?
+L Device:C C29
 U 1 1 5E5FFEE5
 P 7700 5525
-F 0 "C?" H 7815 5571 50  0000 L CNN
+F 0 "C29" H 7815 5571 50  0000 L CNN
 F 1 "0.1µF" H 7815 5480 50  0000 L CNN
 F 2 "Capacitors_SMD:C_0805_HandSoldering" H 7738 5375 50  0001 C CNN
@@
 Wire Wire Line
 	7700 5675 7700 5925
+Wire Wire Line
+	3725 4425 3825 4425
+Text Notes 4550 4700 2    50   ~ 0
+TODO: tweak passives for x2 crystal
+Text Label 5600 4900 2    50   ~ 0
+14MHz
+Wire Wire Line
+	5800 4900 5325 4900
+Wire Wire Line
+	6400 4800 7000 4800
+Text Label 6875 4800 2    50   ~ 0
+7MHz
+Wire Wire Line
+	6400 5000 6575 5000
+Wire Wire Line
+	6575 5000 6575 4325
+Wire Wire Line
+	6575 4325 5650 4325
+Wire Wire Line
+	5650 4325 5650 4800
+Wire Wire Line
+	5650 4800 5800 4800
+Wire Wire Line
+	6425 4600 6100 4600
+Wire Wire Line
+	6100 5200 6425 5200
+Wire Notes Line
+	5600 5350 6650 5350
+Wire Notes Line
+	6650 5350 6650 4275
+Wire Notes Line
+	6650 4275 5600 4275
+Wire Notes Line
+	5600 4275 5600 5350
+Text Notes 5600 5350 0    50   ~ 0
+Clock div/2\n(2x crystal was fitted)
 $EndSCHEMATC

Commit message: notes for later
Other:
- note added: "TODO: dump this entire mess and make an oscillator\ndispense directly to pin 11 of the input flop"
- note added: "actually put in another clock divider first"
Changed lines of the file:
@@
 Text Notes 5600 5350 0    50   ~ 0
 Clock div/2\n(2x crystal was fitted)
+Text Notes 2600 5200 0    50   ~ 0
+TODO: dump this entire mess and make an oscillator\ndispense directly to pin 11 of the input flop
+Text Notes 2900 5500 0    50   ~ 0
+actually put in another clock divider first
 $EndSCHEMATC
