File: Power.sch (KiCad schematic (older format))
At the start: 47 parts, among them J3 PJ-102A, Q2 Q_NJFET_DGS, Q3 2N3904, SW1 Power Toggle, SW2 Reset, U14 74LS02, U18 74LS05, U19 74HC04, U20 74LS74, U21 74HC04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

Commit message: Soon the clock nightmare will be over
Parts:
- removed C3: 2.2nF, Capacitors_SMD:C_0805_HandSoldering, symbol Device:C
- removed R23: 330Ω, Resistors_SMD:R_0805_HandSoldering, symbol Device:R_Small_US
- removed R24: 620Ω, Resistors_SMD:R_0805_HandSoldering, symbol Device:R_Small_US
- removed unit 4 of U19
- removed unit 5 of U19
- removed Y1: 14.31818 (2x), Crystals:Crystal_HC49-U_Vertical, symbol Device:Crystal
- added X1: 14.31818MHz, Oscillators:Oscillator_DIP-8_LargePads, symbol Oscillator:CXO_DIP8
- C2: value 100nF -> 0.1µF
- C27: value 82J? -> 82pF
Connections:
- net labels added: 10MHz, 3.57MHz
- net labels removed: 14MHz
- wire segments 156 -> 146
- no-connect marks 2 -> 3
Other:
- note added: "I dumped this entire mess and made an oscillator\ndispense directly to pin 11 of the new extra clock divider"
- note added: "this is about where U8 on the original schematic starts\n"
- note removed: "TODO: dump this entire mess and make an oscillator\ndispense directly to pin 11 of the input flop"
- note removed: "TODO: tweak passives for x2 crystal"
- note removed: "actually put in another clock divider first"
Changed lines of the file:
@@
 	9950 5625 9950 5900
-$Comp
-L Device:C C3
-U 1 1 5E4427E6
-P 3575 3900
-F 0 "C3" V 3323 3900 50  0000 C CNN
-F 1 "2.2nF" V 3414 3900 50  0000 C CNN
-F 2 "Capacitors_SMD:C_0805_HandSoldering" H 3613 3750 50  0001 C CNN
-F 3 "~" H 3575 3900 50  0001 C CNN
-	1    3575 3900
-	0    1    1    0
-$EndComp
-Wire Wire Line
-	3725 3900 4325 3900
-$Comp
-L Device:C C2
-U 1 1 5E447A87
-P 3275 4425
-F 0 "C2" V 3023 4425 50  0000 C CNN
-F 1 "100nF" V 3114 4425 50  0000 C CNN
-F 2 "Capacitors_SMD:C_0805_HandSoldering" H 3313 4275 50  0001 C CNN
-F 3 "~" H 3275 4425 50  0001 C CNN
-	1    3275 4425
-	0    1    1    0
-$EndComp
-$Comp
-L 74xx:74HC04 U19
-U 4 1 5E44AB08
-P 2825 4425
-F 0 "U19" H 2825 4742 50  0000 C CNN
-F 1 "74HC04" H 2825 4651 50  0000 C CNN
-F 2 "Housings_SOIC:SOIC-14_3.9x8.7mm_Pitch1.27mm" H 2825 4425 50  0001 C CNN
-F 3 "https://assets.nexperia.com/documents/data-sheet/74HC_HCT04.pdf" H 2825 4425 50  0001 C CNN
-	4    2825 4425
-	1    0    0    -1
-$EndComp
-$Comp
-L Device:R_Small_US R23
-U 1 1 5E44C8E1
-P 2825 4050
-F 0 "R23" V 3030 4050 50  0000 C CNN
-F 1 "330Ω" V 2939 4050 50  0000 C CNN
-F 2 "Resistors_SMD:R_0805_HandSoldering" H 2825 4050 50  0001 C CNN
-F 3 "~" H 2825 4050 50  0001 C CNN
-	1    2825 4050
-	0    -1   -1   0
-$EndComp
-Wire Wire Line
-	2675 3900 2675 4050
-Wire Wire Line
-	2675 4050 2725 4050
-Wire Wire Line
-	2675 3900 3425 3900
-Wire Wire Line
-	2675 4050 2525 4050
-Wire Wire Line
-	2525 4050 2525 4425
-Connection ~ 2675 4050
-Wire Wire Line
-	3125 4050 2925 4050
-Connection ~ 3125 4425
-Wire Wire Line
-	3825 4425 3825 4050
-Wire Wire Line
-	3825 4050 3950 4050
-Wire Wire Line
-	4325 4050 4325 3900
-$Comp
-L Device:R_Small_US R24
-U 1 1 5E46CDED
-P 4050 4050
-F 0 "R24" V 3845 4050 50  0000 C CNN
-F 1 "620Ω" V 3936 4050 50  0000 C CNN
-F 2 "Resistors_SMD:R_0805_HandSoldering" H 4050 4050 50  0001 C CNN
-F 3 "~" H 4050 4050 50  0001 C CNN
-	1    4050 4050
-	0    1    1    0
-$EndComp
-Wire Wire Line
-	4150 4050 4325 4050
-$Comp
-L 74xx:74HC04 U19
-U 5 1 5E46EA93
-P 4125 4425
-F 0 "U19" H 4125 4742 50  0000 C CNN
-F 1 "74HC04" H 4125 4651 50  0000 C CNN
-F 2 "Housings_SOIC:SOIC-14_3.9x8.7mm_Pitch1.27mm" H 4125 4425 50  0001 C CNN
-F 3 "https://assets.nexperia.com/documents/data-sheet/74HC_HCT04.pdf" H 4125 4425 50  0001 C CNN
-	5    4125 4425
-	1    0    0    -1
-$EndComp
-Connection ~ 3825 4425
-Wire Wire Line
-	4425 4425 4525 4425
-Wire Wire Line
-	4525 4425 4525 4050
-Wire Wire Line
-	4525 4050 4325 4050
-Connection ~ 4325 4050
 $Comp
 L 74xx:74LS74 U20
@@
 $EndComp
 Wire Wire Line
-	3125 5000 4725 5000
-Wire Wire Line
-	3125 4425 3125 5000
-Wire Wire Line
 	4725 2850 4725 3275
 Wire Wire Line
@@
 Wire Wire Line
 	4875 3700 5150 3700
-Wire Wire Line
-	3125 4050 3125 4425
 Wire Wire Line
 	4725 4900 4725 3850
@@
 	7000 3250 7200 3250
 Connection ~ 7000 3250
-Wire Wire Line
-	7000 3250 7000 4800
 $Comp
 L Device:C C26
@@
 P 7975 3250
 F 0 "C27" V 7723 3250 50  0000 C CNN
-F 1 "82J?" V 7814 3250 50  0000 C CNN
+F 1 "82pF" V 7814 3250 50  0000 C CNN
 F 2 "Capacitors_SMD:C_0805_HandSoldering" H 8013 3100 50  0001 C CNN
 F 3 "~" H 7975 3250 50  0001 C CNN
@@
 	1    0    0    -1
 $EndComp
-Text GLabel 8950 3675 2    50   Input ~ 0
+Text GLabel 9325 3675 2    50   Input ~ 0
 VID_CLK
 Text Notes 6425 3100 2    118  ~ 0
@@
 	8900 5650 8900 6025
 $Comp
-L Device:Crystal Y1
-U 1 1 5E5A5EBE
-P 3575 4425
-F 0 "Y1" H 3575 4693 50  0000 C CNN
-F 1 "14.31818 (2x)" H 3575 4602 50  0000 C CNN
-F 2 "Crystals:Crystal_HC49-U_Vertical" H 3575 4425 50  0001 C CNN
-F 3 "https://www.digikey.ca/product-detail/en/9B-14.31818MBBK-B/887-1862-ND/3522029/?itemSeq=317149689" H 3575 4425 50  0001 C CNN
-	1    3575 4425
-	1    0    0    -1
-$EndComp
-$Comp
 L 74xx:74LS74 U22
 U 1 1 5E5A9C25
-P 6100 4900
-F 0 "U22" H 6100 5381 50  0000 C CNN
-F 1 "74LS74" H 6100 5290 50  0000 C CNN
-F 2 "Housings_SOIC:SOIC-14_3.9x8.7mm_Pitch1.27mm" H 6100 4900 50  0001 C CNN
-F 3 "74xx/74hc_hct74.pdf" H 6100 4900 50  0001 C CNN
-	1    6100 4900
+P 3750 4425
+F 0 "U22" H 3750 4906 50  0000 C CNN
+F 1 "74LS74" H 3750 4815 50  0000 C CNN
+F 2 "Housings_SOIC:SOIC-14_3.9x8.7mm_Pitch1.27mm" H 3750 4425 50  0001 C CNN
+F 3 "74xx/74hc_hct74.pdf" H 3750 4425 50  0001 C CNN
+	1    3750 4425
 	1    0    0    -1
 $EndComp
@@
 L power:VCC #PWR0131
 U 1 1 5E5DE5C6
-P 6425 5200
-F 0 "#PWR0131" H 6425 5050 50  0001 C CNN
-F 1 "VCC" H 6442 5373 50  0000 C CNN
-F 2 "" H 6425 5200 50  0001 C CNN
-F 3 "" H 6425 5200 50  0001 C CNN
-	1    6425 5200
+P 4075 4725
+F 0 "#PWR0131" H 4075 4575 50  0001 C CNN
+F 1 "VCC" H 4092 4898 50  0000 C CNN
+F 2 "" H 4075 4725 50  0001 C CNN
+F 3 "" H 4075 4725 50  0001 C CNN
+	1    4075 4725
 	1    0    0    -1
 $EndComp
@@
 L power:VCC #PWR0132
 U 1 1 5E5ED51B
-P 6425 4600
-F 0 "#PWR0132" H 6425 4450 50  0001 C CNN
-F 1 "VCC" H 6442 4773 50  0000 C CNN
-F 2 "" H 6425 4600 50  0001 C CNN
-F 3 "" H 6425 4600 50  0001 C CNN
-	1    6425 4600
+P 4075 4125
+F 0 "#PWR0132" H 4075 3975 50  0001 C CNN
+F 1 "VCC" H 4092 4298 50  0000 C CNN
+F 2 "" H 4075 4125 50  0001 C CNN
+F 3 "" H 4075 4125 50  0001 C CNN
+	1    4075 4125
 	1    0    0    -1
 $EndComp
@@
 Wire Wire Line
 	7700 5675 7700 5925
-Wire Wire Line
-	3725 4425 3825 4425
-Text Notes 4550 4700 2    50   ~ 0
-TODO: tweak passives for x2 crystal
-Text Label 5600 4900 2    50   ~ 0
-14MHz
-Wire Wire Line
-	5800 4900 5325 4900
-Wire Wire Line
-	6400 4800 7000 4800
-Text Label 6875 4800 2    50   ~ 0
+Text Label 4600 4325 2    50   ~ 0
 7MHz
 Wire Wire Line
-	6400 5000 6575 5000
-Wire Wire Line
-	6575 5000 6575 4325
-Wire Wire Line
-	6575 4325 5650 4325
-Wire Wire Line
-	5650 4325 5650 4800
-Wire Wire Line
-	5650 4800 5800 4800
-Wire Wire Line
-	6425 4600 6100 4600
-Wire Wire Line
-	6100 5200 6425 5200
+	4050 4325 4650 4325
+Wire Wire Line
+	4050 4525 4225 4525
+Wire Wire Line
+	4225 4525 4225 3850
+Wire Wire Line
+	4225 3850 3300 3850
+Wire Wire Line
+	3300 3850 3300 4325
+Wire Wire Line
+	3300 4325 3450 4325
+Wire Wire Line
+	4075 4125 3750 4125
+Wire Wire Line
+	3750 4725 4075 4725
 Wire Notes Line
-	5600 5350 6650 5350
+	3250 4875 4300 4875
 Wire Notes Line
-	6650 5350 6650 4275
+	4300 4875 4300 3800
 Wire Notes Line
-	6650 4275 5600 4275
+	4300 3800 3250 3800
 Wire Notes Line
-	5600 4275 5600 5350
-Text Notes 5600 5350 0    50   ~ 0
+	3250 3800 3250 4875
+Text Notes 3250 4875 0    50   ~ 0
 Clock div/2\n(2x crystal was fitted)
-Text Notes 2600 5200 0    50   ~ 0
-TODO: dump this entire mess and make an oscillator\ndispense directly to pin 11 of the input flop
-Text Notes 2900 5500 0    50   ~ 0
-actually put in another clock divider first
+Text Notes 2000 5075 0    50   ~ 0
+I dumped this entire mess and made an oscillator\ndispense directly to pin 11 of the new extra clock divider
+Text Notes 5450 5025 0    50   ~ 0
+this is about where U8 on the original schematic starts\n
+Wire Wire Line
+	5325 4900 7000 4900
+Wire Wire Line
+	7000 3250 7000 4900
+$Comp
+L Oscillator:CXO_DIP8 X1
+U 1 1 5E6EEF49
+P 2275 4425
+F 0 "X1" H 2619 4471 50  0000 L CNN
+F 1 "14.31818MHz" H 2619 4380 50  0000 L CNN
+F 2 "Oscillators:Oscillator_DIP-8_LargePads" H 2725 4075 50  0001 C CNN
+F 3 "https://www.digikey.ca/product-detail/en/abracon-llc/ACH-14.31818MHZ-EK/535-9170-5-ND/675365" H 2175 4425 50  0001 C CNN
+	1    2275 4425
+	1    0    0    -1
+$EndComp
+Wire Wire Line
+	4650 4325 4650 5000
+Wire Wire Line
+	4650 5000 4725 5000
+$Comp
+L power:VCC #PWR0133
+U 1 1 5E71302C
+P 2275 3825
+F 0 "#PWR0133" H 2275 3675 50  0001 C CNN
+F 1 "VCC" H 2292 3998 50  0000 C CNN
+F 2 "" H 2275 3825 50  0001 C CNN
+F 3 "" H 2275 3825 50  0001 C CNN
+	1    2275 3825
+	1    0    0    -1
+$EndComp
+$Comp
+L Device:C C2
+U 1 1 5E713B31
+P 1975 3825
+F 0 "C2" V 1723 3825 50  0000 C CNN
+F 1 "0.1µF" V 1814 3825 50  0000 C CNN
+F 2 "Capacitors_SMD:C_0805_HandSoldering" H 2013 3675 50  0001 C CNN
+F 3 "~" H 1975 3825 50  0001 C CNN
+	1    1975 3825
+	0    1    1    0
+$EndComp
+Wire Wire Line
+	2275 4125 2275 3825
+Wire Wire Line
+	2125 3825 2275 3825
+Connection ~ 2275 3825
+Wire Wire Line
+	1825 3825 1825 4725
+Wire Wire Line
+	1825 4725 2275 4725
+Wire Wire Line
+	2575 4425 3450 4425
+NoConn ~ 1975 4425
+Wire Wire Line
+	9325 3675 8950 3675
+Text Label 8975 3675 0    50   ~ 0
+10MHz
+Text Label 7000 3500 0    50   ~ 0
+3.57MHz
 $EndSCHEMATC

Commit message: Solder bridge jumpers
Connections:
- wire segments 146 -> 147
Changed lines of the file:
@@
 $EndComp
 Connection ~ 7650 2575
-Text GLabel 7850 2575 2    50   Input ~ 0
+Text GLabel 8625 2575 2    50   Input ~ 0
 CPU_CLK
-Text GLabel 8025 2025 2    50   Input ~ 0
+Text GLabel 8625 2025 2    50   Input ~ 0
 AUD_CLK
-Wire Wire Line
-	8025 2025 7950 2025
 $Comp
 L Device:R_Small_US R30
@@
 Text Label 7000 3500 0    50   ~ 0
 3.57MHz
+Wire Wire Line
+	7950 2025 8625 2025
+Wire Wire Line
+	8625 2575 7850 2575
 $EndSCHEMATC

Commit message: Shunt to ground
Parts:
- added F2: 2A, 0251002.MRT1L:0251002.MRT1L, symbol Device:Fuse_Small
Connections:
- wire segments 147 -> 150
Changed lines of the file:
@@
 L Device:Polyfuse F1
 U 1 1 5E400A91
-P 2800 1825
-F 0 "F1" H 2888 1871 50  0000 L CNN
-F 1 "1.0A" H 2888 1780 50  0000 L CNN
-F 2 "0ZCK-polyfuse:0ZCK0100FF2E" H 2850 1625 50  0001 L CNN
-F 3 "~" H 2800 1825 50  0001 C CNN
-	1    2800 1825
+P 2575 1825
+F 0 "F1" H 2663 1871 50  0000 L CNN
+F 1 "1.0A" H 2663 1780 50  0000 L CNN
+F 2 "0ZCK-polyfuse:0ZCK0100FF2E" H 2625 1625 50  0001 L CNN
+F 3 "~" H 2575 1825 50  0001 C CNN
+	1    2575 1825
 	0    -1   -1   0
 $EndComp
@@
 $EndComp
 Wire Wire Line
-	2150 1825 2650 1825
-Wire Wire Line
 	3275 1225 3275 725
 Wire Wire Line
@@
 Text Label 1325 1675 3    50   ~ 0
 WALL_V
-Wire Wire Line
-	1350 1775 1450 1775
-Wire Wire Line
-	1175 1475 1950 1475
 $Comp
 L Device:D_Schottky D2
 U 1 1 5E473FC7
-P 1600 1775
-F 0 "D2" H 1600 1559 50  0000 C CNN
-F 1 "50V 2A" H 1600 1650 50  0000 C CNN
-F 2 "Diodes_ThroughHole:D_DO-15_P10.16mm_Horizontal" H 1600 1775 50  0001 C CNN
-F 3 "https://www.digikey.ca/product-detail/en/RL201-TP/RL201-TPCT-ND/950498/?itemSeq=317130355" H 1600 1775 50  0001 C CNN
-	1    1600 1775
-	-1   0    0    1
-$EndComp
-Wire Wire Line
-	1750 1775 1950 1775
+P 1725 1625
+F 0 "D2" H 1725 1409 50  0000 C CNN
+F 1 "50V 2A" H 1725 1500 50  0000 C CNN
+F 2 "Diodes_ThroughHole:D_DO-15_P10.16mm_Horizontal" H 1725 1625 50  0001 C CNN
+F 3 "https://www.digikey.ca/product-detail/en/RL201-TP/RL201-TPCT-ND/950498/?itemSeq=317130355" H 1725 1625 50  0001 C CNN
+	1    1725 1625
+	0    1    -1   0
+$EndComp
 $Comp
 L power:PWR_FLAG #FLG0102
@@
 Wire Wire Line
 	8625 2575 7850 2575
+Wire Wire Line
+	2150 1825 2425 1825
+Wire Wire Line
+	2725 1825 2950 1825
+$Comp
+L Device:Fuse_Small F2
+U 1 1 5E46D729
+P 1475 1775
+F 0 "F2" H 1475 1925 50  0000 C CNN
+F 1 "2A" H 1475 1850 50  0000 C CNN
+F 2 "0251002.MRT1L:0251002.MRT1L" H 1475 1775 50  0001 C CNN
+F 3 "https://www.digikey.ca/product-detail/en/littelfuse-inc/0251002.MRT1L/F3171CT-ND/1984467" H 1475 1775 50  0001 C CNN
+	1    1475 1775
+	1    0    0    1
+$EndComp
+Wire Wire Line
+	1175 1475 1725 1475
+Wire Wire Line
+	1350 1775 1375 1775
+Wire Wire Line
+	1575 1775 1725 1775
+Connection ~ 1725 1775
+Wire Wire Line
+	1725 1775 1950 1775
+Connection ~ 1725 1475
+Wire Wire Line
+	1725 1475 1950 1475
 $EndSCHEMATC

Commit message: Ditch the polyfuse
Parts:
- removed F1: 1.0A, 0ZCK-polyfuse:0ZCK0100FF2E, symbol Device:Polyfuse
Connections:
- wire segments 150 -> 149
Changed lines of the file:
@@
-$EndComp
-$Comp
-L Device:Polyfuse F1
-U 1 1 5E400A91
-P 2575 1825
-F 0 "F1" H 2663 1871 50  0000 L CNN
-F 1 "1.0A" H 2663 1780 50  0000 L CNN
-F 2 "0ZCK-polyfuse:0ZCK0100FF2E" H 2625 1625 50  0001 L CNN
-F 3 "~" H 2575 1825 50  0001 C CNN
-	1    2575 1825
-	0    -1   -1   0
 $EndComp
 $Comp
@@
 Wire Wire Line
 	8625 2575 7850 2575
-Wire Wire Line
-	2150 1825 2425 1825
-Wire Wire Line
-	2725 1825 2950 1825
 $Comp
 L Device:Fuse_Small F2
@@
 Wire Wire Line
 	1725 1475 1950 1475
+Wire Wire Line
+	2150 1825 2950 1825
 $EndSCHEMATC

Commit message: All the controller stuff is on the PCB now
Parts:
- U22: footprint (none) -> Housings_SOIC:SOIC-14_3.9x8.7mm_Pitch1.27mm
Changed lines of the file:
@@
 F 0 "U22" H 8530 5571 50  0000 L CNN
 F 1 "74LS74" H 8530 5480 50  0000 L CNN
-F 2 "" H 8300 5525 50  0001 C CNN
+F 2 "Housings_SOIC:SOIC-14_3.9x8.7mm_Pitch1.27mm" H 8300 5525 50  0001 C CNN
 F 3 "74xx/74hc_hct74.pdf" H 8300 5525 50  0001 C CNN
 	3    8300 5525

Commit message: -5V line added
Parts:
- added C? (x2): 1µF, Capacitors_SMD:C_0805_HandSoldering, symbol Device:C
- added C?: C, Capacitors_SMD:C_0805_HandSoldering, symbol Device:C
- added U?: TPS60403DBVR, TO_SOT_Packages_SMD:SOT-23-5_HandSoldering, symbol TPS60403DBVR:TPS60403DBVR
Connections:
- net labels added: -5V
- wire segments 149 -> 165
Other:
- note added: "-5V Generator"
Changed lines of the file:
@@
 Wire Wire Line
 	2150 1825 2950 1825
+$Comp
+L TPS60403DBVR:TPS60403DBVR U?
+U 1 1 5E44B69D
+P 7375 1075
+F 0 "U?" H 7375 1412 60  0000 C CNN
+F 1 "TPS60403DBVR" H 7375 1306 60  0000 C CNN
+F 2 "TO_SOT_Packages_SMD:SOT-23-5_HandSoldering" H 7375 1315 60  0001 C CNN
+F 3 "" H 6775 1075 60  0000 C CNN
+	1    7375 1075
+	1    0    0    -1
+$EndComp
+$Comp
+L power:VCC #PWR?
+U 1 1 5E44CEA9
+P 6200 1175
+F 0 "#PWR?" H 6200 1025 50  0001 C CNN
+F 1 "VCC" H 6217 1348 50  0000 C CNN
+F 2 "" H 6200 1175 50  0001 C CNN
+F 3 "" H 6200 1175 50  0001 C CNN
+	1    6200 1175
+	1    0    0    -1
+$EndComp
+Wire Wire Line
+	6775 1175 6750 1175
+Text GLabel 6375 800  0    50   Input ~ 10
+-5V
+$Comp
+L Device:C C?
+U 1 1 5E455A6F
+P 6750 1325
+F 0 "C?" H 6865 1371 50  0000 L CNN
+F 1 "1µF" H 6865 1280 50  0000 L CNN
+F 2 "Capacitors_SMD:C_0805_HandSoldering" H 6788 1175 50  0001 C CNN
+F 3 "~" H 6750 1325 50  0001 C CNN
+	1    6750 1325
+	1    0    0    -1
+$EndComp
+Connection ~ 6750 1175
+Wire Wire Line
+	6750 1175 6200 1175
+Wire Wire Line
+	6750 1475 7400 1475
+Wire Wire Line
+	8225 1475 8225 1175
+Wire Wire Line
+	8225 1175 7975 1175
+$Comp
+L power:GND #PWR?
+U 1 1 5E45EB9C
+P 7400 1475
+F 0 "#PWR?" H 7400 1225 50  0001 C CNN
+F 1 "GND" H 7405 1302 50  0000 C CNN
+F 2 "" H 7400 1475 50  0001 C CNN
+F 3 "" H 7400 1475 50  0001 C CNN
+	1    7400 1475
+	1    0    0    -1
+$EndComp
+Connection ~ 7400 1475
+Wire Wire Line
+	7400 1475 8225 1475
+$Comp
+L Device:C C?
+U 1 1 5E46030F
+P 8425 1175
+F 0 "C?" H 8540 1221 50  0000 L CNN
+F 1 "1µF" H 8540 1130 50  0000 L CNN
+F 2 "Capacitors_SMD:C_0805_HandSoldering" H 8463 1025 50  0001 C CNN
+F 3 "~" H 8425 1175 50  0001 C CNN
+	1    8425 1175
+	1    0    0    -1
+$EndComp
+Wire Wire Line
+	7975 1275 7975 1350
+Wire Wire Line
+	7975 1350 8425 1350
+Wire Wire Line
+	8425 1350 8425 1325
+Wire Wire Line
+	8425 1025 8425 1000
+Wire Wire Line
+	8425 1000 7975 1000
+Wire Wire Line
+	7975 1000 7975 1075
+Wire Wire Line
+	6775 1075 6450 1075
+Wire Wire Line
+	6450 1075 6450 800
+Wire Wire Line
+	6450 800  6375 800
+$Comp
+L Device:C C?
+U 1 1 5E47B3B1
+P 6450 1525
+F 0 "C?" H 6565 1571 50  0000 L CNN
+F 1 "C" H 6565 1480 50  0000 L CNN
+F 2 "Capacitors_SMD:C_0805_HandSoldering" H 6488 1375 50  0001 C CNN
+F 3 "~" H 6450 1525 50  0001 C CNN
+	1    6450 1525
+	1    0    0    -1
+$EndComp
+$Comp
+L power:GND #PWR?
+U 1 1 5E47BF5D
+P 6450 1675
+F 0 "#PWR?" H 6450 1425 50  0001 C CNN
+F 1 "GND" H 6455 1502 50  0000 C CNN
+F 2 "" H 6450 1675 50  0001 C CNN
+F 3 "" H 6450 1675 50  0001 C CNN
+	1    6450 1675
+	1    0    0    -1
+$EndComp
+Wire Wire Line
+	6450 1375 6450 1075
+Connection ~ 6450 1075
+Wire Notes Line
+	5775 600  5775 2000
+Wire Notes Line
+	5775 2000 7600 2000
+Wire Notes Line
+	7600 2000 7600 1650
+Wire Notes Line
+	7600 1650 8875 1650
+Wire Notes Line
+	8875 1650 8875 600
+Wire Notes Line
+	8875 600  5775 600
+Text Notes 8275 700  0    50   ~ 0
+-5V Generator
 $EndSCHEMATC

Commit message: -5V updated
Parts:
- C39: renamed from C?; value C -> 1µF
- gave numbers to parts that had none: 3
Changed lines of the file:
@@
 	2150 1825 2950 1825
 $Comp
-L TPS60403DBVR:TPS60403DBVR U?
+L TPS60403DBVR:TPS60403DBVR U24
 U 1 1 5E44B69D
 P 7375 1075
-F 0 "U?" H 7375 1412 60  0000 C CNN
+F 0 "U24" H 7375 1412 60  0000 C CNN
 F 1 "TPS60403DBVR" H 7375 1306 60  0000 C CNN
 F 2 "TO_SOT_Packages_SMD:SOT-23-5_HandSoldering" H 7375 1315 60  0001 C CNN
@@
 $EndComp
 $Comp
-L power:VCC #PWR?
+L power:VCC #PWR0144
 U 1 1 5E44CEA9
 P 6200 1175
-F 0 "#PWR?" H 6200 1025 50  0001 C CNN
+F 0 "#PWR0144" H 6200 1025 50  0001 C CNN
 F 1 "VCC" H 6217 1348 50  0000 C CNN
 F 2 "" H 6200 1175 50  0001 C CNN
@@
 -5V
 $Comp
-L Device:C C?
+L Device:C C40
 U 1 1 5E455A6F
 P 6750 1325
-F 0 "C?" H 6865 1371 50  0000 L CNN
+F 0 "C40" H 6865 1371 50  0000 L CNN
 F 1 "1µF" H 6865 1280 50  0000 L CNN
 F 2 "Capacitors_SMD:C_0805_HandSoldering" H 6788 1175 50  0001 C CNN
@@
 	8225 1175 7975 1175
 $Comp
-L power:GND #PWR?
+L power:GND #PWR0145
 U 1 1 5E45EB9C
 P 7400 1475
-F 0 "#PWR?" H 7400 1225 50  0001 C CNN
+F 0 "#PWR0145" H 7400 1225 50  0001 C CNN
 F 1 "GND" H 7405 1302 50  0000 C CNN
 F 2 "" H 7400 1475 50  0001 C CNN
@@
 	7400 1475 8225 1475
 $Comp
-L Device:C C?
+L Device:C C41
 U 1 1 5E46030F
 P 8425 1175
-F 0 "C?" H 8540 1221 50  0000 L CNN
+F 0 "C41" H 8540 1221 50  0000 L CNN
 F 1 "1µF" H 8540 1130 50  0000 L CNN
 F 2 "Capacitors_SMD:C_0805_HandSoldering" H 8463 1025 50  0001 C CNN
@@
 	6450 800  6375 800
 $Comp
-L Device:C C?
+L Device:C C39
 U 1 1 5E47B3B1
 P 6450 1525
-F 0 "C?" H 6565 1571 50  0000 L CNN
-F 1 "C" H 6565 1480 50  0000 L CNN
+F 0 "C39" H 6565 1571 50  0000 L CNN
+F 1 "1µF" H 6565 1480 50  0000 L CNN
 F 2 "Capacitors_SMD:C_0805_HandSoldering" H 6488 1375 50  0001 C CNN
 F 3 "~" H 6450 1525 50  0001 C CNN
@@
 $EndComp
 $Comp
-L power:GND #PWR?
+L power:GND #PWR0146
 U 1 1 5E47BF5D
 P 6450 1675
-F 0 "#PWR?" H 6450 1425 50  0001 C CNN
+F 0 "#PWR0146" H 6450 1425 50  0001 C CNN
 F 1 "GND" H 6455 1502 50  0000 C CNN
 F 2 "" H 6450 1675 50  0001 C CNN

Commit message: Add test point
Parts:
- added TP?: -5V, Measurement_Points:Measurement_Point_Round-SMD-Pad_Small, symbol Connector:TestPoint
Connections:
- wire segments 165 -> 166
Changed lines of the file:
@@
 	6775 1075 6450 1075
 Wire Wire Line
-	6450 1075 6450 800
+	6450 1075 6450 875
 Wire Wire Line
 	6450 800  6375 800
@@
 Text Notes 8275 700  0    50   ~ 0
 -5V Generator
+$Comp
+L Connector:TestPoint TP?
+U 1 1 5E49426A
+P 6450 875
+F 0 "TP?" V 6404 1063 50  0000 L CNN
+F 1 "-5V" V 6495 1063 50  0000 L CNN
+F 2 "Measurement_Points:Measurement_Point_Round-SMD-Pad_Small" H 6650 875 50  0001 C CNN
+F 3 "~" H 6650 875 50  0001 C CNN
+	1    6450 875
+	0    1    1    0
+$EndComp
+Connection ~ 6450 875
+Wire Wire Line
+	6450 875  6450 800
 $EndSCHEMATC
