File: Power.sch (KiCad schematic (older format))
At the start: 38 parts, among them J3 USB-B1HSB6, Q2 Q_NJFET_GSD, SW1 Power Toggle, SW2 Reset, U11 74LS04, U14 74LS02, U17 74LS05, U18 74LS05, U2 ICL7660, U20 74LS74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

Commit message: U17 unused inputs grounded
Parts:
- added unit 2 of U17
- added unit 3 of U17
- added unit 4 of U17
- added unit 5 of U17
Connections:
- wire segments 128 -> 136
- no-connect marks 5 -> 9
Changed lines of the file:
@@
 Text Notes 600  1050 0    50   ~ 0
 Revised Jan 2022:\nRemoved barrel jack and reverse-polarity protection diode\nfor 5V USB-B jack (should make it easier to find a PSU as well)
+$Comp
+L 74xx:74LS05 U17
+U 2 1 61D42566
+P 7450 4650
+F 0 "U17" H 7450 4967 50  0000 C CNN
+F 1 "74LS05" H 7450 4876 50  0000 C CNN
+F 2 "" H 7450 4650 50  0001 C CNN
+F 3 "http://www.ti.com/lit/gpn/sn74LS05" H 7450 4650 50  0001 C CNN
+	2    7450 4650
+	1    0    0    -1
+$EndComp
+$Comp
+L 74xx:74LS05 U17
+U 3 1 61D432FA
+P 7450 5050
+F 0 "U17" H 7450 5367 50  0000 C CNN
+F 1 "74LS05" H 7450 5276 50  0000 C CNN
+F 2 "" H 7450 5050 50  0001 C CNN
+F 3 "http://www.ti.com/lit/gpn/sn74LS05" H 7450 5050 50  0001 C CNN
+	3    7450 5050
+	1    0    0    -1
+$EndComp
+$Comp
+L 74xx:74LS05 U17
+U 4 1 61D447EC
+P 7450 5450
+F 0 "U17" H 7450 5767 50  0000 C CNN
+F 1 "74LS05" H 7450 5676 50  0000 C CNN
+F 2 "" H 7450 5450 50  0001 C CNN
+F 3 "http://www.ti.com/lit/gpn/sn74LS05" H 7450 5450 50  0001 C CNN
+	4    7450 5450
+	1    0    0    -1
+$EndComp
+$Comp
+L 74xx:74LS05 U17
+U 5 1 61D45FA1
+P 7450 5850
+F 0 "U17" H 7450 6167 50  0000 C CNN
+F 1 "74LS05" H 7450 6076 50  0000 C CNN
+F 2 "" H 7450 5850 50  0001 C CNN
+F 3 "http://www.ti.com/lit/gpn/sn74LS05" H 7450 5850 50  0001 C CNN
+	5    7450 5850
+	1    0    0    -1
+$EndComp
+NoConn ~ 7750 4650
+NoConn ~ 7750 5050
+NoConn ~ 7750 5450
+NoConn ~ 7750 5850
+$Comp
+L power:GND #PWR?
+U 1 1 61D5A562
+P 7050 6000
+F 0 "#PWR?" H 7050 5750 50  0001 C CNN
+F 1 "GND" H 7055 5827 50  0000 C CNN
+F 2 "" H 7050 6000 50  0001 C CNN
+F 3 "" H 7050 6000 50  0001 C CNN
+	1    7050 6000
+	1    0    0    -1
+$EndComp
+Wire Wire Line
+	7050 6000 7050 5850
+Wire Wire Line
+	7050 4650 7150 4650
+Wire Wire Line
+	7150 5050 7050 5050
+Connection ~ 7050 5050
+Wire Wire Line
+	7050 5050 7050 4650
+Wire Wire Line
+	7150 5450 7050 5450
+Connection ~ 7050 5450
+Wire Wire Line
+	7050 5450 7050 5050
+Wire Wire Line
+	7150 5850 7050 5850
+Connection ~ 7050 5850
+Wire Wire Line
+	7050 5850 7050 5450
 $EndSCHEMATC

Commit message: Ground unused inputs of u11
Parts:
- added unit 1 of U11
- added unit 2 of U11
- added unit 4 of U11
- added unit 5 of U11
- added unit 6 of U11
- U11: footprint (none) -> Housings_SOIC:SOIC-14_3.9x8.7mm_Pitch1.27mm
Connections:
- wire segments 136 -> 146
- no-connect marks 9 -> 14
Changed lines of the file:
@@
 F 0 "U11" H 9805 1196 50  0000 L CNN
 F 1 "74LS04" H 9805 1105 50  0000 L CNN
-F 2 "" H 9575 1150 50  0001 C CNN
+F 2 "Housings_SOIC:SOIC-14_3.9x8.7mm_Pitch1.27mm" H 9575 1150 50  0001 C CNN
 F 3 "http://www.ti.com/lit/gpn/sn74LS04" H 9575 1150 50  0001 C CNN
 	7    9575 1150
@@
 L 74xx:74LS05 U17
 U 2 1 61D42566
-P 7450 4650
-F 0 "U17" H 7450 4967 50  0000 C CNN
-F 1 "74LS05" H 7450 4876 50  0000 C CNN
-F 2 "" H 7450 4650 50  0001 C CNN
-F 3 "http://www.ti.com/lit/gpn/sn74LS05" H 7450 4650 50  0001 C CNN
-	2    7450 4650
+P 8050 4650
+F 0 "U17" H 8050 4967 50  0000 C CNN
+F 1 "74LS05" H 8050 4876 50  0000 C CNN
+F 2 "" H 8050 4650 50  0001 C CNN
+F 3 "http://www.ti.com/lit/gpn/sn74LS05" H 8050 4650 50  0001 C CNN
+	2    8050 4650
 	1    0    0    -1
 $EndComp
@@
 L 74xx:74LS05 U17
 U 3 1 61D432FA
-P 7450 5050
-F 0 "U17" H 7450 5367 50  0000 C CNN
-F 1 "74LS05" H 7450 5276 50  0000 C CNN
-F 2 "" H 7450 5050 50  0001 C CNN
-F 3 "http://www.ti.com/lit/gpn/sn74LS05" H 7450 5050 50  0001 C CNN
-	3    7450 5050
+P 8050 5050
+F 0 "U17" H 8050 5275 50  0000 C CNN
+F 1 "74LS05" H 8050 5276 50  0001 C CNN
+F 2 "" H 8050 5050 50  0001 C CNN
+F 3 "http://www.ti.com/lit/gpn/sn74LS05" H 8050 5050 50  0001 C CNN
+	3    8050 5050
 	1    0    0    -1
 $EndComp
@@
 L 74xx:74LS05 U17
 U 4 1 61D447EC
-P 7450 5450
-F 0 "U17" H 7450 5767 50  0000 C CNN
-F 1 "74LS05" H 7450 5676 50  0000 C CNN
-F 2 "" H 7450 5450 50  0001 C CNN
-F 3 "http://www.ti.com/lit/gpn/sn74LS05" H 7450 5450 50  0001 C CNN
-	4    7450 5450
+P 8050 5450
+F 0 "U17" H 8050 5675 50  0000 C CNN
+F 1 "74LS05" H 8050 5676 50  0001 C CNN
+F 2 "" H 8050 5450 50  0001 C CNN
+F 3 "http://www.ti.com/lit/gpn/sn74LS05" H 8050 5450 50  0001 C CNN
+	4    8050 5450
 	1    0    0    -1
 $EndComp
@@
 L 74xx:74LS05 U17
 U 5 1 61D45FA1
-P 7450 5850
-F 0 "U17" H 7450 6167 50  0000 C CNN
-F 1 "74LS05" H 7450 6076 50  0000 C CNN
-F 2 "" H 7450 5850 50  0001 C CNN
-F 3 "http://www.ti.com/lit/gpn/sn74LS05" H 7450 5850 50  0001 C CNN
-	5    7450 5850
-	1    0    0    -1
-$EndComp
-NoConn ~ 7750 4650
-NoConn ~ 7750 5050
-NoConn ~ 7750 5450
-NoConn ~ 7750 5850
-$Comp
-L power:GND #PWR?
+P 8050 5850
+F 0 "U17" H 8050 6075 50  0000 C CNN
+F 1 "74LS05" H 8050 6076 50  0001 C CNN
+F 2 "" H 8050 5850 50  0001 C CNN
+F 3 "http://www.ti.com/lit/gpn/sn74LS05" H 8050 5850 50  0001 C CNN
+	5    8050 5850
+	1    0    0    -1
+$EndComp
+NoConn ~ 8350 4650
+NoConn ~ 8350 5050
+NoConn ~ 8350 5450
+NoConn ~ 8350 5850
+$Comp
+L power:GND #PWR0134
 U 1 1 61D5A562
-P 7050 6000
-F 0 "#PWR?" H 7050 5750 50  0001 C CNN
-F 1 "GND" H 7055 5827 50  0000 C CNN
-F 2 "" H 7050 6000 50  0001 C CNN
-F 3 "" H 7050 6000 50  0001 C CNN
-	1    7050 6000
-	1    0    0    -1
-$EndComp
-Wire Wire Line
-	7050 6000 7050 5850
-Wire Wire Line
-	7050 4650 7150 4650
-Wire Wire Line
-	7150 5050 7050 5050
-Connection ~ 7050 5050
-Wire Wire Line
-	7050 5050 7050 4650
-Wire Wire Line
-	7150 5450 7050 5450
-Connection ~ 7050 5450
-Wire Wire Line
-	7050 5450 7050 5050
-Wire Wire Line
-	7150 5850 7050 5850
-Connection ~ 7050 5850
-Wire Wire Line
-	7050 5850 7050 5450
+P 7650 6000
+F 0 "#PWR0134" H 7650 5750 50  0001 C CNN
+F 1 "GND" H 7655 5827 50  0000 C CNN
+F 2 "" H 7650 6000 50  0001 C CNN
+F 3 "" H 7650 6000 50  0001 C CNN
+	1    7650 6000
+	1    0    0    -1
+$EndComp
+Wire Wire Line
+	7650 6000 7650 5850
+Wire Wire Line
+	7650 4650 7750 4650
+Wire Wire Line
+	7750 5050 7650 5050
+Connection ~ 7650 5050
+Wire Wire Line
+	7650 5050 7650 4650
+Wire Wire Line
+	7750 5450 7650 5450
+Connection ~ 7650 5450
+Wire Wire Line
+	7650 5450 7650 5050
+Wire Wire Line
+	7750 5850 7650 5850
+Connection ~ 7650 5850
+Wire Wire Line
+	7650 5850 7650 5450
+$Comp
+L 74xx:74LS04 U11
+U 1 1 61D7B6C8
+P 6750 4650
+F 0 "U11" H 6750 4967 50  0000 C CNN
+F 1 "74LS04" H 6750 4876 50  0000 C CNN
+F 2 "Housings_SOIC:SOIC-14_3.9x8.7mm_Pitch1.27mm" H 6750 4650 50  0001 C CNN
+F 3 "http://www.ti.com/lit/gpn/sn74LS04" H 6750 4650 50  0001 C CNN
+	1    6750 4650
+	1    0    0    -1
+$EndComp
+$Comp
+L 74xx:74LS04 U11
+U 2 1 61D7CE87
+P 6750 5050
+F 0 "U11" H 6750 5275 50  0000 C CNN
+F 1 "74LS04" H 6750 5276 50  0001 C CNN
+F 2 "Housings_SOIC:SOIC-14_3.9x8.7mm_Pitch1.27mm" H 6750 5050 50  0001 C CNN
+F 3 "http://www.ti.com/lit/gpn/sn74LS04" H 6750 5050 50  0001 C CNN
+	2    6750 5050
+	1    0    0    -1
+$EndComp
+$Comp
+L 74xx:74LS04 U11
+U 4 1 61D7E168
+P 6750 5450
+F 0 "U11" H 6750 5675 50  0000 C CNN
+F 1 "74LS04" H 6750 5676 50  0001 C CNN
+F 2 "Housings_SOIC:SOIC-14_3.9x8.7mm_Pitch1.27mm" H 6750 5450 50  0001 C CNN
+F 3 "http://www.ti.com/lit/gpn/sn74LS04" H 6750 5450 50  0001 C CNN
+	4    6750 5450
+	1    0    0    -1
+$EndComp
+$Comp
+L 74xx:74LS04 U11
+U 5 1 61D7F5D8
+P 6750 5850
+F 0 "U11" H 6750 6075 50  0000 C CNN
+F 1 "74LS04" H 6750 6076 50  0001 C CNN
+F 2 "Housings_SOIC:SOIC-14_3.9x8.7mm_Pitch1.27mm" H 6750 5850 50  0001 C CNN
+F 3 "http://www.ti.com/lit/gpn/sn74LS04" H 6750 5850 50  0001 C CNN
+	5    6750 5850
+	1    0    0    -1
+$EndComp
+$Comp
+L 74xx:74LS04 U11
+U 6 1 61D80D4F
+P 6750 6250
+F 0 "U11" H 6750 6475 50  0000 C CNN
+F 1 "74LS04" H 6750 6476 50  0001 C CNN
+F 2 "Housings_SOIC:SOIC-14_3.9x8.7mm_Pitch1.27mm" H 6750 6250 50  0001 C CNN
+F 3 "http://www.ti.com/lit/gpn/sn74LS04" H 6750 6250 50  0001 C CNN
+	6    6750 6250
+	1    0    0    -1
+$EndComp
+$Comp
+L power:GND #PWR0144
+U 1 1 61D82314
+P 6200 6500
+F 0 "#PWR0144" H 6200 6250 50  0001 C CNN
+F 1 "GND" H 6205 6327 50  0000 C CNN
+F 2 "" H 6200 6500 50  0001 C CNN
+F 3 "" H 6200 6500 50  0001 C CNN
+	1    6200 6500
+	1    0    0    -1
+$EndComp
+Wire Wire Line
+	6200 6500 6200 6250
+Wire Wire Line
+	6200 4650 6450 4650
+Wire Wire Line
+	6450 5050 6200 5050
+Connection ~ 6200 5050
+Wire Wire Line
+	6200 5050 6200 4650
+Wire Wire Line
+	6450 5450 6200 5450
+Connection ~ 6200 5450
+Wire Wire Line
+	6200 5450 6200 5050
+Wire Wire Line
+	6450 5850 6200 5850
+Connection ~ 6200 5850
+Wire Wire Line
+	6200 5850 6200 5450
+Wire Wire Line
+	6450 6250 6200 6250
+Connection ~ 6200 6250
+Wire Wire Line
+	6200 6250 6200 5850
+NoConn ~ 7050 4650
+NoConn ~ 7050 5050
+NoConn ~ 7050 5450
+NoConn ~ 7050 5850
+NoConn ~ 7050 6250
 $EndSCHEMATC

Commit message: BOM update
Parts:
- C2, C20, C22, C24, C27, C29: DigiKey (none) -> 1276-1099-1-ND
- U17: DigiKey (none) -> 296-1630-1-ND
- U20, U22: DigiKey (none) -> 296-14899-1-ND
- U20, U22: DigiKey SN74LS74ADR‎ -> 296-14899-1-ND
- X1: DigiKey (none) -> 535-9170-5-ND
Changed lines of the file:
@@
 F 2 "Capacitors_SMD:C_0805_HandSoldering" H 10213 1550 50  0001 C CNN
 F 3 "~" H 10175 1700 50  0001 C CNN
+F 4 "1276-1099-1-ND" H 10175 1700 50  0001 C CNN "DigiKey"
 	1    10175 1700
 	1    0    0    1
@@
 F 2 "Capacitors_SMD:C_0805_HandSoldering" H 9963 2925 50  0001 C CNN
 F 3 "~" H 9925 3075 50  0001 C CNN
+F 4 "1276-1099-1-ND" H 9925 3075 50  0001 C CNN "DigiKey"
 	1    9925 3075
 	1    0    0    -1
@@
 F 2 "Housings_SOIC:SOIC-14_3.9x8.7mm_Pitch1.27mm" H 10475 5500 50  0001 C CNN
 F 3 "74xx/74hc_hct74.pdf" H 10475 5500 50  0001 C CNN
+F 4 "296-14899-1-ND" H 10475 5500 50  0001 C CNN "DigiKey"
 	3    10475 5500
 	1    0    0    -1
@@
 F 2 "Capacitors_SMD:C_0805_HandSoldering" H 9988 5325 50  0001 C CNN
 F 3 "~" H 9950 5475 50  0001 C CNN
+F 4 "1276-1099-1-ND" H 9950 5475 50  0001 C CNN "DigiKey"
 	1    9950 5475
 	1    0    0    -1
@@
 F 2 "Housings_SOIC:SOIC-14_3.9x8.7mm_Pitch1.27mm" H 5025 5000 50  0001 C CNN
 F 3 "74xx/74hc_hct74.pdf" H 5025 5000 50  0001 C CNN
-F 4 "SN74LS74ADR‎" H 5025 5000 50  0001 C CNN "DigiKey"
+F 4 "296-14899-1-ND" H 5025 5000 50  0001 C CNN "DigiKey"
 	2    5025 5000
 	1    0    0    -1
@@
 F 2 "Housings_SOIC:SOIC-14_3.9x8.7mm_Pitch1.27mm" H 3750 4425 50  0001 C CNN
 F 3 "74xx/74hc_hct74.pdf" H 3750 4425 50  0001 C CNN
-F 4 "SN74LS74ADR‎" H 3750 4425 50  0001 C CNN "DigiKey"
+F 4 "296-14899-1-ND" H 3750 4425 50  0001 C CNN "DigiKey"
 	1    3750 4425
 	1    0    0    -1
@@
 F 2 "Housings_SOIC:SOIC-14_3.9x8.7mm_Pitch1.27mm" H 10225 4300 50  0001 C CNN
 F 3 "74xx/74hc_hct74.pdf" H 10225 4300 50  0001 C CNN
+F 4 "296-14899-1-ND" H 10225 4300 50  0001 C CNN "DigiKey"
 	3    10225 4300
 	1    0    0    -1
@@
 F 2 "Capacitors_SMD:C_0805_HandSoldering" H 9663 4150 50  0001 C CNN
 F 3 "~" H 9625 4300 50  0001 C CNN
+F 4 "1276-1099-1-ND" H 9625 4300 50  0001 C CNN "DigiKey"
 	1    9625 4300
 	1    0    0    -1
@@
 F 2 "Oscillators:Oscillator_DIP-8_LargePads" H 2725 4075 50  0001 C CNN
 F 3 "https://www.digikey.ca/product-detail/en/abracon-llc/ACH-14.31818MHZ-EK/535-9170-5-ND/675365" H 2175 4425 50  0001 C CNN
+F 4 "535-9170-5-ND" H 2275 4425 50  0001 C CNN "DigiKey"
 	1    2275 4425
 	1    0    0    -1
@@
 F 2 "Capacitors_SMD:C_0805_HandSoldering" H 2013 3675 50  0001 C CNN
 F 3 "~" H 1975 3825 50  0001 C CNN
+F 4 "1276-1099-1-ND" H 1975 3825 50  0001 C CNN "DigiKey"
 	1    1975 3825
 	0    1    1    0
@@
 F 2 "Housings_SOIC:SOIC-14_3.9x8.7mm_Pitch1.27mm" H 7350 2775 50  0001 C CNN
 F 3 "74xx/74hc_hct74.pdf" H 7350 2775 50  0001 C CNN
+F 4 "296-14899-1-ND" H 7350 2775 50  0001 C CNN "DigiKey"
 	1    7350 2775
 	-1   0    0    1
@@
 F 2 "Capacitors_SMD:C_0805_HandSoldering" H 9213 1000 50  0001 C CNN
 F 3 "~" H 9175 1150 50  0001 C CNN
+F 4 "1276-1099-1-ND" H 9175 1150 50  0001 C CNN "DigiKey"
 	1    9175 1150
 	1    0    0    1
@@
 F 2 "" H 8000 3550 50  0001 C CNN
 F 3 "http://www.ti.com/lit/gpn/sn74LS05" H 8000 3550 50  0001 C CNN
+F 4 "296-1630-1-ND" H 8000 3550 50  0001 C CNN "DigiKey"
 	6    8000 3550
 	1    0    0    -1
@@
 F 2 "" H 8050 4650 50  0001 C CNN
 F 3 "http://www.ti.com/lit/gpn/sn74LS05" H 8050 4650 50  0001 C CNN
+F 4 "296-1630-1-ND" H 8050 4650 50  0001 C CNN "DigiKey"
 	2    8050 4650
 	1    0    0    -1
@@
 F 2 "" H 8050 5050 50  0001 C CNN
 F 3 "http://www.ti.com/lit/gpn/sn74LS05" H 8050 5050 50  0001 C CNN
+F 4 "296-1630-1-ND" H 8050 5050 50  0001 C CNN "DigiKey"
 	3    8050 5050
 	1    0    0    -1
@@
 F 2 "" H 8050 5450 50  0001 C CNN
 F 3 "http://www.ti.com/lit/gpn/sn74LS05" H 8050 5450 50  0001 C CNN
+F 4 "296-1630-1-ND" H 8050 5450 50  0001 C CNN "DigiKey"
 	4    8050 5450
 	1    0    0    -1
@@
 F 2 "" H 8050 5850 50  0001 C CNN
 F 3 "http://www.ti.com/lit/gpn/sn74LS05" H 8050 5850 50  0001 C CNN
+F 4 "296-1630-1-ND" H 8050 5850 50  0001 C CNN "DigiKey"
 	5    8050 5850
 	1    0    0    -1

Commit message: DigiKey BOM complete
Parts:
- C12: DigiKey (none) -> 493-1037-ND
- C14, C28: DigiKey (none) -> 1276-1298-1-ND
- C21: DigiKey (none) -> 1276-2926-1-ND
- D1: DigiKey (none) -> 1497-1022-ND
- F2: DigiKey (none) -> F3171CT-ND
- R12: DigiKey (none) -> RMCF0805JT330RCT-ND
- R13: DigiKey (none) -> RMCF0805JT10K0CT-ND
- R16: DigiKey (none) -> RMCF0805JT91K0CT-ND
- R17: DigiKey (none) -> RMCF0805JT1M00CT-ND
- R18, R21, R28: DigiKey (none) -> RMCF0805FT1K00CT-ND
- R19: DigiKey (none) -> RMCF0805JT3K30CT-ND
- R20: DigiKey (none) -> RMCF0805JT22K0CT-ND
- R7: DigiKey (none) -> RMCF0805JT150RCT-ND
- SW1: DigiKey (none) -> 401-1132-ND
- SW2: DigiKey (none) -> 679-2428-ND
- U11: value 74LS04 -> 74HCT04; DigiKey 296-14875-1-ND‎ -> 296-31832-1-ND
- U11: value 74LS04 -> 74HCT04; DigiKey (none) -> 296-31832-1-ND
- U14: DigiKey (none) -> 296-14874-1-ND
- U2: DigiKey (none) -> ICL7660CSA+TCT-ND
Changed lines of the file:
@@
 F 2 "Capacitors_ThroughHole:CP_Radial_D5.0mm_P2.50mm" H 1988 1475 50  0001 C CNN
 F 3 "~" H 1950 1625 50  0001 C CNN
+F 4 "493-1037-ND" H 1950 1625 50  0001 C CNN "DigiKey"
 	1    1950 1625
 	-1   0    0    -1
@@
 F 2 "LeakyChips:PVA1_Switch" H 2500 2575 50  0001 C CNN
 F 3 "https://www.digikey.ca/product-detail/en/Y17P11141FP/CKN10276-ND/2296958/?itemSeq=317120675" H 2500 2575 50  0001 C CNN
+F 4 "401-1132-ND" H 2500 2375 50  0001 C CNN "DigiKey"
 	1    2500 2375
 	1    0    0    -1
@@
 F 2 "Resistors_SMD:R_0805_HandSoldering" H 3050 2375 50  0001 C CNN
 F 3 "~" H 3050 2375 50  0001 C CNN
+F 4 "RMCF0805JT330RCT-ND" H 3050 2375 50  0001 C CNN "DigiKey"
 	1    3050 2375
 	0    1    1    0
@@
 F 2 "Resistors_SMD:R_0805_HandSoldering" H 4275 1175 50  0001 C CNN
 F 3 "~" H 4275 1175 50  0001 C CNN
+F 4 "RMCF0805JT150RCT-ND" H 4275 1175 50  0001 C CNN "DigiKey"
 	1    4275 1175
 	-1   0    0    1
@@
 F 2 "LEDs:LED_D3.0mm" H 4275 1475 50  0001 C CNN
 F 3 "~" H 4275 1475 50  0001 C CNN
+F 4 "1497-1022-ND" H 4275 1475 50  0001 C CNN "DigiKey"
 	1    4275 1475
 	0    -1   -1   0
@@
 F 2 "Resistors_SMD:R_0805_HandSoldering" H 2850 2700 50  0001 C CNN
 F 3 "~" H 2850 2700 50  0001 C CNN
+F 4 "RMCF0805JT10K0CT-ND" H 2850 2700 50  0001 C CNN "DigiKey"
 	1    2850 2700
 	1    0    0    -1
@@
 F 2 "Housings_SOIC:SOIC-14_3.9x8.7mm_Pitch1.27mm" H 10475 1725 50  0001 C CNN
 F 3 "http://www.ti.com/lit/gpn/sn74ls02" H 10475 1725 50  0001 C CNN
+F 4 "296-14874-1-ND" H 10475 1725 50  0001 C CNN "DigiKey"
 	5    10475 1725
 	1    0    0    -1
@@
 F 2 "Buttons_Switches_ThroughHole:SW_PUSH_6mm" H 1225 6975 50  0001 C CNN
 F 3 "~" H 1225 6975 50  0001 C CNN
+F 4 "679-2428-ND" H 1225 6775 50  0001 C CNN "DigiKey"
 	1    1225 6775
 	1    0    0    -1
@@
 F 2 "Capacitors_SMD:C_0805_HandSoldering" H 1563 6975 50  0001 C CNN
 F 3 "~" H 1525 7125 50  0001 C CNN
+F 4 "1276-2926-1-ND" H 1525 7125 50  0001 C CNN "DigiKey"
 	1    1525 7125
 	1    0    0    -1
@@
 F 2 "Resistors_SMD:R_0805_HandSoldering" H 1875 7125 50  0001 C CNN
 F 3 "~" H 1875 7125 50  0001 C CNN
+F 4 "RMCF0805JT1M00CT-ND" H 1875 7125 50  0001 C CNN "DigiKey"
 	1    1875 7125
 	1    0    0    -1
@@
 F 2 "Resistors_SMD:R_0805_HandSoldering" H 1875 6450 50  0001 C CNN
 F 3 "~" H 1875 6450 50  0001 C CNN
+F 4 "RMCF0805JT91K0CT-ND" H 1875 6450 50  0001 C CNN "DigiKey"
 	1    1875 6450
 	1    0    0    -1
@@
 F 2 "Resistors_SMD:R_0805_HandSoldering" H 2200 6775 50  0001 C CNN
 F 3 "~" H 2200 6775 50  0001 C CNN
+F 4 "RMCF0805FT1K00CT-ND" H 2200 6775 50  0001 C CNN "DigiKey"
 	1    2200 6775
 	0    1    1    0
@@
 F 2 "Resistors_SMD:R_0805_HandSoldering" H 3600 6500 50  0001 C CNN
 F 3 "~" H 3600 6500 50  0001 C CNN
+F 4 "RMCF0805JT3K30CT-ND" H 3600 6500 50  0001 C CNN "DigiKey"
 	1    3600 6500
 	1    0    0    -1
@@
 F 2 "Resistors_SMD:R_0805_HandSoldering" H 4325 6775 50  0001 C CNN
 F 3 "~" H 4325 6775 50  0001 C CNN
+F 4 "RMCF0805JT22K0CT-ND" H 4325 6775 50  0001 C CNN "DigiKey"
 	1    4325 6775
 	0    1    1    0
@@
 F 2 "Resistors_SMD:R_0805_HandSoldering" H 4725 6500 50  0001 C CNN
 F 3 "~" H 4725 6500 50  0001 C CNN
+F 4 "RMCF0805FT1K00CT-ND" H 4725 6500 50  0001 C CNN "DigiKey"
 	1    4725 6500
 	1    0    0    -1
@@
 P 6600 2400
 F 0 "U11" H 6600 2717 50  0000 C CNN
-F 1 "74LS04" H 6600 2626 50  0000 C CNN
+F 1 "74HCT04" H 6600 2626 50  0000 C CNN
 F 2 "Housings_SOIC:SOIC-14_3.9x8.7mm_Pitch1.27mm" H 6600 2400 50  0001 C CNN
 F 3 "http://www.ti.com/lit/gpn/sn74LS04" H 6600 2400 50  0001 C CNN
-F 4 "296-14875-1-ND‎" H 6600 2400 50  0001 C CNN "DigiKey"
+F 4 "296-31832-1-ND" H 6600 2400 50  0001 C CNN "DigiKey"
 	3    6600 2400
 	1    0    0    -1
@@
 F 2 "Resistors_SMD:R_0805_HandSoldering" H 8150 3125 50  0001 C CNN
 F 3 "~" H 8150 3125 50  0001 C CNN
+F 4 "RMCF0805FT1K00CT-ND" H 8150 3125 50  0001 C CNN "DigiKey"
 	1    8150 3125
 	0    1    1    0
@@
 P 9575 1150
 F 0 "U11" H 9805 1196 50  0000 L CNN
-F 1 "74LS04" H 9805 1105 50  0000 L CNN
+F 1 "74HCT04" H 9805 1105 50  0000 L CNN
 F 2 "Housings_SOIC:SOIC-14_3.9x8.7mm_Pitch1.27mm" H 9575 1150 50  0001 C CNN
 F 3 "http://www.ti.com/lit/gpn/sn74LS04" H 9575 1150 50  0001 C CNN
+F 4 "296-31832-1-ND" H 9575 1150 50  0001 C CNN "DigiKey"
 	7    9575 1150
 	1    0    0    -1
@@
 F 2 "Package_SO:SOIC-8_3.9x4.9mm_P1.27mm" H 6775 1250 50  0001 C CNN
 F 3 "http://datasheets.maximintegrated.com/en/ds/ICL7660-MAX1044.pdf" H 6775 1250 50  0001 C CNN
+F 4 "ICL7660CSA+TCT-ND" H 6675 1350 50  0001 C CNN "DigiKey"
 	1    6675 1350
 	1    0    0    -1
@@
 F 2 "Capacitor_SMD:C_0805_2012Metric_Pad1.15x1.40mm_HandSolder" H 7250 1450 50  0001 C CNN
 F 3 "~" H 7250 1450 50  0001 C CNN
+F 4 "1276-1298-1-ND" H 7250 1450 50  0001 C CNN "DigiKey"
 	1    7250 1450
 	1    0    0    -1
@@
 F 2 "Capacitor_SMD:C_0805_2012Metric_Pad1.15x1.40mm_HandSolder" H 8075 1300 50  0001 C CNN
 F 3 "~" H 8075 1300 50  0001 C CNN
+F 4 "1276-1298-1-ND" H 8075 1300 50  0001 C CNN "DigiKey"
 	1    8075 1300
 	1    0    0    -1
@@
 F 2 "0251002.MRT1L:0251002.MRT1L" H 1475 1475 50  0001 C CNN
 F 3 "https://www.digikey.ca/product-detail/en/littelfuse-inc/0251002.MRT1L/F3171CT-ND/1984467" H 1475 1475 50  0001 C CNN
+F 4 "F3171CT-ND" H 1475 1475 50  0001 C CNN "DigiKey"
 	1    1475 1475
 	1    0    0    1
@@
 P 6750 4650
 F 0 "U11" H 6750 4967 50  0000 C CNN
-F 1 "74LS04" H 6750 4876 50  0000 C CNN
+F 1 "74HCT04" H 6750 4876 50  0000 C CNN
 F 2 "Housings_SOIC:SOIC-14_3.9x8.7mm_Pitch1.27mm" H 6750 4650 50  0001 C CNN
 F 3 "http://www.ti.com/lit/gpn/sn74LS04" H 6750 4650 50  0001 C CNN
+F 4 "296-31832-1-ND" H 6750 4650 50  0001 C CNN "DigiKey"
 	1    6750 4650
 	1    0    0    -1
@@
 P 6750 5050
 F 0 "U11" H 6750 5275 50  0000 C CNN
-F 1 "74LS04" H 6750 5276 50  0001 C CNN
+F 1 "74HCT04" H 6750 5276 50  0001 C CNN
 F 2 "Housings_SOIC:SOIC-14_3.9x8.7mm_Pitch1.27mm" H 6750 5050 50  0001 C CNN
 F 3 "http://www.ti.com/lit/gpn/sn74LS04" H 6750 5050 50  0001 C CNN
+F 4 "296-31832-1-ND" H 6750 5050 50  0001 C CNN "DigiKey"
 	2    6750 5050
 	1    0    0    -1
@@
 P 6750 5450
 F 0 "U11" H 6750 5675 50  0000 C CNN
-F 1 "74LS04" H 6750 5676 50  0001 C CNN
+F 1 "74HCT04" H 6750 5676 50  0001 C CNN
 F 2 "Housings_SOIC:SOIC-14_3.9x8.7mm_Pitch1.27mm" H 6750 5450 50  0001 C CNN
 F 3 "http://www.ti.com/lit/gpn/sn74LS04" H 6750 5450 50  0001 C CNN
+F 4 "296-31832-1-ND" H 6750 5450 50  0001 C CNN "DigiKey"
 	4    6750 5450
 	1    0    0    -1
@@
 P 6750 5850
 F 0 "U11" H 6750 6075 50  0000 C CNN
-F 1 "74LS04" H 6750 6076 50  0001 C CNN
+F 1 "74HCT04" H 6750 6076 50  0001 C CNN
 F 2 "Housings_SOIC:SOIC-14_3.9x8.7mm_Pitch1.27mm" H 6750 5850 50  0001 C CNN
 F 3 "http://www.ti.com/lit/gpn/sn74LS04" H 6750 5850 50  0001 C CNN
+F 4 "296-31832-1-ND" H 6750 5850 50  0001 C CNN "DigiKey"
 	5    6750 5850
 	1    0    0    -1
@@
 P 6750 6250
 F 0 "U11" H 6750 6475 50  0000 C CNN
-F 1 "74LS04" H 6750 6476 50  0001 C CNN
+F 1 "74HCT04" H 6750 6476 50  0001 C CNN
 F 2 "Housings_SOIC:SOIC-14_3.9x8.7mm_Pitch1.27mm" H 6750 6250 50  0001 C CNN
 F 3 "http://www.ti.com/lit/gpn/sn74LS04" H 6750 6250 50  0001 C CNN
+F 4 "296-31832-1-ND" H 6750 6250 50  0001 C CNN "DigiKey"
 	6    6750 6250
 	1    0    0    -1

Commit message: CSV BOM exporter
Parts:
- J3: DigiKey ED2983-ND -> ED2982-ND
Changed lines of the file:
@@
 F 3 "" H 1025 1575 50  0001 L BNN
 F 4 "ON-SHORE TECHNOLOGY" H 1025 1575 50  0001 L BNN "MANUFACTURER"
-F 5 "ED2983-ND" H 1025 1575 50  0001 C CNN "DigiKey"
+F 5 "ED2982-ND" H 1025 1575 50  0001 C CNN "DigiKey"
 	1    1025 1575
 	-1   0    0    -1

Commit message: Change to more available power FET
Parts:
- Q2: DigiKey DMN6075S-7DICT-ND -> DMN2046U-7DICT-ND
Changed lines of the file:
@@
 F 2 "TO_SOT_Packages_SMD:SOT-23_Handsoldering" H 3650 2475 50  0001 C CNN
 F 3 "https://www.digikey.ca/product-detail/en/diodes-incorporated/DMN6075S-7/DMN6075S-7DICT-ND/5149299" H 3450 2375 50  0001 C CNN
-F 4 "DMN6075S-7DICT-ND" H 3450 2375 50  0001 C CNN "DigiKey"
+F 4 "DMN2046U-7DICT-ND" H 3450 2375 50  0001 C CNN "DigiKey"
 	1    3450 2375
 	1    0    0    -1

Commit message: Replace 1k with 1.5k across the board to reduce BOM
Parts:
- R18, R21, R28: value 1kΩ -> 1.5kΩ
Changed lines of the file:
@@
 P 2200 6775
 F 0 "R18" V 1995 6775 50  0000 C CNN
-F 1 "1kΩ" V 2086 6775 50  0000 C CNN
+F 1 "1.5kΩ" V 2086 6775 50  0000 C CNN
 F 2 "Resistors_SMD:R_0805_HandSoldering" H 2200 6775 50  0001 C CNN
 F 3 "~" H 2200 6775 50  0001 C CNN
@@
 P 4725 6500
 F 0 "R21" H 4793 6546 50  0000 L CNN
-F 1 "1kΩ" H 4793 6455 50  0000 L CNN
+F 1 "1.5kΩ" H 4793 6455 50  0000 L CNN
 F 2 "Resistors_SMD:R_0805_HandSoldering" H 4725 6500 50  0001 C CNN
 F 3 "~" H 4725 6500 50  0001 C CNN
@@
 P 8150 3125
 F 0 "R28" V 7945 3125 50  0000 C CNN
-F 1 "1kΩ" V 8036 3125 50  0000 C CNN
+F 1 "1.5kΩ" V 8036 3125 50  0000 C CNN
 F 2 "Resistors_SMD:R_0805_HandSoldering" H 8150 3125 50  0001 C CNN
 F 3 "~" H 8150 3125 50  0001 C CNN
