File: Controllers.sch (KiCad schematic (older format))
At the start: 4 parts

Commit message: Swap tip and ring for composite, finish up power
Parts:
- U15, U16: renamed from U?; footprint (none) -> Housings_SSOP:TSSOP-20_4.4x6.5mm_Pitch0.65mm
- gave numbers to parts that had none: 2
Changed lines of the file:
@@
 $EndDescr
 $Comp
-L Connector:DB9_Male J?
+L Connector:DB9_Male J5
 U 1 1 5E4296AD
 P 3675 3000
-F 0 "J?" H 3855 3046 50  0000 L CNN
+F 0 "J5" H 3855 3046 50  0000 L CNN
 F 1 "Controller Port 1" H 3855 2955 50  0000 L CNN
 F 2 "" H 3675 3000 50  0001 C CNN
@@
 $EndComp
 $Comp
-L Connector:DB9_Male J?
+L Connector:DB9_Male J6
 U 1 1 5E429B8A
 P 3675 5050
-F 0 "J?" H 3855 5096 50  0000 L CNN
+F 0 "J6" H 3855 5096 50  0000 L CNN
 F 1 "Controller Port 2" H 3855 5005 50  0000 L CNN
 F 2 "" H 3675 5050 50  0001 C CNN
@@
 Common
 $Comp
-L 74xx_IEEE:74LS541 U?
+L 74xx_IEEE:74LS541 U15
 U 1 1 5E42D33F
 P 6450 2825
-F 0 "U?" H 6450 3691 50  0000 C CNN
+F 0 "U15" H 6450 3691 50  0000 C CNN
 F 1 "74LS541" H 6450 3600 50  0000 C CNN
-F 2 "" H 6450 2825 50  0001 C CNN
+F 2 "Housings_SSOP:TSSOP-20_4.4x6.5mm_Pitch0.65mm" H 6450 2825 50  0001 C CNN
 F 3 "" H 6450 2825 50  0001 C CNN
 	1    6450 2825
@@
 $EndComp
 $Comp
-L 74xx_IEEE:74LS541 U?
+L 74xx_IEEE:74LS541 U16
 U 1 1 5E42EB2C
 P 6450 5150
-F 0 "U?" H 6450 6016 50  0000 C CNN
+F 0 "U16" H 6450 6016 50  0000 C CNN
 F 1 "74LS541" H 6450 5925 50  0000 C CNN
-F 2 "" H 6450 5150 50  0001 C CNN
+F 2 "Housings_SSOP:TSSOP-20_4.4x6.5mm_Pitch0.65mm" H 6450 5150 50  0001 C CNN
 F 3 "" H 6450 5150 50  0001 C CNN
 	1    6450 5150

Commit message: Controller ports
Parts:
- J5, J6: footprint (none) -> Connector_Dsub:DSUB-9_Male_Horizontal_P2.77x2.84mm_EdgePinOffset4.94mm_Housed_MountingHolesOffset7.48mm
Changed lines of the file:
@@
 F 0 "J5" H 3855 3046 50  0000 L CNN
 F 1 "Controller Port 1" H 3855 2955 50  0000 L CNN
-F 2 "" H 3675 3000 50  0001 C CNN
-F 3 " ~" H 3675 3000 50  0001 C CNN
+F 2 "Connector_Dsub:DSUB-9_Male_Horizontal_P2.77x2.84mm_EdgePinOffset4.94mm_Housed_MountingHolesOffset7.48mm" H 3675 3000 50  0001 C CNN
+F 3 "https://www.digikey.com/product-detail/en/te-connectivity-amp-connectors/5747250-4/A32072-ND/808627" H 3675 3000 50  0001 C CNN
 	1    3675 3000
 	1    0    0    -1
@@
 F 0 "J6" H 3855 5096 50  0000 L CNN
 F 1 "Controller Port 2" H 3855 5005 50  0000 L CNN
-F 2 "" H 3675 5050 50  0001 C CNN
-F 3 " ~" H 3675 5050 50  0001 C CNN
+F 2 "Connector_Dsub:DSUB-9_Male_Horizontal_P2.77x2.84mm_EdgePinOffset4.94mm_Housed_MountingHolesOffset7.48mm" H 3675 5050 50  0001 C CNN
+F 3 "https://www.digikey.com/product-detail/en/te-connectivity-amp-connectors/5747250-4/A32072-ND/808627 ~" H 3675 5050 50  0001 C CNN
 	1    3675 5050
 	1    0    0    -1

Commit message: More messing with controllers
Parts:
- added R14: 3.3kΩ, Resistors_SMD:R_0805_HandSoldering, symbol Device:R_Small_US
- added U17: 74LS05, Housings_SOIC:SOIC-14_3.9x8.7mm_Pitch1.27mm, symbol 74xx:74LS05
- U15: value 74LS541 -> Controller 1; footprint Housings_SSOP:TSSOP-20_4.4x6.5mm_Pitch0.65mm -> Housings_SOIC:SOIC-20W_7.5x12.8mm_Pitch1.27mm
- U16: value 74LS541 -> Controller 2; footprint Housings_SSOP:TSSOP-20_4.4x6.5mm_Pitch0.65mm -> Housings_SOIC:SOIC-20W_7.5x12.8mm_Pitch1.27mm
Connections:
- net labels added: A1, D0, D1, D2, D3, D4, D5, D6, D7, VCC
- wire segments 4 -> 12
Changed lines of the file:
@@
 F 3 "https://www.digikey.com/product-detail/en/te-connectivity-amp-connectors/5747250-4/A32072-ND/808627" H 3675 3000 50  0001 C CNN
 	1    3675 3000
-	1    0    0    -1
+	-1   0    0    1
 $EndComp
 $Comp
@@
 F 3 "https://www.digikey.com/product-detail/en/te-connectivity-amp-connectors/5747250-4/A32072-ND/808627 ~" H 3675 5050 50  0001 C CNN
 	1    3675 5050
-	1    0    0    -1
+	-1   0    0    1
 $EndComp
-Text Label 3375 2600 2    50   ~ 0
-Select
-Text Label 3375 2900 2    50   ~ 0
-Common
 $Comp
 L 74xx_IEEE:74LS541 U15
@@
 P 6450 2825
 F 0 "U15" H 6450 3691 50  0000 C CNN
-F 1 "74LS541" H 6450 3600 50  0000 C CNN
-F 2 "Housings_SSOP:TSSOP-20_4.4x6.5mm_Pitch0.65mm" H 6450 2825 50  0001 C CNN
-F 3 "" H 6450 2825 50  0001 C CNN
+F 1 "Controller 1" H 6450 3600 50  0000 C CNN
+F 2 "Housings_SOIC:SOIC-20W_7.5x12.8mm_Pitch1.27mm" H 6450 2825 50  0001 C CNN
+F 3 "https://www.digikey.ca/product-detail/en/SN74HCT541DWR/296-14870-1-ND/562554/?itemSeq=317132221" H 6450 2825 50  0001 C CNN
 	1    6450 2825
 	1    0    0    -1
@@
 P 6450 5150
 F 0 "U16" H 6450 6016 50  0000 C CNN
-F 1 "74LS541" H 6450 5925 50  0000 C CNN
-F 2 "Housings_SSOP:TSSOP-20_4.4x6.5mm_Pitch0.65mm" H 6450 5150 50  0001 C CNN
-F 3 "" H 6450 5150 50  0001 C CNN
+F 1 "Controller 2" H 6450 5925 50  0000 C CNN
+F 2 "Housings_SOIC:SOIC-20W_7.5x12.8mm_Pitch1.27mm" H 6450 5150 50  0001 C CNN
+F 3 "https://www.digikey.ca/product-detail/en/SN74HCT541DWR/296-14870-1-ND/562554/?itemSeq=317132221" H 6450 5150 50  0001 C CNN
 	1    6450 5150
 	1    0    0    -1
@@
 Text Notes 5175 3950 1    50   ~ 0
 TODO: everything else
+Text Label 3975 3400 0    50   ~ 0
+Select
+Text Label 3975 3100 0    50   ~ 0
+Common
+Text GLabel 3825 4425 0    50   Input ~ 0
+A1
+Wire Wire Line
+	3825 4425 5450 4425
+Wire Wire Line
+	5450 4425 5450 4700
+Wire Wire Line
+	5450 4700 5900 4700
+Text GLabel 3825 1675 1    50   Input ~ 0
+A1
+Wire Wire Line
+	3825 1675 3825 1775
+Wire Wire Line
+	4425 1775 4650 1775
+Wire Wire Line
+	5400 1775 5400 2375
+Wire Wire Line
+	5400 2375 5900 2375
+$Comp
+L Device:R_Small_US R14
+U 1 1 5E4048A8
+P 4650 1675
+F 0 "R14" H 4718 1721 50  0000 L CNN
+F 1 "3.3kΩ" H 4718 1630 50  0000 L CNN
+F 2 "Resistors_SMD:R_0805_HandSoldering" H 4650 1675 50  0001 C CNN
+F 3 "~" H 4650 1675 50  0001 C CNN
+	1    4650 1675
+	1    0    0    -1
+$EndComp
+Connection ~ 4650 1775
+Wire Wire Line
+	4650 1775 5400 1775
+$Comp
+L power:VCC #PWR0115
+U 1 1 5E40500D
+P 4650 1575
+F 0 "#PWR0115" H 4650 1425 50  0001 C CNN
+F 1 "VCC" H 4667 1748 50  0000 C CNN
+F 2 "" H 4650 1575 50  0001 C CNN
+F 3 "" H 4650 1575 50  0001 C CNN
+	1    4650 1575
+	1    0    0    -1
+$EndComp
+Text GLabel 7000 2575 2    50   Input ~ 0
+D7
+Text GLabel 7000 3275 2    50   Input ~ 0
+D0
+Text GLabel 7000 3175 2    50   Input ~ 0
+D1
+Text GLabel 7000 3075 2    50   Input ~ 0
+D2
+Text GLabel 7000 2975 2    50   Input ~ 0
+D3
+Text GLabel 7000 2875 2    50   Input ~ 0
+D4
+Text GLabel 7000 2775 2    50   Input ~ 0
+D5
+Text GLabel 7000 2675 2    50   Input ~ 0
+D6
+Text GLabel 7000 4900 2    50   Input ~ 0
+D0
+Text GLabel 7000 5000 2    50   Input ~ 0
+D1
+Text GLabel 7000 5100 2    50   Input ~ 0
+D2
+Text GLabel 7000 5200 2    50   Input ~ 0
+D3
+Text GLabel 7000 5300 2    50   Input ~ 0
+D4
+Text GLabel 7000 5400 2    50   Input ~ 0
+D5
+Text GLabel 7000 5500 2    50   Input ~ 0
+D6
+Text GLabel 7000 5600 2    50   Input ~ 0
+D7
+$Comp
+L 74xx:74LS05 U17
+U 1 1 5E402BF3
+P 4125 1775
+F 0 "U17" H 4125 2092 50  0000 C CNN
+F 1 "74LS05" H 4125 2001 50  0000 C CNN
+F 2 "Housings_SOIC:SOIC-14_3.9x8.7mm_Pitch1.27mm" H 4125 1775 50  0001 C CNN
+F 3 "https://www.digikey.ca/product-detail/en/MM74HCT05MX/MM74HCT05MXCT-ND/2094424/?itemSeq=317132076" H 4125 1775 50  0001 C CNN
+	1    4125 1775
+	1    0    0    -1
+$EndComp
 $EndSCHEMATC

Commit message: Jesus
Parts:
- added C? (x2): 0.1µF, symbol Device:C
- added C? (x2): 47nF, symbol Device:C
- added C? (x2): 100pF, symbol Device:C
- added C? (x2): 10nF, symbol Device:C
- added D? (x2): 1N4001, Diode_THT:D_DO-41_SOD81_P10.16mm_Horizontal, symbol Diode:1N4001
- added Q? (x2): 2N3904, Package_TO_SOT_THT:TO-92_Inline, symbol Transistor_BJT:2N3904
- added R? (x2): 270Ω, symbol Device:R_Small_US
- added R? (x2): 1.8kΩ, symbol Device:R_Small_US
- added R? (x2): R_Small_US, symbol Device:R_Small_US
- added R? (x2): 22k, symbol Device:R_Small_US
- added R?: 1.5kΩ, symbol Device:R_Small_US
- added R? (x2): 100kΩ, symbol Device:R_Small_US
- added RN? (x2): 22kΩ, Resistor_THT:R_Array_SIP8, symbol Device:R_Network07_US
- added U? (x3): 74HCT00, symbol 74xx:74HCT00
- added U?: 74LS05, symbol 74xx:74LS05
Connections:
- net labels added: !INT, 2v5, GND, QUAD
- wire segments 12 -> 153
Other:
- note added: "TODO: weird flip flop thing"

Commit message: All the controller stuff is on the PCB now
Parts:
- added C37, C38: 10nF, Capacitors_SMD:C_0805_HandSoldering, symbol Device:C
- added R40, R41: 1.5kΩ, Resistors_SMD:R_0805_HandSoldering, symbol Device:R_Small_US
- added R42, R43: 120Ω, Resistors_SMD:R_0805_HandSoldering, symbol Device:R_Small_US
- added unit 1 of U23
- added unit 2 of U23
- C3, C30, C31, C32, C33, C34, C35, C36: renamed from C?; footprint (none) -> Capacitors_SMD:C_0805_HandSoldering
- D3, D4: renamed from D?; footprint Diode_THT:D_DO-41_SOD81_P10.16mm_Horizontal -> Diodes_ThroughHole:D_DO-41_SOD81_P2.54mm_Vertical_AnodeUp
- Q4, Q5: renamed from Q?; footprint Package_TO_SOT_THT:TO-92_Inline -> TO_SOT_Packages_THT:TO-92_Inline_Narrow_Oval
- R23, R24: renamed from R?; value R_Small_US -> 10kΩ; footprint (none) -> Resistors_SMD:R_0805_HandSoldering
- R31, R32, R33, R34, R35, R36, R37, R38, R39: renamed from R?; footprint (none) -> Resistors_SMD:R_0805_HandSoldering
- RN1, RN2: renamed from RN?; footprint Resistor_THT:R_Array_SIP8 -> Resistors_ThroughHole:R_Array_SIP8
- U18, U23: renamed from U?; footprint (none) -> Housings_SOIC:SOIC-14_3.9x8.7mm_Pitch1.27mm
Connections:
- net labels added: -5V, CTRL_EN_1, CTRL_EN_2, CTRL_PIN_5, CTRL_PIN_8
- wire segments 153 -> 184
Other:
- note added: "80w"
- note added: "TODO: how the fuck do we get -5v"
- note added: "c0w"
- note removed: "TODO: weird flip flop thing"

Commit message: Knocking out bugs
Connections:
- net labels added: EXT_QUAD
- net labels removed: QUAD
Changed lines of the file:
@@
 Connection ~ 7825 3725
 Text GLabel 8600 3725 2    50   Input ~ 0
-QUAD
+EXT_QUAD
 $Comp
 L Device:R_Small_US R36

Commit message: Bugs patched
Connections:
- wire segments 184 -> 187
Changed lines of the file:
@@
 Text Label 2625 3950 2    50   ~ 0
 CTRL_PIN_8
+$Comp
+L power:GND #PWR0158
+U 1 1 5E49F995
+P 3425 2000
+F 0 "#PWR0158" H 3425 1750 50  0001 C CNN
+F 1 "GND" H 3430 1827 50  0000 C CNN
+F 2 "" H 3425 2000 50  0001 C CNN
+F 3 "" H 3425 2000 50  0001 C CNN
+	1    3425 2000
+	1    0    0    -1
+$EndComp
+$Comp
+L power:GND #PWR0159
+U 1 1 5E4A0B07
+P 3400 6250
+F 0 "#PWR0159" H 3400 6000 50  0001 C CNN
+F 1 "GND" H 3405 6077 50  0000 C CNN
+F 2 "" H 3400 6250 50  0001 C CNN
+F 3 "" H 3400 6250 50  0001 C CNN
+	1    3400 6250
+	1    0    0    -1
+$EndComp
+Wire Wire Line
+	3575 6375 3575 6175
+Wire Wire Line
+	3575 6175 3400 6175
+Wire Wire Line
+	3400 6175 3400 6250
 $EndSCHEMATC
