File: Controllers.sch (KiCad schematic (older format))
At the start: 39 parts, among them J5 Controller Port 1, J6 Controller Port 2, Q4 2N3904, Q5 2N3904, U15 Controller 1, U16 Controller 2, U17 74LS05, U18 74LS05, U23 74HCT00

Commit message: More chips
Other:
- note removed: "TODO: how the fuck do we get -5v"
Changed lines of the file:
@@
 	1    0    0    -1
 $EndComp
-Text Notes 9850 1800 2    50   ~ 0
-TODO: how the fuck do we get -5v
 Text Label 4375 6200 3    50   ~ 0
 2v5

Commit message: Some more chips
Parts:
- U15, U16: DigiKey (none) -> 296-14870-1-ND
Changed lines of the file:
@@
 F 2 "Housings_SOIC:SOIC-20W_7.5x12.8mm_Pitch1.27mm" H 6450 2825 50  0001 C CNN
 F 3 "https://www.digikey.ca/product-detail/en/SN74HCT541DWR/296-14870-1-ND/562554/?itemSeq=317132221" H 6450 2825 50  0001 C CNN
+F 4 "296-14870-1-ND" H 6450 2825 50  0001 C CNN "DigiKey"
 	1    6450 2825
 	1    0    0    -1
@@
 F 2 "Housings_SOIC:SOIC-20W_7.5x12.8mm_Pitch1.27mm" H 6450 5150 50  0001 C CNN
 F 3 "https://www.digikey.ca/product-detail/en/SN74HCT541DWR/296-14870-1-ND/562554/?itemSeq=317132221" H 6450 5150 50  0001 C CNN
+F 4 "296-14870-1-ND" H 6450 5150 50  0001 C CNN "DigiKey"
 	1    6450 5150
 	1    0    0    -1

Commit message: Unit fix again
Parts:
- R31, R32: value 22k -> 22kΩ
Changed lines of the file:
@@
 P 2200 1950
 F 0 "R31" V 1995 1950 50  0000 C CNN
-F 1 "22k" V 2086 1950 50  0000 C CNN
+F 1 "22kΩ" V 2086 1950 50  0000 C CNN
 F 2 "Resistors_SMD:R_0805_HandSoldering" H 2200 1950 50  0001 C CNN
 F 3 "~" H 2200 1950 50  0001 C CNN
@@
 P 2350 6425
 F 0 "R32" V 2145 6425 50  0000 C CNN
-F 1 "22k" V 2236 6425 50  0000 C CNN
+F 1 "22kΩ" V 2236 6425 50  0000 C CNN
 F 2 "Resistors_SMD:R_0805_HandSoldering" H 2350 6425 50  0001 C CNN
 F 3 "~" H 2350 6425 50  0001 C CNN

Commit message: Wide TO-92s for the controller 2n3904s
Parts:
- Q4, Q5: footprint TO_SOT_Packages_THT:TO-92_Inline_Narrow_Oval -> TO_SOT_Packages_THT:TO-92_Inline_Wide
Changed lines of the file:
@@
 F 0 "Q4" H 2041 1646 50  0000 L CNN
 F 1 "2N3904" H 2041 1555 50  0000 L CNN
-F 2 "TO_SOT_Packages_THT:TO-92_Inline_Narrow_Oval" H 2050 1525 50  0001 L CIN
+F 2 "TO_SOT_Packages_THT:TO-92_Inline_Wide" H 2050 1525 50  0001 L CIN
 F 3 "https://www.fairchildsemi.com/datasheets/2N/2N3904.pdf" H 1850 1600 50  0001 L CNN
 	1    1850 1600
@@
 F 0 "Q5" H 2191 6729 50  0000 L CNN
 F 1 "2N3904" H 2191 6820 50  0000 L CNN
-F 2 "TO_SOT_Packages_THT:TO-92_Inline_Narrow_Oval" H 2200 6700 50  0001 L CIN
+F 2 "TO_SOT_Packages_THT:TO-92_Inline_Wide" H 2200 6700 50  0001 L CIN
 F 3 "https://www.fairchildsemi.com/datasheets/2N/2N3904.pdf" H 2000 6775 50  0001 L CNN
 	1    2000 6775

Commit message: Update LS05 to 296-1630-1-ND
Parts:
- U17: DigiKey (none) -> 296-1630-1-ND
Changed lines of the file:
@@
 F 2 "Housings_SOIC:SOIC-14_3.9x8.7mm_Pitch1.27mm" H 4125 1775 50  0001 C CNN
 F 3 "https://www.digikey.ca/product-detail/en/MM74HCT05MX/MM74HCT05MXCT-ND/2094424/?itemSeq=317132076" H 4125 1775 50  0001 C CNN
+F 4 "296-1630-1-ND" H 4125 1775 50  0001 C CNN "DigiKey"
 	1    4125 1775
 	1    0    0    -1

Commit message: Fix missing junction and bump version to 0.7
Connections:
- wire segments 187 -> 189
Other:
- note removed: "TODO: everything else"
Changed lines of the file:
@@
 EESchema Schematic File Version 4
-LIBS:ColecoVision Clone-cache
 EELAYER 30 0
 EELAYER END
@@
 	5475 2025 5475 2225
 Connection ~ 5475 2225
-Text Notes 5175 3950 1    50   ~ 0
-TODO: everything else
 Text Label 2275 3275 0    50   ~ 0
 Select
@@
 	7700 3725 7825 3725
 Wire Wire Line
-	8250 3250 8250 4175
-Wire Wire Line
-	7825 3725 8600 3725
+	8250 3250 8250 3725
+Wire Wire Line
+	7825 3725 8250 3725
 Connection ~ 7825 3725
 Text GLabel 8600 3725 2    50   Input ~ 0
@@
 Wire Wire Line
 	3400 6175 3400 6250
+Connection ~ 8250 3725
+Wire Wire Line
+	8250 3725 8250 4175
+Wire Wire Line
+	8250 3725 8600 3725
 $EndSCHEMATC

Commit message: Reorganize for easier reading
Connections:
- net labels removed: Common, Select
- wire segments 189 -> 186
Changed lines of the file:
@@
 	5475 2025 5475 2225
 Connection ~ 5475 2225
-Text Label 2275 3275 0    50   ~ 0
-Select
-Text Label 2275 2975 0    50   ~ 0
-Common
 Text GLabel 3825 4425 0    50   Input ~ 0
 A1
@@
 $EndComp
 $Comp
-L power:VCC #PWR0134
-U 1 1 5E45C599
-P 2225 5925
-F 0 "#PWR0134" H 2225 5775 50  0001 C CNN
-F 1 "VCC" H 2242 6098 50  0000 C CNN
-F 2 "" H 2225 5925 50  0001 C CNN
-F 3 "" H 2225 5925 50  0001 C CNN
-	1    2225 5925
-	1    0    0    -1
-$EndComp
-$Comp
 L power:GND #PWR0135
 U 1 1 5E45CBE1
@@
 L Device:C C34
 U 1 1 5E5087E7
-P 3575 6525
-F 0 "C34" H 3461 6479 50  0000 R CNN
-F 1 "0.1µF" H 3461 6570 50  0000 R CNN
-F 2 "Capacitors_SMD:C_0805_HandSoldering" H 3613 6375 50  0001 C CNN
-F 3 "~" H 3575 6525 50  0001 C CNN
-	1    3575 6525
+P 3575 6825
+F 0 "C34" H 3875 6750 50  0000 R CNN
+F 1 "0.1µF" H 3925 6850 50  0000 R CNN
+F 2 "Capacitors_SMD:C_0805_HandSoldering" H 3613 6675 50  0001 C CNN
+F 3 "~" H 3575 6825 50  0001 C CNN
+	1    3575 6825
 	1    0    0    -1
 $EndComp
@@
 L power:GND #PWR0159
 U 1 1 5E4A0B07
-P 3400 6250
-F 0 "#PWR0159" H 3400 6000 50  0001 C CNN
-F 1 "GND" H 3405 6077 50  0000 C CNN
-F 2 "" H 3400 6250 50  0001 C CNN
-F 3 "" H 3400 6250 50  0001 C CNN
-	1    3400 6250
-	1    0    0    -1
-$EndComp
-Wire Wire Line
-	3575 6375 3575 6175
-Wire Wire Line
-	3575 6175 3400 6175
-Wire Wire Line
-	3400 6175 3400 6250
+P 3575 6975
+F 0 "#PWR0159" H 3575 6725 50  0001 C CNN
+F 1 "GND" H 3580 6802 50  0000 C CNN
+F 2 "" H 3575 6975 50  0001 C CNN
+F 3 "" H 3575 6975 50  0001 C CNN
+	1    3575 6975
+	1    0    0    -1
+$EndComp
 Connection ~ 8250 3725
 Wire Wire Line

Commit message: Base to rewire quadrature
Connections:
- wire segments 186 -> 187
Changed lines of the file:
@@
 Wire Wire Line
 	3775 6675 3575 6675
-$Comp
-L Device:C C34
-U 1 1 5E5087E7
-P 3575 6825
-F 0 "C34" H 3875 6750 50  0000 R CNN
-F 1 "0.1µF" H 3925 6850 50  0000 R CNN
-F 2 "Capacitors_SMD:C_0805_HandSoldering" H 3613 6675 50  0001 C CNN
-F 3 "~" H 3575 6825 50  0001 C CNN
-	1    3575 6825
-	1    0    0    -1
-$EndComp
 Wire Wire Line
 	3575 6675 3200 6675
@@
 Text Label 9425 5675 2    50   ~ 0
 2v5
-Text GLabel 8250 1150 0    50   Input ~ 0
-CTRL_EN_1
-Text Notes 8075 1275 2    50   ~ 0
-c0w
-Text GLabel 8250 750  0    50   Input ~ 0
-CTRL_EN_2
-Text Notes 7925 875  0    50   ~ 0
-80w
-$Comp
-L 74xx:74HCT00 U23
-U 1 1 5E65E065
-P 8775 1400
-F 0 "U23" H 8775 1725 50  0000 C CNN
-F 1 "74HCT00" H 8775 1634 50  0000 C CNN
-F 2 "Housings_SOIC:SOIC-14_3.9x8.7mm_Pitch1.27mm" H 8775 1400 50  0001 C CNN
-F 3 "http://www.ti.com/lit/gpn/sn74hct00" H 8775 1400 50  0001 C CNN
-	1    8775 1400
-	1    0    0    -1
-$EndComp
-$Comp
-L 74xx:74HCT00 U23
-U 2 1 5E6609D8
-P 8775 850
-F 0 "U23" H 8775 1175 50  0000 C CNN
-F 1 "74HCT00" H 8775 1084 50  0000 C CNN
-F 2 "Housings_SOIC:SOIC-14_3.9x8.7mm_Pitch1.27mm" H 8775 850 50  0001 C CNN
-F 3 "http://www.ti.com/lit/gpn/sn74hct00" H 8775 850 50  0001 C CNN
-	2    8775 850
-	1    0    0    -1
-$EndComp
+Text Label 1075 3950 0    50   ~ 0
+CTRL_PIN_5
+Text Label 2625 3950 2    50   ~ 0
+CTRL_PIN_8
+$Comp
+L power:GND #PWR0158
+U 1 1 5E49F995
+P 3425 2000
+F 0 "#PWR0158" H 3425 1750 50  0001 C CNN
+F 1 "GND" H 3430 1827 50  0000 C CNN
+F 2 "" H 3425 2000 50  0001 C CNN
+F 3 "" H 3425 2000 50  0001 C CNN
+	1    3425 2000
+	1    0    0    -1
+$EndComp
+Connection ~ 8250 3725
+Wire Wire Line
+	8250 3725 8250 4175
+Wire Wire Line
+	8250 3725 8600 3725
 Wire Wire Line
 	8475 950  8250 950
@@
 	8400 750  8475 750
 Wire Wire Line
-	9075 1400 9575 1400
+	9575 1200 9575 1125
+Wire Wire Line
+	9575 1125 9350 1125
+Connection ~ 9575 1125
+Wire Wire Line
+	9575 1125 9575 1050
+Wire Wire Line
+	10700 1100 10700 1175
+Wire Wire Line
+	10150 1025 10150 1100
+Wire Wire Line
+	10150 1100 10150 1175
+Connection ~ 10150 1100
+Wire Wire Line
+	10150 1100 10700 1100
+Wire Wire Line
+	9925 1400 10025 1400
+Wire Wire Line
+	10025 1475 10150 1475
+Wire Wire Line
+	9925 850  10025 850
+Wire Wire Line
+	10025 725  10150 725
+Wire Wire Line
+	10025 1400 10025 1475
+Wire Wire Line
+	10025 1475 10025 1850
+Connection ~ 10025 1475
+Wire Wire Line
+	10025 600  10525 600
+Wire Wire Line
+	10025 850  10025 725
+Wire Wire Line
+	10025 725  10025 600
+Connection ~ 10025 725
+$Comp
+L power:GND #PWR0143
+U 1 1 5E6E0C9B
+P 10700 1175
+F 0 "#PWR0143" H 10700 925 50  0001 C CNN
+F 1 "GND" H 10705 1002 50  0000 C CNN
+F 2 "" H 10700 1175 50  0001 C CNN
+F 3 "" H 10700 1175 50  0001 C CNN
+	1    10700 1175
+	1    0    0    -1
+$EndComp
+Text Label 10525 600  0    50   ~ 0
+CTRL_PIN_8
+$Comp
+L Device:C C37
+U 1 1 5E6DE0A9
+P 10150 875
+F 0 "C37" H 10265 921 50  0000 L CNN
+F 1 "10nF" H 10265 830 50  0000 L CNN
+F 2 "Capacitors_SMD:C_0805_HandSoldering" H 10188 725 50  0001 C CNN
+F 3 "~" H 10150 875 50  0001 C CNN
+	1    10150 875
+	1    0    0    -1
+$EndComp
+$Comp
+L Device:R_Small_US R42
+U 1 1 5E6ACC7E
+P 9825 850
+F 0 "R42" V 9620 850 50  0000 C CNN
+F 1 "120Ω" V 9711 850 50  0000 C CNN
+F 2 "Resistors_SMD:R_0805_HandSoldering" H 9825 850 50  0001 C CNN
+F 3 "~" H 9825 850 50  0001 C CNN
+	1    9825 850
+	0    1    1    0
+$EndComp
 Wire Wire Line
 	9575 850  9075 850
-Connection ~ 9075 1400
-Connection ~ 9075 850
+Wire Wire Line
+	9575 850  9725 850
+Connection ~ 9575 850
 $Comp
 L Device:R_Small_US R40
@@
 	1    0    0    1
 $EndComp
+Text GLabel 9350 1125 0    50   Input ~ 10
+-5V
+Text Label 10025 1850 3    50   ~ 0
+CTRL_PIN_5
+$Comp
+L Device:C C38
+U 1 1 5E6DD3B0
+P 10150 1325
+F 0 "C38" H 10265 1371 50  0000 L CNN
+F 1 "10nF" H 10265 1280 50  0000 L CNN
+F 2 "Capacitors_SMD:C_0805_HandSoldering" H 10188 1175 50  0001 C CNN
+F 3 "~" H 10150 1325 50  0001 C CNN
+	1    10150 1325
+	1    0    0    -1
+$EndComp
+$Comp
+L Device:R_Small_US R43
+U 1 1 5E6AD9B9
+P 9825 1400
+F 0 "R43" V 9620 1400 50  0000 C CNN
+F 1 "120Ω" V 9711 1400 50  0000 C CNN
+F 2 "Resistors_SMD:R_0805_HandSoldering" H 9825 1400 50  0001 C CNN
+F 3 "~" H 9825 1400 50  0001 C CNN
+	1    9825 1400
+	0    1    1    0
+$EndComp
+Wire Wire Line
+	9075 1400 9575 1400
+Wire Wire Line
+	9575 1400 9725 1400
+Connection ~ 9575 1400
 $Comp
 L Device:R_Small_US R41
@@
 	1    0    0    1
 $EndComp
-Wire Wire Line
-	9575 1200 9575 1125
-Wire Wire Line
-	9575 1125 9350 1125
-Connection ~ 9575 1125
-Wire Wire Line
-	9575 1125 9575 1050
-Text GLabel 9350 1125 0    50   Input ~ 10
--5V
-$Comp
-L Device:R_Small_US R42
-U 1 1 5E6ACC7E
-P 9825 850
-F 0 "R42" V 9620 850 50  0000 C CNN
-F 1 "120Ω" V 9711 850 50  0000 C CNN
-F 2 "Resistors_SMD:R_0805_HandSoldering" H 9825 850 50  0001 C CNN
-F 3 "~" H 9825 850 50  0001 C CNN
-	1    9825 850
-	0    1    1    0
-$EndComp
-$Comp
-L Device:R_Small_US R43
-U 1 1 5E6AD9B9
-P 9825 1400
-F 0 "R43" V 9620 1400 50  0000 C CNN
-F 1 "120Ω" V 9711 1400 50  0000 C CNN
-F 2 "Resistors_SMD:R_0805_HandSoldering" H 9825 1400 50  0001 C CNN
-F 3 "~" H 9825 1400 50  0001 C CNN
-	1    9825 1400
-	0    1    1    0
-$EndComp
-Wire Wire Line
-	9575 850  9725 850
-Connection ~ 9575 850
-Wire Wire Line
-	9575 1400 9725 1400
-Connection ~ 9575 1400
-$Comp
-L Device:C C38
-U 1 1 5E6DD3B0
-P 10150 1325
-F 0 "C38" H 10265 1371 50  0000 L CNN
-F 1 "10nF" H 10265 1280 50  0000 L CNN
-F 2 "Capacitors_SMD:C_0805_HandSoldering" H 10188 1175 50  0001 C CNN
-F 3 "~" H 10150 1325 50  0001 C CNN
-	1    10150 1325
-	1    0    0    -1
-$EndComp
-$Comp
-L Device:C C37
-U 1 1 5E6DE0A9
-P 10150 875
-F 0 "C37" H 10265 921 50  0000 L CNN
-F 1 "10nF" H 10265 830 50  0000 L CNN
-F 2 "Capacitors_SMD:C_0805_HandSoldering" H 10188 725 50  0001 C CNN
-F 3 "~" H 10150 875 50  0001 C CNN
-	1    10150 875
-	1    0    0    -1
-$EndComp
-$Comp
-L power:GND #PWR0143
-U 1 1 5E6E0C9B
-P 10700 1175
-F 0 "#PWR0143" H 10700 925 50  0001 C CNN
-F 1 "GND" H 10705 1002 50  0000 C CNN
-F 2 "" H 10700 1175 50  0001 C CNN
-F 3 "" H 10700 1175 50  0001 C CNN
-	1    10700 1175
-	1    0    0    -1
-$EndComp
-Wire Wire Line
-	10150 1025 10150 1100
-Connection ~ 10150 1100
-Wire Wire Line
-	10150 1100 10150 1175
-Wire Wire Line
-	10700 1100 10700 1175
-Wire Wire Line
-	10150 1100 10700 1100
-Wire Wire Line
-	9925 1400 10025 1400
-Wire Wire Line
-	10025 1400 10025 1475
-Wire Wire Line
-	10025 1475 10150 1475
-Wire Wire Line
-	9925 850  10025 850
-Wire Wire Line
-	10025 850  10025 725
-Wire Wire Line
-	10025 725  10150 725
-Wire Wire Line
-	10025 1475 10025 1850
-Connection ~ 10025 1475
-Wire Wire Line
-	10025 725  10025 600
-Wire Wire Line
-	10025 600  10525 600
-Connection ~ 10025 725
-Text Label 10525 600  0    50   ~ 0
-CTRL_PIN_8
-Text Label 10025 1850 3    50   ~ 0
-CTRL_PIN_5
-Text Label 1075 3950 0    50   ~ 0
-CTRL_PIN_5
-Text Label 2625 3950 2    50   ~ 0
-CTRL_PIN_8
-$Comp
-L power:GND #PWR0158
-U 1 1 5E49F995
-P 3425 2000
-F 0 "#PWR0158" H 3425 1750 50  0001 C CNN
-F 1 "GND" H 3430 1827 50  0000 C CNN
-F 2 "" H 3425 2000 50  0001 C CNN
-F 3 "" H 3425 2000 50  0001 C CNN
-	1    3425 2000
+Text Notes 7925 875  0    50   ~ 0
+80w
+Text GLabel 8250 750  0    50   Input ~ 0
+CTRL_EN_2
+Text Notes 8075 1275 2    50   ~ 0
+c0w
+Connection ~ 9075 1400
+Connection ~ 9075 850
+Text GLabel 8250 1150 0    50   Input ~ 0
+CTRL_EN_1
+$Comp
+L 74xx:74HCT00 U23
+U 1 1 5E65E065
+P 8775 1400
+F 0 "U23" H 8775 1725 50  0000 C CNN
+F 1 "74HCT00" H 8775 1634 50  0000 C CNN
+F 2 "Housings_SOIC:SOIC-14_3.9x8.7mm_Pitch1.27mm" H 8775 1400 50  0001 C CNN
+F 3 "http://www.ti.com/lit/gpn/sn74hct00" H 8775 1400 50  0001 C CNN
+	1    8775 1400
+	1    0    0    -1
+$EndComp
+$Comp
+L 74xx:74HCT00 U23
+U 2 1 5E6609D8
+P 8775 850
+F 0 "U23" H 8775 1175 50  0000 C CNN
+F 1 "74HCT00" H 8775 1084 50  0000 C CNN
+F 2 "Housings_SOIC:SOIC-14_3.9x8.7mm_Pitch1.27mm" H 8775 850 50  0001 C CNN
+F 3 "http://www.ti.com/lit/gpn/sn74hct00" H 8775 850 50  0001 C CNN
+	2    8775 850
 	1    0    0    -1
 $EndComp
@@
 L power:GND #PWR0159
 U 1 1 5E4A0B07
-P 3575 6975
-F 0 "#PWR0159" H 3575 6725 50  0001 C CNN
-F 1 "GND" H 3580 6802 50  0000 C CNN
-F 2 "" H 3575 6975 50  0001 C CNN
-F 3 "" H 3575 6975 50  0001 C CNN
-	1    3575 6975
-	1    0    0    -1
-$EndComp
-Connection ~ 8250 3725
-Wire Wire Line
-	8250 3725 8250 4175
-Wire Wire Line
-	8250 3725 8600 3725
+P 3575 7050
+F 0 "#PWR0159" H 3575 6800 50  0001 C CNN
+F 1 "GND" H 3580 6877 50  0000 C CNN
+F 2 "" H 3575 7050 50  0001 C CNN
+F 3 "" H 3575 7050 50  0001 C CNN
+	1    3575 7050
+	1    0    0    -1
+$EndComp
+Wire Wire Line
+	3575 7050 3575 6975
+$Comp
+L Device:C C34
+U 1 1 5E5087E7
+P 3575 6825
+F 0 "C34" H 3461 6779 50  0000 R CNN
+F 1 "0.1µF" H 3461 6870 50  0000 R CNN
+F 2 "Capacitors_SMD:C_0805_HandSoldering" H 3613 6675 50  0001 C CNN
+F 3 "~" H 3575 6825 50  0001 C CNN
+	1    3575 6825
+	1    0    0    -1
+$EndComp
 $EndSCHEMATC
