File: Controllers.sch (KiCad schematic (older format))
At the start: 39 parts, among them J5 Controller Port 1, J6 Controller Port 2, Q4 2N3904, Q5 2N3904, U15 Controller 1, U16 Controller 2, U17 74LS05, U18 74LS05, U23 74HCT00

Commit message: Flip controller port #s
Parts:
- J5: value Controller Port 1 -> Controller Port 2
- J6: value Controller Port 2 -> Controller Port 1
Changed lines of the file:
@@
 P 1975 2875
 F 0 "J5" H 2155 2921 50  0000 L CNN
-F 1 "Controller Port 1" H 2155 2830 50  0000 L CNN
+F 1 "Controller Port 2" H 2155 2830 50  0000 L CNN
 F 2 "Connector_Dsub:DSUB-9_Male_Horizontal_P2.77x2.84mm_EdgePinOffset4.94mm_Housed_MountingHolesOffset7.48mm" H 1975 2875 50  0001 C CNN
 F 3 "https://www.digikey.com/product-detail/en/te-connectivity-amp-connectors/5747250-4/A32072-ND/808627" H 1975 2875 50  0001 C CNN
@@
 P 1975 5225
 F 0 "J6" H 2155 5271 50  0000 L CNN
-F 1 "Controller Port 2" H 2155 5180 50  0000 L CNN
+F 1 "Controller Port 1" H 2155 5180 50  0000 L CNN
 F 2 "Connector_Dsub:DSUB-9_Male_Horizontal_P2.77x2.84mm_EdgePinOffset4.94mm_Housed_MountingHolesOffset7.48mm" H 1975 5225 50  0001 C CNN
 F 3 "https://www.digikey.com/product-detail/en/te-connectivity-amp-connectors/5747250-4/A32072-ND/808627 ~" H 1975 5225 50  0001 C CNN

Commit message: Use different 74541 symbol
Parts:
- removed U15: Controller 1, Housings_SOIC:SOIC-20W_7.5x12.8mm_Pitch1.27mm, symbol 74xx_IEEE:74LS541
- removed U16: Controller 2, Housings_SOIC:SOIC-20W_7.5x12.8mm_Pitch1.27mm, symbol 74xx_IEEE:74LS541
- added U15: 74LS541 (Ctrl. 2), Package_SO:SOIC-20W_7.5x12.8mm_P1.27mm, symbol 74xx:74LS541
- added U16: 74LS541 (Ctrl. 1), Package_SO:SOIC-20W_7.5x12.8mm_P1.27mm, symbol 74xx:74LS541
Connections:
- wire segments 187 -> 193
Changed lines of the file:
@@
 	-1   0    0    1
 $EndComp
-$Comp
-L 74xx_IEEE:74LS541 U15
-U 1 1 5E42D33F
-P 6450 2825
-F 0 "U15" H 6450 3691 50  0000 C CNN
-F 1 "Controller 1" H 6450 3600 50  0000 C CNN
-F 2 "Housings_SOIC:SOIC-20W_7.5x12.8mm_Pitch1.27mm" H 6450 2825 50  0001 C CNN
-F 3 "https://www.digikey.ca/product-detail/en/SN74HCT541DWR/296-14870-1-ND/562554/?itemSeq=317132221" H 6450 2825 50  0001 C CNN
-F 4 "296-14870-1-ND" H 6450 2825 50  0001 C CNN "DigiKey"
-	1    6450 2825
-	1    0    0    -1
-$EndComp
-$Comp
-L 74xx_IEEE:74LS541 U16
-U 1 1 5E42EB2C
-P 6450 5150
-F 0 "U16" H 6450 6016 50  0000 C CNN
-F 1 "Controller 2" H 6450 5925 50  0000 C CNN
-F 2 "Housings_SOIC:SOIC-20W_7.5x12.8mm_Pitch1.27mm" H 6450 5150 50  0001 C CNN
-F 3 "https://www.digikey.ca/product-detail/en/SN74HCT541DWR/296-14870-1-ND/562554/?itemSeq=317132221" H 6450 5150 50  0001 C CNN
-F 4 "296-14870-1-ND" H 6450 5150 50  0001 C CNN "DigiKey"
-	1    6450 5150
-	1    0    0    -1
-$EndComp
-Wire Wire Line
-	5900 2225 5475 2225
-Wire Wire Line
-	5475 2225 5475 4550
-Wire Wire Line
-	5475 4550 5900 4550
 Text GLabel 5475 2025 1    50   Input ~ 0
 CTRL_R
-Wire Wire Line
-	5475 2025 5475 2225
-Connection ~ 5475 2225
 Text GLabel 3825 4425 0    50   Input ~ 0
 A1
 Wire Wire Line
 	3825 4425 5450 4425
-Wire Wire Line
-	5450 4425 5450 4700
-Wire Wire Line
-	5450 4700 5900 4700
 Text GLabel 3825 1675 1    50   Input ~ 0
 A1
@@
 Wire Wire Line
 	4425 1775 4650 1775
-Wire Wire Line
-	5400 1775 5400 2375
-Wire Wire Line
-	5400 2375 5900 2375
 $Comp
 L Device:R_Small_US R14
@@
 	1    0    0    -1
 $EndComp
-Text GLabel 7000 2575 2    50   Input ~ 0
+Text GLabel 6900 2575 2    50   Input ~ 0
 D7
-Text GLabel 7000 3275 2    50   Input ~ 0
+Text GLabel 6900 3275 2    50   Input ~ 0
 D0
-Text GLabel 7000 3175 2    50   Input ~ 0
+Text GLabel 6900 3175 2    50   Input ~ 0
 D1
-Text GLabel 7000 3075 2    50   Input ~ 0
+Text GLabel 6900 3075 2    50   Input ~ 0
 D2
-Text GLabel 7000 2975 2    50   Input ~ 0
+Text GLabel 6900 2975 2    50   Input ~ 0
 D3
-Text GLabel 7000 2875 2    50   Input ~ 0
+Text GLabel 6900 2875 2    50   Input ~ 0
 D4
-Text GLabel 7000 2775 2    50   Input ~ 0
+Text GLabel 6900 2775 2    50   Input ~ 0
 D5
-Text GLabel 7000 2675 2    50   Input ~ 0
+Text GLabel 6900 2675 2    50   Input ~ 0
 D6
-Text GLabel 7000 4900 2    50   Input ~ 0
+Text GLabel 6900 4900 2    50   Input ~ 0
 D0
-Text GLabel 7000 5000 2    50   Input ~ 0
+Text GLabel 6900 5000 2    50   Input ~ 0
 D1
-Text GLabel 7000 5100 2    50   Input ~ 0
+Text GLabel 6900 5100 2    50   Input ~ 0
 D2
-Text GLabel 7000 5200 2    50   Input ~ 0
+Text GLabel 6900 5200 2    50   Input ~ 0
 D3
-Text GLabel 7000 5300 2    50   Input ~ 0
+Text GLabel 6900 5300 2    50   Input ~ 0
 D4
-Text GLabel 7000 5400 2    50   Input ~ 0
+Text GLabel 6900 5400 2    50   Input ~ 0
 D5
-Text GLabel 7000 5500 2    50   Input ~ 0
+Text GLabel 6900 5500 2    50   Input ~ 0
 D6
-Text GLabel 7000 5600 2    50   Input ~ 0
+Text GLabel 6900 5600 2    50   Input ~ 0
 D7
 $Comp
@@
 	1    0    0    -1
 $EndComp
+$Comp
+L 74xx:74LS541 U15
+U 1 1 6178D08C
+P 6400 3075
+F 0 "U15" H 6400 4056 50  0000 C CNN
+F 1 "74LS541 (Ctrl. 2)" H 6400 3965 50  0000 C CNN
+F 2 "Package_SO:SOIC-20W_7.5x12.8mm_P1.27mm" H 6400 3075 50  0001 C CNN
+F 3 "http://www.ti.com/lit/gpn/sn74LS541" H 6400 3075 50  0001 C CNN
+F 4 "296-14870-1-ND" H 6400 3075 50  0001 C CNN "DigiKey"
+	1    6400 3075
+	1    0    0    -1
+$EndComp
+$Comp
+L power:VCC #PWR0134
+U 1 1 6178F899
+P 7975 1975
+F 0 "#PWR0134" H 7975 1825 50  0001 C CNN
+F 1 "VCC" H 7992 2148 50  0000 C CNN
+F 2 "" H 7975 1975 50  0001 C CNN
+F 3 "" H 7975 1975 50  0001 C CNN
+	1    7975 1975
+	1    0    0    -1
+$EndComp
+Wire Wire Line
+	7975 1975 7700 1975
+Wire Wire Line
+	5475 2025 5475 3475
+Wire Wire Line
+	5900 3475 5475 3475
+Connection ~ 5475 3475
+Wire Wire Line
+	5400 3575 5900 3575
+Wire Wire Line
+	5400 1775 5400 3575
+$Comp
+L power:VCC #PWR0166
+U 1 1 617BF5B7
+P 6825 2275
+F 0 "#PWR0166" H 6825 2125 50  0001 C CNN
+F 1 "VCC" H 6842 2448 50  0000 C CNN
+F 2 "" H 6825 2275 50  0001 C CNN
+F 3 "" H 6825 2275 50  0001 C CNN
+	1    6825 2275
+	1    0    0    -1
+$EndComp
+Wire Wire Line
+	6825 2275 6400 2275
+$Comp
+L power:GND #PWR0167
+U 1 1 617C96EB
+P 6400 3875
+F 0 "#PWR0167" H 6400 3625 50  0001 C CNN
+F 1 "GND" H 6405 3702 50  0000 C CNN
+F 2 "" H 6400 3875 50  0001 C CNN
+F 3 "" H 6400 3875 50  0001 C CNN
+	1    6400 3875
+	1    0    0    -1
+$EndComp
+$Comp
+L 74xx:74LS541 U16
+U 1 1 617CC064
+P 6400 5400
+F 0 "U16" H 6400 6381 50  0000 C CNN
+F 1 "74LS541 (Ctrl. 1)" H 6400 6290 50  0000 C CNN
+F 2 "Package_SO:SOIC-20W_7.5x12.8mm_P1.27mm" H 6400 5400 50  0001 C CNN
+F 3 "http://www.ti.com/lit/gpn/sn74LS541" H 6400 5400 50  0001 C CNN
+F 4 "296-14870-1-ND" H 6400 5400 50  0001 C CNN "DigiKey"
+	1    6400 5400
+	1    0    0    -1
+$EndComp
+Wire Wire Line
+	5450 5900 5900 5900
+Wire Wire Line
+	5450 4425 5450 5900
+Wire Wire Line
+	5475 5800 5900 5800
+Wire Wire Line
+	5475 3475 5475 5800
+$Comp
+L power:GND #PWR0168
+U 1 1 617ED5C8
+P 6775 6050
+F 0 "#PWR0168" H 6775 5800 50  0001 C CNN
+F 1 "GND" H 6780 5877 50  0000 C CNN
+F 2 "" H 6775 6050 50  0001 C CNN
+F 3 "" H 6775 6050 50  0001 C CNN
+	1    6775 6050
+	1    0    0    -1
+$EndComp
+$Comp
+L power:VCC #PWR0169
+U 1 1 617F7236
+P 6825 4600
+F 0 "#PWR0169" H 6825 4450 50  0001 C CNN
+F 1 "VCC" H 6842 4773 50  0000 C CNN
+F 2 "" H 6825 4600 50  0001 C CNN
+F 3 "" H 6825 4600 50  0001 C CNN
+	1    6825 4600
+	1    0    0    -1
+$EndComp
+Wire Wire Line
+	6825 4600 6400 4600
+Wire Wire Line
+	6775 6050 6525 6050
+Wire Wire Line
+	6525 6050 6525 6200
+Wire Wire Line
+	6525 6200 6400 6200
 $EndSCHEMATC

Commit message: Remove stray vcc pin
Connections:
- wire segments 193 -> 192
Changed lines of the file:
@@
-	1    0    0    -1
-$EndComp
-$Comp
-L power:VCC #PWR0134
-U 1 1 6178F899
-P 7975 1975
-F 0 "#PWR0134" H 7975 1825 50  0001 C CNN
-F 1 "VCC" H 7992 2148 50  0000 C CNN
-F 2 "" H 7975 1975 50  0001 C CNN
-F 3 "" H 7975 1975 50  0001 C CNN
-	1    7975 1975
 	1    0    0    -1
 $EndComp
 Wire Wire Line
-	7975 1975 7700 1975
-Wire Wire Line
 	5475 2025 5475 3475

Commit message: Make the ground switching flipflop look better
Connections:
- net labels added: ~A1
- wire segments 192 -> 193
Changed lines of the file:
@@
 	8250 1500 8250 1150
-Wire Wire Line
-	9075 850  9075 1050
-Wire Wire Line
-	8475 1050 8475 1300
-Wire Wire Line
-	8475 1050 9075 1050
-Wire Wire Line
-	9075 1400 9075 1150
-Wire Wire Line
-	9075 1150 8400 1150
-Wire Wire Line
-	8400 1150 8400 750
-Wire Wire Line
-	8400 750  8475 750
 Wire Wire Line
 	9575 1200 9575 1125
@@
 Text Notes 8075 1275 2    50   ~ 0
 c0w
-Connection ~ 9075 1400
-Connection ~ 9075 850
 Text GLabel 8250 1150 0    50   Input ~ 0
 CTRL_EN_1
-$Comp
-L 74xx:74HCT00 U23
-U 1 1 5E65E065
-P 8775 1400
-F 0 "U23" H 8775 1725 50  0000 C CNN
-F 1 "74HCT00" H 8775 1634 50  0000 C CNN
-F 2 "Housings_SOIC:SOIC-14_3.9x8.7mm_Pitch1.27mm" H 8775 1400 50  0001 C CNN
-F 3 "http://www.ti.com/lit/gpn/sn74hct00" H 8775 1400 50  0001 C CNN
-	1    8775 1400
-	1    0    0    -1
-$EndComp
 $Comp
 L 74xx:74HCT00 U23
@@
 Wire Wire Line
 	6525 6200 6400 6200
+Text Label 5750 3575 0    50   ~ 0
+~A1
+$Comp
+L 74xx:74HCT00 U23
+U 1 1 5E65E065
+P 8775 1400
+F 0 "U23" H 8775 1175 50  0000 C CNN
+F 1 "74HCT00" H 8775 1100 50  0000 C CNN
+F 2 "Housings_SOIC:SOIC-14_3.9x8.7mm_Pitch1.27mm" H 8775 1400 50  0001 C CNN
+F 3 "http://www.ti.com/lit/gpn/sn74hct00" H 8775 1400 50  0001 C CNN
+	1    8775 1400
+	1    0    0    -1
+$EndComp
+Wire Wire Line
+	8475 750  8425 750
+Wire Wire Line
+	8425 750  8425 1050
+Wire Wire Line
+	8425 1050 9075 1225
+Wire Wire Line
+	9075 1225 9075 1400
+Connection ~ 9075 1400
+Wire Wire Line
+	9075 850  9075 1000
+Wire Wire Line
+	9075 1000 8425 1175
+Wire Wire Line
+	8425 1175 8425 1300
+Wire Wire Line
+	8425 1300 8475 1300
+Connection ~ 9075 850
 $EndSCHEMATC

Commit message: Change jacks for board (not routed yet)
Parts:
- J5, J6: footprint Connector_Dsub:DSUB-9_Male_Horizontal_P2.77x2.84mm_EdgePinOffset4.94mm_Housed_MountingHolesOffset7.48mm -> Jacks:A-DS 09 A-KG-T2S; DigiKey (none) -> AE10968-ND
Changed lines of the file:
@@
 F 0 "J5" H 2155 2921 50  0000 L CNN
 F 1 "Controller Port 2" H 2155 2830 50  0000 L CNN
-F 2 "Connector_Dsub:DSUB-9_Male_Horizontal_P2.77x2.84mm_EdgePinOffset4.94mm_Housed_MountingHolesOffset7.48mm" H 1975 2875 50  0001 C CNN
-F 3 "https://www.digikey.com/product-detail/en/te-connectivity-amp-connectors/5747250-4/A32072-ND/808627" H 1975 2875 50  0001 C CNN
+F 2 "Jacks:A-DS 09 A-KG-T2S" H 1975 2875 50  0001 C CNN
+F 3 "http://www.assmann-wsw.com/fileadmin/datasheets/ASS_4888_CO.pdf" H 1975 2875 50  0001 C CNN
+F 4 "AE10968-ND" H 1975 2875 50  0001 C CNN "DigiKey"
 	1    1975 2875
 	-1   0    0    -1
@@
 F 0 "J6" H 2155 5271 50  0000 L CNN
 F 1 "Controller Port 1" H 2155 5180 50  0000 L CNN
-F 2 "Connector_Dsub:DSUB-9_Male_Horizontal_P2.77x2.84mm_EdgePinOffset4.94mm_Housed_MountingHolesOffset7.48mm" H 1975 5225 50  0001 C CNN
-F 3 "https://www.digikey.com/product-detail/en/te-connectivity-amp-connectors/5747250-4/A32072-ND/808627 ~" H 1975 5225 50  0001 C CNN
+F 2 "Jacks:A-DS 09 A-KG-T2S" H 1975 5225 50  0001 C CNN
+F 3 "http://www.assmann-wsw.com/fileadmin/datasheets/ASS_4888_CO.pdf" H 1975 5225 50  0001 C CNN
+F 4 "AE10968-ND" H 1975 5225 50  0001 C CNN "DigiKey"
 	1    1975 5225
 	-1   0    0    1
@@
 F 3 "http://www.vishay.com/docs/31509/csc.pdf" H 4675 6000 50  0001 C CNN
 	1    4675 6000
-	1    0    0    1
+	-1   0    0    1
 $EndComp
 Wire Wire Line
@@
 	1    0    0    -1
 $EndComp
-Text Label 4375 6200 3    50   ~ 0
+Text Label 4975 6200 3    50   ~ 0
 2v5
 Text Label 4375 4025 3    50   ~ 0

Commit message: Squashed commit of the following:
commit 92abf32cadf827114d19584acd122949932597b3
Author: mike <barbeque@users.noreply.github.com>
Date:   Mon Jan 3 10:32:57 2022 -0700

    Routing complete for new controller port part

commit b2f35945ec75921dc30cd07b50809f4682bd367a
Author: mike <barbeque@users.noreply.github.com>
Date:   Mon Jan 3 10:19:43 2022 -0700

    Fix the stupid pin assignment

commit 4990d3c33f922ec1addda2a0fcbaea749a56b64e
Author: mike <barbeque@users.noreply.github.com>
Date:   Mon Jan 3 10:18:26 2022 -0700

    Checking numbering on controller port
Changed lines of the file:
@@
 F 3 "http://www.vishay.com/docs/31509/csc.pdf" H 4675 6000 50  0001 C CNN
 	1    4675 6000
-	-1   0    0    1
+	1    0    0    1
 $EndComp
 Wire Wire Line
@@
 	1    0    0    -1
 $EndComp
-Text Label 4975 6200 3    50   ~ 0
+Text Label 4375 6200 3    50   ~ 0
 2v5
 Text Label 4375 4025 3    50   ~ 0

Commit message: v0.7 release notes
Parts:
- J5, J6: DigiKey AE10968-ND -> AE10968-ND
Changed lines of the file:
@@
 F 2 "Jacks:A-DS 09 A-KG-T2S" H 1975 2875 50  0001 C CNN
 F 3 "http://www.assmann-wsw.com/fileadmin/datasheets/ASS_4888_CO.pdf" H 1975 2875 50  0001 C CNN
-F 4 "AE10968-ND" H 1975 2875 50  0001 C CNN "DigiKey"
+F 4 "AE10968-ND" H 1975 2875 50  0001 C CNN "DigiKey"
 	1    1975 2875
 	-1   0    0    -1
@@
 F 2 "Jacks:A-DS 09 A-KG-T2S" H 1975 5225 50  0001 C CNN
 F 3 "http://www.assmann-wsw.com/fileadmin/datasheets/ASS_4888_CO.pdf" H 1975 5225 50  0001 C CNN
-F 4 "AE10968-ND" H 1975 5225 50  0001 C CNN "DigiKey"
+F 4 "AE10968-ND" H 1975 5225 50  0001 C CNN "DigiKey"
 	1    1975 5225
 	-1   0    0    1

Commit message: BOM update
Parts:
- C3, C32: DigiKey (none) -> 732-8059-1-ND
- C33, C34: DigiKey (none) -> 1276-1099-1-ND
- U18: DigiKey (none) -> 296-1630-1-ND
Changed lines of the file:
@@
 F 2 "Capacitors_SMD:C_0805_HandSoldering" H 3463 1700 50  0001 C CNN
 F 3 "~" H 3425 1850 50  0001 C CNN
+F 4 "1276-1099-1-ND" H 3425 1850 50  0001 C CNN "DigiKey"
 	1    3425 1850
 	1    0    0    1
@@
 F 2 "Capacitors_SMD:C_0805_HandSoldering" H 2238 925 50  0001 C CNN
 F 3 "~" H 2200 1075 50  0001 C CNN
+F 4 "732-8059-1-ND" H 2200 1075 50  0001 C CNN "DigiKey"
 	1    2200 1075
 	0    1    1    0
@@
 F 2 "Capacitors_SMD:C_0805_HandSoldering" H 2388 7150 50  0001 C CNN
 F 3 "~" H 2350 7300 50  0001 C CNN
+F 4 "732-8059-1-ND" H 2350 7300 50  0001 C CNN "DigiKey"
 	1    2350 7300
 	0    1    -1   0
@@
 F 2 "Housings_SOIC:SOIC-14_3.9x8.7mm_Pitch1.27mm" H 7400 3725 50  0001 C CNN
 F 3 "http://www.ti.com/lit/gpn/sn74LS05" H 7400 3725 50  0001 C CNN
+F 4 "296-1630-1-ND" H 7400 3725 50  0001 C CNN "DigiKey"
 	4    7400 3725
 	-1   0    0    -1
@@
 F 2 "Capacitors_SMD:C_0805_HandSoldering" H 3613 6675 50  0001 C CNN
 F 3 "~" H 3575 6825 50  0001 C CNN
+F 4 "1276-1099-1-ND" H 3575 6825 50  0001 C CNN "DigiKey"
 	1    3575 6825
 	1    0    0    -1
